Commit message: enable ros2 controller

File: spacediver_ros2_control/description/gazebo/spacediver_gazebo.xacro (robot description, xacro)
@@ -8,5 +8,5 @@
     <!-- ros_control plugin -->
     <plugin filename="libgazebo_ros2_control.so" name="gazebo_ros2_control">
-      <parameters>$(find spacediver_ros2_control)/bringup/config/sar_controllers.yaml</parameters>
+      <parameters>$(find spacediver_ros2_control)/bringup/config/spacediver_controllers.yaml</parameters>
     </plugin>
     <!-- get true robot position plugin -->
@@ -65,16 +65,3 @@
     <provideFeedback>true</provideFeedback>
   </gazebo>
-  <!-- Joint for FT sensor -->
-  <gazebo reference="joint_f">
-    <provideFeedback>true</provideFeedback>
-    <turnGravityOff>false</turnGravityOff>
-  </gazebo>
-  <!-- FT Sensor -->
-  <gazebo>
-    <plugin name="ft_sensor" filename="libgazebo_ros_ft_sensor.so">
-      <updateRate>10.0</updateRate>
-      <body_name>link_6</body_name>
-      <joint_name>joint_f</joint_name>
-    </plugin>
-  </gazebo>
 </robot>

File: spacediver_ros2_control/description/urdf/parts/spacediver_left_arm.xacro (robot description, xacro)
@@ -60,5 +60,5 @@
     </link>
     <!-- Joint 3 -->
-    <joint name="active_joint_c" type="revolute">
+    <joint name="active_joint_lc" type="revolute">
       <parent link="link_2"/>
       <child link="link_3"/>

File: spacediver_ros2_control/description/urdf/parts/spacediver_right.xacro (robot description, xacro)
@@ -6,5 +6,5 @@
   <xacro:macro name="right_arm" params="base_name *origin">
     <!-- Joint 4 -->
-    <joint name="joint_d" type="revolute">
+    <joint name="active_joint_ra" type="revolute">
       <parent link="right_arm"/>
       <child link="link_4"/>
@@ -34,5 +34,5 @@
     </link>
     <!-- Joint 5 -->
-    <joint name="joint_e" type="revolute">
+    <joint name="active_joint_rb" type="revolute">
       <parent link="link_4"/>
       <child link="link_5"/>
@@ -62,5 +62,5 @@
     </link>
     <!-- Joint 6 -->
-    <joint name="joint_f" type="revolute">
+    <joint name="active_joint_rc" type="revolute">
       <parent link="link_5"/>
       <child link="link_6"/>

File: spacediver_ros2_control/description/urdf/spacediver.urdf.xacro (robot description, xacro)
@@ -1,3 +1,4 @@
 <robot name="single_arm_robot" xmlns:xacro="http://ros.org/wiki/xacro">
+  <!-- Include macros -->
   <xacro:include filename="$(find spacediver_ros2_control)/description/urdf/macros/inertial_macros.xacro"/>
   <xacro:include filename="$(find spacediver_ros2_control)/description/urdf/macros/properties.xacro"/>
@@ -14,4 +15,5 @@
   <xacro:include filename="$(find spacediver_ros2_control)/description/gazebo/spacediver_gazebo.xacro" />
   <!-- ros2 control plugin -->
-  <!-- <xacro:include filename="$(find spacediver_ros2_control)/description/ros2_control/spacediver_ros2_control.xacro" /> -->
+  <xacro:include filename="$(find spacediver_ros2_control)/description/ros2_control/spacediver_ros2_control.xacro" />
+  <xacro:ros2_control_hardware use_gazebo="true" />
 </robot>

Commit message: add single arm controller

File: spacediver_ros2_control/description/gazebo/spacediver_gazebo.xacro (robot description, xacro)
@@ -22,46 +22,3 @@
     </plugin>
   </gazebo>
-  <!-- Base link -->
-  <gazebo reference="base_link">
-    <mu1>0.2</mu1>
-    <mu2>0.2</mu2>
-    <material>Gazebo/White</material>
-  </gazebo>
-  <!-- Link 1 -->
-  <gazebo reference="link_1">
-    <mu1>0.8</mu1>
-    <mu2>0.8</mu2>
-    <material>Gazebo/White</material>
-  </gazebo>
-  <!-- Link 2 -->
-  <gazebo reference="link_2">
-    <mu1>0.8</mu1>
-    <mu2>0.8</mu2>
-    <material>Gazebo/White</material>
-  </gazebo>
-  <!-- Link 3 -->
-  <gazebo reference="link_3">
-    <material>Gazebo/White</material>
-  </gazebo>
-  <!-- Link 4 -->
-  <gazebo reference="link_4">
-    <mu1>0.8</mu1>
-    <mu2>0.8</mu2>
-    <material>Gazebo/White</material>
-  </gazebo>
-  <!-- Link 5 -->
-  <gazebo reference="link_5">
-    <mu1>0.8</mu1>
-    <mu2>0.8</mu2>
-    <material>Gazebo/White</material>
-  </gazebo>
-  <!-- Link 6 -->
-  <gazebo reference="link_6">
-    <mu1>0.6</mu1>
-    <mu2>0.6</mu2>
-    <kp>1000.0</kp>
-    <kd>1.0</kd>
-    <material>Gazebo/White</material>
-    <provideFeedback>true</provideFeedback>
-  </gazebo>
 </robot>
