Commit message: simplified urdf + single arm sdf and launch file

File: spacediver_ros2_control/description/urdf/spacediver.urdf.xacro (robot description, xacro)
@@ -1,7 +1,8 @@
 <robot name="single_arm_robot" xmlns:xacro="http://ros.org/wiki/xacro">
   <!-- Include macros -->
-  <xacro:include filename="$(find spacediver_ros2_control)/description/urdf/macros/inertial_macros.xacro"/>
-  <xacro:include filename="$(find spacediver_ros2_control)/description/urdf/macros/properties.xacro"/>
-  <xacro:include filename="$(find spacediver_ros2_control)/description/urdf/macros/materials.xacro"/>
+  <xacro:include
+    filename="$(find spacediver_ros2_control)/description/urdf/macros/inertial_macros.xacro" />
+  <xacro:include filename="$(find spacediver_ros2_control)/description/urdf/macros/properties.xacro" />
+  <xacro:include filename="$(find spacediver_ros2_control)/description/urdf/macros/materials.xacro" />
   <!-- Select if the robot is going to be used in gazebo -->
   <!-- This is set in spacediver.launch.py -->
@@ -9,11 +10,14 @@
   <!-- robot shape and phisics -->
   <!-- Base Link -->
-  <xacro:include filename="$(find spacediver_ros2_control)/description/urdf/parts/spacediver_base.xacro" />
+  <xacro:include
+    filename="$(find spacediver_ros2_control)/description/urdf/parts/spacediver_base.xacro" />
   <!-- Left Arm -->
-  <xacro:include filename="$(find spacediver_ros2_control)/description/urdf/parts/spacediver_left_arm.xacro" />
+  <xacro:include
+    filename="$(find spacediver_ros2_control)/description/urdf/parts/simple_left_arm.xacro" />
   <xacro:left_arm base_name="base_link">
-    <origin xyz="0 0 ${BASE_Z/2}" rpy="0 0 0"/>
+    <origin xyz="0 0 ${BASE_Z/2}" rpy="0 0 0" />
   </xacro:left_arm>
   <!-- ros2 control plugin -->
-  <xacro:include filename="$(find spacediver_ros2_control)/description/ros2_control/spacediver_ros2_control.xacro" />
+  <xacro:include
+    filename="$(find spacediver_ros2_control)/description/ros2_control/spacediver_single_arm_ros2_control.xacro" />
 </robot>
