Commit message: switched joint order

File: spacediver_ros2_control/description/ros2_control/spacediver_single_arm_ros2_control.xacro (robot description, xacro)
@@ -37,7 +37,30 @@
       </xacro:if>
     </joint>
+    <!-- BOTTOM DYNAMIXEL TO MISUMI LN -->
+    <joint name="${LEFT_DYNAMIXELBOT_TO_LEFTMISUMILN_JOINT_NAME}">
+      <param name="id">2</param>
+      <command_interface name="position">
+        <param name="min">${BOT_DYNAMIXEL_LOWER}</param>
+        <param name="max">${BOT_DYNAMIXEL_UPPER}</param>
+      </command_interface>
+      <xacro:if value="$(arg use_gazebo)">
+        <command_interface name="velocity">
+          <param name="min">"-${BOT_DYNAMIXEL_VELOCITY}"</param>
+          <param name="max">" ${BOT_DYNAMIXEL_VELOCITY}"</param>
+        </command_interface>
+        <command_interface name="effort">
+          <param name="min">"-${BOT_DYNAMIXEL_EFFORT}"</param>
+          <param name="max">" ${BOT_DYNAMIXEL_EFFORT}"</param>
+        </command_interface>
+      </xacro:if>
+      <state_interface name="position" />
+      <state_interface name="velocity" />
+      <xacro:if value="$(arg use_gazebo)">
+        <state_interface name="effort" />
+      </xacro:if>
+    </joint>
     <!-- TOP DYNAMIXEL TO DRIVING LINK -->
     <joint name="${LEFTDYNAMIXELTOP_TO_LEFTDRIVING_JOINT_NAME}">
-      <param name="id">2</param>
+      <param name="id">3</param>
       <command_interface name="position">
         <param name="min">${TOP_DYNAMIXEL_LOWER}</param>
@@ -60,27 +83,4 @@
       </xacro:if>
     </joint>
-    <!-- BOTTOM DYNAMIXEL TO MISUMI LN -->
-    <joint name="${LEFT_DYNAMIXELBOT_TO_LEFTMISUMILN_JOINT_NAME}">
-      <param name="id">3</param>
-      <command_interface name="position">
-        <param name="min">${BOT_DYNAMIXEL_LOWER}</param>
-        <param name="max">${BOT_DYNAMIXEL_UPPER}</param>
-      </command_interface>
-      <xacro:if value="$(arg use_gazebo)">
-        <command_interface name="velocity">
-          <param name="min">"-${BOT_DYNAMIXEL_VELOCITY}"</param>
-          <param name="max">" ${BOT_DYNAMIXEL_VELOCITY}"</param>
-        </command_interface>
-        <command_interface name="effort">
-          <param name="min">"-${BOT_DYNAMIXEL_EFFORT}"</param>
-          <param name="max">" ${BOT_DYNAMIXEL_EFFORT}"</param>
-        </command_interface>
-      </xacro:if>
-      <state_interface name="position" />
-      <state_interface name="velocity" />
-      <xacro:if value="$(arg use_gazebo)">
-        <state_interface name="effort" />
-      </xacro:if>
-    </joint>
   </ros2_control>
 </robot>
