Commit message: Update xacros and enable ROS2 controller

File: spacediver_ros2_control/description/ros2_control/spacediver_ros2_control.xacro (robot description, xacro)
@@ -1,125 +1,123 @@
 <?xml version="1.0"?>
 <robot xmlns:xacro="http://www.ros.org/wiki/xacro">
-  <xacro:macro name="ros2_control_hardware" params="use_gazebo">
-    <ros2_control name="spacediver" type="system">
-      <xacro:if value="${use_gazebo}">
-        <hardware>
-          <plugin>gazebo_ros2_control/GazeboSystem</plugin>
-        </hardware>
-      </xacro:if>
-      <xacro:unless value="${use_gazebo}">
-        <hardware>
-          <plugin>spacediver_ros2_control/SpacediverSystem</plugin>
-        </hardware>
-      </xacro:unless>
-      <!-- Joint 1 -->
-      <joint name="active_joint_la">
-        <command_interface name="position">
-          <param name="min">"${ACTIVE_JOINT_LA_LOWER}"</param>
-          <param name="max">"${ACTIVE_JOINT_LA_UPPER}"</param>
-        </command_interface>
-        <command_interface name="velocity">
-          <param name="min">"-${ACTIVE_JOINT_LA_VELOCITY}"</param>
-          <param name="max">" ${ACTIVE_JOINT_LA_VELOCITY}"</param>
-        </command_interface>
-        <command_interface name="effort">
-          <param name="min">"-${ACTIVE_JOINT_LA_EFFORT}"</param>
-          <param name="max">" ${ACTIVE_JOINT_LA_EFFORT}"</param>
-        </command_interface>
-        <state_interface name="position"/>
-        <state_interface name="velocity"/>
-        <state_interface name="effort"/>
-      </joint>
-      <!-- Joint 2 -->
-      <joint name="active_joint_lb">
-        <command_interface name="position">
-          <param name="min">"${ACTIVE_JOINT_LB_LOWER}"</param>
-          <param name="max">"${ACTIVE_JOINT_LB_UPPER}"</param>
-        </command_interface>
-        <command_interface name="velocity">
-          <param name="min">"-${ACTIVE_JOINT_LB_VELOCITY}"</param>
-          <param name="max">" ${ACTIVE_JOINT_LB_VELOCITY}"</param>
-        </command_interface>
-        <command_interface name="effort">
-          <param name="min">"-${ACTIVE_JOINT_LB_EFFORT}"</param>
-          <param name="max">" ${ACTIVE_JOINT_LB_EFFORT}"</param>
-        </command_interface>
-        <state_interface name="position"/>
-        <state_interface name="velocity"/>
-        <state_interface name="effort"/>
-      </joint>
-      <!-- Joint 3 -->
-      <joint name="active_joint_lc">
-        <command_interface name="position">
-          <param name="min">"${ACTIVE_JOINT_LC_LOWER}"</param>
-          <param name="max">"${ACTIVE_JOINT_LC_UPPER}"</param>
-        </command_interface>
-        <command_interface name="velocity">
-          <param name="min">"-${ACTIVE_JOINT_LC_VELOCITY}"</param>
-          <param name="max">" ${ACTIVE_JOINT_LC_VELOCITY}"</param>
-        </command_interface>
-        <command_interface name="effort">
-          <param name="min">"-${ACTIVE_JOINT_LC_EFFORT}"</param>
-          <param name="max">" ${ACTIVE_JOINT_LC_EFFORT}"</param>
-        </command_interface>
-        <state_interface name="position"/>
-        <state_interface name="velocity"/>
-        <state_interface name="effort"/>
-      </joint>
-      <!-- Joint 4 -->
-      <joint name="active_joint_ra">
-        <command_interface name="position">
-          <param name="min">"-${ACTIVE_JOINT_RA_UPPER}"</param>
-          <param name="max">"-${ACTIVE_JOINT_RA_LOWER}"</param>
-        </command_interface>
-        <command_interface name="velocity">
-          <param name="min">"-${ACTIVE_JOINT_RA_VELOCITY}"</param>
-          <param name="max">" ${ACTIVE_JOINT_RA_VELOCITY}"</param>
-        </command_interface>
-        <command_interface name="effort">
-          <param name="min">"-${ACTIVE_JOINT_RA_EFFORT}"</param>
-          <param name="max">" ${ACTIVE_JOINT_RA_EFFORT}"</param>
-        </command_interface>
-        <state_interface name="position"/>
-        <state_interface name="velocity"/>
-        <state_interface name="effort"/>
-      </joint>
-      <!-- Joint 5 -->
-      <joint name="active_joint_rb">
-        <command_interface name="position">
-          <param name="min">"-${ACTIVE_JOINT_RB_UPPER}"</param>
-          <param name="max">"-${ACTIVE_JOINT_RB_LOWER}"</param>
-        </command_interface>
-        <command_interface name="velocity">
-          <param name="min">"-${ACTIVE_JOINT_RB_VELOCITY}"</param>
-          <param name="max">" ${ACTIVE_JOINT_RB_VELOCITY}"</param>
-        </command_interface>
-        <command_interface name="effort">
-          <param name="min">"-${ACTIVE_JOINT_RB_EFFORT}"</param>
-          <param name="max">" ${ACTIVE_JOINT_RB_EFFORT}"</param>
-        </command_interface>
-        <state_interface name="position"/>
-        <state_interface name="velocity"/>
-        <state_interface name="effort"/>
-      </joint>
-      <!-- Joint 6 -->
-      <joint name="active_joint_rc">
-        <command_interface name="position">
-          <param name="min">"-${ACTIVE_JOINT_RC_UPPER}"</param>
-          <param name="max">"-${ACTIVE_JOINT_RC_LOWER}"</param>
-        </command_interface>
-        <command_interface name="velocity">
-          <param name="min">"-${ACTIVE_JOINT_RC_VELOCITY}"</param>
-          <param name="max">" ${ACTIVE_JOINT_RC_VELOCITY}"</param>
-        </command_interface>
-        <command_interface name="effort">
-          <param name="min">"-${ACTIVE_JOINT_RC_EFFORT}"</param>
-          <param name="max">" ${ACTIVE_JOINT_RC_EFFORT}"</param>
-        </command_interface>
-        <state_interface name="position"/>
-        <state_interface name="velocity"/>
-        <state_interface name="effort"/>
-      </joint>
-    </ros2_control>
-  </xacro:macro>
+  <ros2_control name="spacediver" type="system">
+    <xacro:if value="$(arg use_gazebo)">
+      <hardware>
+        <plugin>gazebo_ros2_control/GazeboSystem</plugin>
+      </hardware>
+    </xacro:if>
+    <xacro:unless value="$(arg use_gazebo)">
+      <hardware>
+        <plugin>spacediver_ros2_control/SpacediverSystem</plugin>
+      </hardware>
+    </xacro:unless>
+    <!-- Joint 1 -->
+    <joint name="active_joint_la">
+      <command_interface name="position">
+        <param name="min">"${ACTIVE_JOINT_LA_LOWER}"</param>
+        <param name="max">"${ACTIVE_JOINT_LA_UPPER}"</param>
+      </command_interface>
+      <command_interface name="velocity">
+        <param name="min">"-${ACTIVE_JOINT_LA_VELOCITY}"</param>
+        <param name="max">" ${ACTIVE_JOINT_LA_VELOCITY}"</param>
+      </command_interface>
+      <command_interface name="effort">
+        <param name="min">"-${ACTIVE_JOINT_LA_EFFORT}"</param>
+        <param name="max">" ${ACTIVE_JOINT_LA_EFFORT}"</param>
+      </command_interface>
+      <state_interface name="position"/>
+      <state_interface name="velocity"/>
+      <state_interface name="effort"/>
+    </joint>
+    <!-- Joint 2 -->
+    <joint name="active_joint_lb">
+      <command_interface name="position">
+        <param name="min">"${ACTIVE_JOINT_LB_LOWER}"</param>
+        <param name="max">"${ACTIVE_JOINT_LB_UPPER}"</param>
+      </command_interface>
+      <command_interface name="velocity">
+        <param name="min">"-${ACTIVE_JOINT_LB_VELOCITY}"</param>
+        <param name="max">" ${ACTIVE_JOINT_LB_VELOCITY}"</param>
+      </command_interface>
+      <command_interface name="effort">
+        <param name="min">"-${ACTIVE_JOINT_LB_EFFORT}"</param>
+        <param name="max">" ${ACTIVE_JOINT_LB_EFFORT}"</param>
+      </command_interface>
+      <state_interface name="position"/>
+      <state_interface name="velocity"/>
+      <state_interface name="effort"/>
+    </joint>
+    <!-- Joint 3 -->
+    <joint name="active_joint_lc">
+      <command_interface name="position">
+        <param name="min">"${ACTIVE_JOINT_LC_LOWER}"</param>
+        <param name="max">"${ACTIVE_JOINT_LC_UPPER}"</param>
+      </command_interface>
+      <command_interface name="velocity">
+        <param name="min">"-${ACTIVE_JOINT_LC_VELOCITY}"</param>
+        <param name="max">" ${ACTIVE_JOINT_LC_VELOCITY}"</param>
+      </command_interface>
+      <command_interface name="effort">
+        <param name="min">"-${ACTIVE_JOINT_LC_EFFORT}"</param>
+        <param name="max">" ${ACTIVE_JOINT_LC_EFFORT}"</param>
+      </command_interface>
+      <state_interface name="position"/>
+      <state_interface name="velocity"/>
+      <state_interface name="effort"/>
+    </joint>
+    <!-- Joint 4 -->
+    <joint name="active_joint_ra">
+      <command_interface name="position">
+        <param name="min">"-${ACTIVE_JOINT_RA_UPPER}"</param>
+        <param name="max">"-${ACTIVE_JOINT_RA_LOWER}"</param>
+      </command_interface>
+      <command_interface name="velocity">
+        <param name="min">"-${ACTIVE_JOINT_RA_VELOCITY}"</param>
+        <param name="max">" ${ACTIVE_JOINT_RA_VELOCITY}"</param>
+      </command_interface>
+      <command_interface name="effort">
+        <param name="min">"-${ACTIVE_JOINT_RA_EFFORT}"</param>
+        <param name="max">" ${ACTIVE_JOINT_RA_EFFORT}"</param>
+      </command_interface>
+      <state_interface name="position"/>
+      <state_interface name="velocity"/>
+      <state_interface name="effort"/>
+    </joint>
+    <!-- Joint 5 -->
+    <joint name="active_joint_rb">
+      <command_interface name="position">
+        <param name="min">"-${ACTIVE_JOINT_RB_UPPER}"</param>
+        <param name="max">"-${ACTIVE_JOINT_RB_LOWER}"</param>
+      </command_interface>
+      <command_interface name="velocity">
+        <param name="min">"-${ACTIVE_JOINT_RB_VELOCITY}"</param>
+        <param name="max">" ${ACTIVE_JOINT_RB_VELOCITY}"</param>
+      </command_interface>
+      <command_interface name="effort">
+        <param name="min">"-${ACTIVE_JOINT_RB_EFFORT}"</param>
+        <param name="max">" ${ACTIVE_JOINT_RB_EFFORT}"</param>
+      </command_interface>
+      <state_interface name="position"/>
+      <state_interface name="velocity"/>
+      <state_interface name="effort"/>
+    </joint>
+    <!-- Joint 6 -->
+    <joint name="active_joint_rc">
+      <command_interface name="position">
+        <param name="min">"-${ACTIVE_JOINT_RC_UPPER}"</param>
+        <param name="max">"-${ACTIVE_JOINT_RC_LOWER}"</param>
+      </command_interface>
+      <command_interface name="velocity">
+        <param name="min">"-${ACTIVE_JOINT_RC_VELOCITY}"</param>
+        <param name="max">" ${ACTIVE_JOINT_RC_VELOCITY}"</param>
+      </command_interface>
+      <command_interface name="effort">
+        <param name="min">"-${ACTIVE_JOINT_RC_EFFORT}"</param>
+        <param name="max">" ${ACTIVE_JOINT_RC_EFFORT}"</param>
+      </command_interface>
+      <state_interface name="position"/>
+      <state_interface name="velocity"/>
+      <state_interface name="effort"/>
+    </joint>
+  </ros2_control>
 </robot>

File: spacediver_ros2_control/description/urdf/spacediver.urdf.xacro (robot description, xacro)
@@ -4,4 +4,7 @@
   <xacro:include filename="$(find spacediver_ros2_control)/description/urdf/macros/properties.xacro"/>
   <xacro:include filename="$(find spacediver_ros2_control)/description/urdf/macros/materials.xacro"/>
+  <!-- Select if the robot is going to be used in gazebo -->
+  <!-- This is set in spacediver.launch.py -->
+  <xacro:arg name="use_gazebo" default="true" />
   <!-- robot shape and phisics -->
   <!-- Base Link -->
@@ -16,4 +19,3 @@
   <!-- ros2 control plugin -->
   <xacro:include filename="$(find spacediver_ros2_control)/description/ros2_control/spacediver_ros2_control.xacro" />
-  <xacro:ros2_control_hardware use_gazebo="true" />
 </robot>

Commit message: removing and replacing placeholder joints

File: spacediver_ros2_control/description/ros2_control/spacediver_ros2_control.xacro (robot description, xacro)
@@ -118,112 +118,4 @@
       <state_interface name="effort"/>
     </joint>
-    <!-- Joint 1 -->
-    <joint name="active_joint_la">
-      <command_interface name="position">
-        <param name="min">"${ACTIVE_JOINT_LA_LOWER}"</param>
-        <param name="max">"${ACTIVE_JOINT_LA_UPPER}"</param>
-      </command_interface>
-      <command_interface name="velocity">
-        <param name="min">"-${ACTIVE_JOINT_LA_VELOCITY}"</param>
-        <param name="max">" ${ACTIVE_JOINT_LA_VELOCITY}"</param>
-      </command_interface>
-      <command_interface name="effort">
-        <param name="min">"-${ACTIVE_JOINT_LA_EFFORT}"</param>
-        <param name="max">" ${ACTIVE_JOINT_LA_EFFORT}"</param>
-      </command_interface>
-      <state_interface name="position"/>
-      <state_interface name="velocity"/>
-      <state_interface name="effort"/>
-    </joint>
-    <!-- Joint 2 -->
-    <joint name="active_joint_lb">
-      <command_interface name="position">
-        <param name="min">"${ACTIVE_JOINT_LB_LOWER}"</param>
-        <param name="max">"${ACTIVE_JOINT_LB_UPPER}"</param>
-      </command_interface>
-      <command_interface name="velocity">
-        <param name="min">"-${ACTIVE_JOINT_LB_VELOCITY}"</param>
-        <param name="max">" ${ACTIVE_JOINT_LB_VELOCITY}"</param>
-      </command_interface>
-      <command_interface name="effort">
-        <param name="min">"-${ACTIVE_JOINT_LB_EFFORT}"</param>
-        <param name="max">" ${ACTIVE_JOINT_LB_EFFORT}"</param>
-      </command_interface>
-      <state_interface name="position"/>
-      <state_interface name="velocity"/>
-      <state_interface name="effort"/>
-    </joint>
-    <!-- Joint 3 -->
-    <joint name="active_joint_lc">
-      <command_interface name="position">
-        <param name="min">"${ACTIVE_JOINT_LC_LOWER}"</param>
-        <param name="max">"${ACTIVE_JOINT_LC_UPPER}"</param>
-      </command_interface>
-      <command_interface name="velocity">
-        <param name="min">"-${ACTIVE_JOINT_LC_VELOCITY}"</param>
-        <param name="max">" ${ACTIVE_JOINT_LC_VELOCITY}"</param>
-      </command_interface>
-      <command_interface name="effort">
-        <param name="min">"-${ACTIVE_JOINT_LC_EFFORT}"</param>
-        <param name="max">" ${ACTIVE_JOINT_LC_EFFORT}"</param>
-      </command_interface>
-      <state_interface name="position"/>
-      <state_interface name="velocity"/>
-      <state_interface name="effort"/>
-    </joint>
-    <!-- Joint 4 -->
-    <joint name="active_joint_ra">
-      <command_interface name="position">
-        <param name="min">"-${ACTIVE_JOINT_RA_UPPER}"</param>
-        <param name="max">"-${ACTIVE_JOINT_RA_LOWER}"</param>
-      </command_interface>
-      <command_interface name="velocity">
-        <param name="min">"-${ACTIVE_JOINT_RA_VELOCITY}"</param>
-        <param name="max">" ${ACTIVE_JOINT_RA_VELOCITY}"</param>
-      </command_interface>
-      <command_interface name="effort">
-        <param name="min">"-${ACTIVE_JOINT_RA_EFFORT}"</param>
-        <param name="max">" ${ACTIVE_JOINT_RA_EFFORT}"</param>
-      </command_interface>
-      <state_interface name="position"/>
-      <state_interface name="velocity"/>
-      <state_interface name="effort"/>
-    </joint>
-    <!-- Joint 5 -->
-    <joint name="active_joint_rb">
-      <command_interface name="position">
-        <param name="min">"-${ACTIVE_JOINT_RB_UPPER}"</param>
-        <param name="max">"-${ACTIVE_JOINT_RB_LOWER}"</param>
-      </command_interface>
-      <command_interface name="velocity">
-        <param name="min">"-${ACTIVE_JOINT_RB_VELOCITY}"</param>
-        <param name="max">" ${ACTIVE_JOINT_RB_VELOCITY}"</param>
-      </command_interface>
-      <command_interface name="effort">
-        <param name="min">"-${ACTIVE_JOINT_RB_EFFORT}"</param>
-        <param name="max">" ${ACTIVE_JOINT_RB_EFFORT}"</param>
-      </command_interface>
-      <state_interface name="position"/>
-      <state_interface name="velocity"/>
-      <state_interface name="effort"/>
-    </joint>
-    <!-- Joint 6 -->
-    <joint name="active_joint_rc">
-      <command_interface name="position">
-        <param name="min">"-${ACTIVE_JOINT_RC_UPPER}"</param>
-        <param name="max">"-${ACTIVE_JOINT_RC_LOWER}"</param>
-      </command_interface>
-      <command_interface name="velocity">
-        <param name="min">"-${ACTIVE_JOINT_RC_VELOCITY}"</param>
-        <param name="max">" ${ACTIVE_JOINT_RC_VELOCITY}"</param>
-      </command_interface>
-      <command_interface name="effort">
-        <param name="min">"-${ACTIVE_JOINT_RC_EFFORT}"</param>
-        <param name="max">" ${ACTIVE_JOINT_RC_EFFORT}"</param>
-      </command_interface>
-      <state_interface name="position"/>
-      <state_interface name="velocity"/>
-      <state_interface name="effort"/>
-    </joint>
   </ros2_control>
 </robot>

Commit message: changed hardware to DynamixelHardware

File: spacediver_ros2_control/description/ros2_control/spacediver_ros2_control.xacro (robot description, xacro)
@@ -2,5 +2,5 @@
 <robot xmlns:xacro="http://www.ros.org/wiki/xacro">
   <ros2_control name="spacediver" type="system">
-    <xacro:if value="$(arg use_gazebo)">
+    <!-- <xacro:if value="$(arg use_gazebo)">
       <hardware>
         <plugin>gazebo_ros2_control/GazeboSystem</plugin>
@@ -11,5 +11,10 @@
         <plugin>spacediver_ros2_control/SpacediverSystem</plugin>
       </hardware>
-    </xacro:unless>
+    </xacro:unless> -->
+    <hardware>
+      <plugin>dynamixel_hardware/DynamixelHardware</plugin>
+      <param name="usb_port">"/dev/ttyUSB0"</param>
+      <param name="baud_rate">57600</param>
+    </hardware>
     <!-- BASE TO LEFT SHOULDER PLATE -->
     <joint name="base_to_leftshoulder_joint">
@@ -32,5 +37,5 @@
     </joint>
     <!-- BASE TO RIGHT SHOULDER PLATE -->
-    <joint name="base_to_rightshoulder_joint">
+    <!-- <joint name="base_to_rightshoulder_joint">
       <command_interface name="position">
         <param name="min">"${BASE_DYNAMIXEL_UPPER}"</param>
@@ -48,5 +53,5 @@
       <state_interface name="velocity"/>
       <state_interface name="effort"/>
-    </joint>
+    </joint> -->
     <!-- TOP DYNAMIXEL TO DRIVING LINK -->
     <joint name="leftdynamixeltop_to_leftdriving_joint">
@@ -68,5 +73,5 @@
       <state_interface name="effort"/>
     </joint>
-    <joint name="rightdynamixeltop_to_rightdriving_joint">
+    <!-- <joint name="rightdynamixeltop_to_rightdriving_joint">
       <command_interface name="position">
         <param name="min">"${TOP_DYNAMIXEL_UPPER}"</param>
@@ -84,5 +89,5 @@
       <state_interface name="velocity"/>
       <state_interface name="effort"/>
-    </joint>
+    </joint> -->
     <!-- BOTTOM DYNAMIXEL TO MISUMI LN -->
     <joint name="leftdynamixelbottom_to_leftmisumiln_joint">
@@ -104,5 +109,5 @@
       <state_interface name="effort"/>
     </joint>
-    <joint name="rightdynamixelbottom_to_rightmisumiln_joint">
+    <!-- <joint name="rightdynamixelbottom_to_rightmisumiln_joint">
       <command_interface name="position">
         <param name="min">"${BOT_DYNAMIXEL_UPPER}"</param>
@@ -120,5 +125,5 @@
       <state_interface name="velocity"/>
       <state_interface name="effort"/>
-    </joint>
+    </joint> -->
   </ros2_control>
 </robot>

Commit message: uncommented right arm's joints in ros2_control file

File: spacediver_ros2_control/description/ros2_control/spacediver_ros2_control.xacro (robot description, xacro)
@@ -37,10 +37,11 @@
     </joint>
     <!-- BASE TO RIGHT SHOULDER PLATE -->
-    <!-- <joint name="base_to_rightshoulder_joint">
+    <joint name="base_to_rightshoulder_joint">
+      <param name="id">4</param>
       <command_interface name="position">
         <param name="min">"${BASE_DYNAMIXEL_UPPER}"</param>
         <param name="max">"${BASE_DYNAMIXEL_LOWER}"</param>
       </command_interface>
-      <command_interface name="velocity">
+      <!-- <command_interface name="velocity">
         <param name="min">"-${BASE_DYNAMIXEL_VELOCITY}"</param>
         <param name="max">" ${BASE_DYNAMIXEL_VELOCITY}"</param>
@@ -49,9 +50,9 @@
         <param name="min">"-${BASE_DYNAMIXEL_EFFORT}"</param>
         <param name="max">" ${BASE_DYNAMIXEL_EFFORT}"</param>
-      </command_interface>
+      </command_interface> -->
       <state_interface name="position"/>
       <state_interface name="velocity"/>
-      <state_interface name="effort"/>
-    </joint> -->
+      <!-- <state_interface name="effort"/> -->
+    </joint>
     <!-- TOP DYNAMIXEL TO DRIVING LINK -->
     <joint name="leftdynamixeltop_to_leftdriving_joint">
@@ -73,10 +74,11 @@
       <!-- <state_interface name="effort"/> -->
     </joint>
-    <!-- <joint name="rightdynamixeltop_to_rightdriving_joint">
+    <joint name="rightdynamixeltop_to_rightdriving_joint">
+      <param name="id">5</param>
       <command_interface name="position">
         <param name="min">"${TOP_DYNAMIXEL_UPPER}"</param>
         <param name="max">"${TOP_DYNAMIXEL_LOWER}"</param>
       </command_interface>
-      <command_interface name="velocity">
+      <!-- <command_interface name="velocity">
         <param name="min">"-${TOP_DYNAMIXEL_VELOCITY}"</param>
         <param name="max">" ${TOP_DYNAMIXEL_VELOCITY}"</param>
@@ -85,9 +87,9 @@
         <param name="min">"-${TOP_DYNAMIXEL_EFFORT}"</param>
         <param name="max">" ${TOP_DYNAMIXEL_EFFORT}"</param>
-      </command_interface>
+      </command_interface> -->
       <state_interface name="position"/>
       <state_interface name="velocity"/>
-      <state_interface name="effort"/>
-    </joint> -->
+      <!-- <state_interface name="effort"/> -->
+    </joint>
     <!-- BOTTOM DYNAMIXEL TO MISUMI LN -->
     <joint name="leftdynamixelbottom_to_leftmisumiln_joint">
@@ -109,10 +111,11 @@
       <!-- <state_interface name="effort"/> -->
     </joint>
-    <!-- <joint name="rightdynamixelbottom_to_rightmisumiln_joint">
+    <joint name="rightdynamixelbottom_to_rightmisumiln_joint">
+      <param name="id">6</param>
       <command_interface name="position">
         <param name="min">"${BOT_DYNAMIXEL_UPPER}"</param>
         <param name="max">"${BOT_DYNAMIXEL_LOWER}"</param>
       </command_interface>
-      <command_interface name="velocity">
+      <!-- <command_interface name="velocity">
         <param name="min">"-${BOT_DYNAMIXEL_VELOCITY}"</param>
         <param name="max">" ${BOT_DYNAMIXEL_VELOCITY}"</param>
@@ -121,9 +124,9 @@
         <param name="min">"-${BOT_DYNAMIXEL_EFFORT}"</param>
         <param name="max">" ${BOT_DYNAMIXEL_EFFORT}"</param>
-      </command_interface>
+      </command_interface> -->
       <state_interface name="position"/>
       <state_interface name="velocity"/>
-      <state_interface name="effort"/>
-    </joint> -->
+      <!-- <state_interface name="effort"/> -->
+    </joint>
   </ros2_control>
 </robot>
