Commit message: commented out right arm's joints

File: spacediver_ros2_control/description/ros2_control/spacediver_ros2_control.xacro (robot description, xacro)
@@ -17,5 +17,5 @@
       <param name="baud_rate">57600</param>
     </hardware>
-    <!-- BASE TO LEFT SHOULDER PLATE -->
+    <!-- BASE TO SHOULDER PLATE -->
     <joint name="base_to_leftshoulder_joint">
       <param name="id">1</param>
@@ -36,6 +36,5 @@
       <!-- <state_interface name="effort"/> -->
     </joint>
-    <!-- BASE TO RIGHT SHOULDER PLATE -->
-    <joint name="base_to_rightshoulder_joint">
+    <!-- <joint name="base_to_rightshoulder_joint">
       <param name="id">4</param>
       <command_interface name="position">
@@ -43,16 +42,7 @@
         <param name="max">"${BASE_DYNAMIXEL_LOWER}"</param>
       </command_interface>
-      <!-- <command_interface name="velocity">
-        <param name="min">"-${BASE_DYNAMIXEL_VELOCITY}"</param>
-        <param name="max">" ${BASE_DYNAMIXEL_VELOCITY}"</param>
-      </command_interface>
-      <command_interface name="effort">
-        <param name="min">"-${BASE_DYNAMIXEL_EFFORT}"</param>
-        <param name="max">" ${BASE_DYNAMIXEL_EFFORT}"</param>
-      </command_interface> -->
       <state_interface name="position"/>
       <state_interface name="velocity"/>
-      <!-- <state_interface name="effort"/> -->
-    </joint>
+    </joint> -->
     <!-- TOP DYNAMIXEL TO DRIVING LINK -->
     <joint name="leftdynamixeltop_to_leftdriving_joint">
@@ -74,5 +64,5 @@
       <!-- <state_interface name="effort"/> -->
     </joint>
-    <joint name="rightdynamixeltop_to_rightdriving_joint">
+    <!-- <joint name="rightdynamixeltop_to_rightdriving_joint">
       <param name="id">5</param>
       <command_interface name="position">
@@ -80,16 +70,7 @@
         <param name="max">"${TOP_DYNAMIXEL_LOWER}"</param>
       </command_interface>
-      <!-- <command_interface name="velocity">
-        <param name="min">"-${TOP_DYNAMIXEL_VELOCITY}"</param>
-        <param name="max">" ${TOP_DYNAMIXEL_VELOCITY}"</param>
-      </command_interface>
-      <command_interface name="effort">
-        <param name="min">"-${TOP_DYNAMIXEL_EFFORT}"</param>
-        <param name="max">" ${TOP_DYNAMIXEL_EFFORT}"</param>
-      </command_interface> -->
       <state_interface name="position"/>
       <state_interface name="velocity"/>
-      <!-- <state_interface name="effort"/> -->
-    </joint>
+    </joint> -->
     <!-- BOTTOM DYNAMIXEL TO MISUMI LN -->
     <joint name="leftdynamixelbottom_to_leftmisumiln_joint">
@@ -111,5 +92,5 @@
       <!-- <state_interface name="effort"/> -->
     </joint>
-    <joint name="rightdynamixelbottom_to_rightmisumiln_joint">
+    <!-- <joint name="rightdynamixelbottom_to_rightmisumiln_joint">
       <param name="id">6</param>
       <command_interface name="position">
@@ -117,16 +98,7 @@
         <param name="max">"${BOT_DYNAMIXEL_LOWER}"</param>
       </command_interface>
-      <!-- <command_interface name="velocity">
-        <param name="min">"-${BOT_DYNAMIXEL_VELOCITY}"</param>
-        <param name="max">" ${BOT_DYNAMIXEL_VELOCITY}"</param>
-      </command_interface>
-      <command_interface name="effort">
-        <param name="min">"-${BOT_DYNAMIXEL_EFFORT}"</param>
-        <param name="max">" ${BOT_DYNAMIXEL_EFFORT}"</param>
-      </command_interface> -->
       <state_interface name="position"/>
       <state_interface name="velocity"/>
-      <!-- <state_interface name="effort"/> -->
-    </joint>
+    </joint> -->
   </ros2_control>
 </robot>

Commit message: additional command interfaces and right arm joints only for gazebo

File: spacediver_ros2_control/description/ros2_control/spacediver_ros2_control.xacro (robot description, xacro)
@@ -2,5 +2,5 @@
 <robot xmlns:xacro="http://www.ros.org/wiki/xacro">
   <ros2_control name="spacediver" type="system">
-    <!-- <xacro:if value="$(arg use_gazebo)">
+    <xacro:if value="$(arg use_gazebo)">
       <hardware>
         <plugin>gazebo_ros2_control/GazeboSystem</plugin>
@@ -9,14 +9,11 @@
     <xacro:unless value="$(arg use_gazebo)">
       <hardware>
-        <plugin>spacediver_ros2_control/SpacediverSystem</plugin>
+        <plugin>dynamixel_hardware/DynamixelHardware</plugin>
+        <param name="usb_port">/dev/ttyUSB0</param>
+        <param name="baud_rate">57600</param>
       </hardware>
-    </xacro:unless> -->
-    <hardware>
-      <plugin>dynamixel_hardware/DynamixelHardware</plugin>
-      <param name="usb_port">/dev/ttyUSB0</param>
-      <param name="baud_rate">57600</param>
-    </hardware>
+    </xacro:unless>
     <!-- BASE TO SHOULDER PLATE -->
-    <joint name="base_to_leftshoulder_joint">
+    <joint name="${BASE_TO_LEFTSHOULDER_JOINT_NAME}">
       <param name="id">1</param>
       <command_interface name="position">
@@ -24,27 +21,42 @@
         <param name="max">${BASE_DYNAMIXEL_UPPER}</param>
       </command_interface>
-      <!-- <command_interface name="velocity">
-        <param name="min">"-${BASE_DYNAMIXEL_VELOCITY}"</param>
-        <param name="max">" ${BASE_DYNAMIXEL_VELOCITY}"</param>
-      </command_interface>
-      <command_interface name="effort">
-        <param name="min">"-${BASE_DYNAMIXEL_EFFORT}"</param>
-        <param name="max">" ${BASE_DYNAMIXEL_EFFORT}"</param>
-      </command_interface> -->
-      <state_interface name="position"/>
-      <state_interface name="velocity"/>
-      <!-- <state_interface name="effort"/> -->
+      <xacro:if value="$(arg use_gazebo)">
+        <command_interface name="velocity">
+          <param name="min">"-${BASE_DYNAMIXEL_VELOCITY}"</param>
+          <param name="max">" ${BASE_DYNAMIXEL_VELOCITY}"</param>
+        </command_interface>
+        <command_interface name="effort">
+          <param name="min">"-${BASE_DYNAMIXEL_EFFORT}"</param>
+          <param name="max">" ${BASE_DYNAMIXEL_EFFORT}"</param>
+        </command_interface>
+      </xacro:if>
+      <state_interface name="position" />
+      <state_interface name="velocity" />
+      <xacro:if value="$(arg use_gazebo)">
+        <state_interface name="effort" />
+      </xacro:if>
     </joint>
-    <!-- <joint name="base_to_rightshoulder_joint">
-      <param name="id">4</param>
-      <command_interface name="position">
-        <param name="min">"${BASE_DYNAMIXEL_UPPER}"</param>
-        <param name="max">"${BASE_DYNAMIXEL_LOWER}"</param>
-      </command_interface>
-      <state_interface name="position"/>
-      <state_interface name="velocity"/>
-    </joint> -->
+    <xacro:if value="$(arg use_gazebo)">
+      <joint name="${BASE_TO_RIGHTSHOULDER_JOINT_NAME}">
+        <param name="id">4</param>
+        <command_interface name="position">
+          <param name="min">"${BASE_DYNAMIXEL_UPPER}"</param>
+          <param name="max">"${BASE_DYNAMIXEL_LOWER}"</param>
+        </command_interface>
+        <command_interface name="velocity">
+          <param name="min">"-${BASE_DYNAMIXEL_VELOCITY}"</param>
+          <param name="max">" ${BASE_DYNAMIXEL_VELOCITY}"</param>
+        </command_interface>
+        <command_interface name="effort">
+          <param name="min">"-${BASE_DYNAMIXEL_EFFORT}"</param>
+          <param name="max">" ${BASE_DYNAMIXEL_EFFORT}"</param>
+        </command_interface>
+        <state_interface name="position" />
+        <state_interface name="velocity" />
+        <state_interface name="effort" />
+      </joint>
+    </xacro:if>
     <!-- TOP DYNAMIXEL TO DRIVING LINK -->
-    <joint name="leftdynamixeltop_to_leftdriving_joint">
+    <joint name="${LEFTDYNAMIXELTOP_TO_LEFTDRIVING_JOINT_NAME}">
       <param name="id">2</param>
       <command_interface name="position">
@@ -52,27 +64,42 @@
         <param name="max">${TOP_DYNAMIXEL_UPPER}</param>
       </command_interface>
-      <!-- <command_interface name="velocity">
-        <param name="min">"-${TOP_DYNAMIXEL_VELOCITY}"</param>
-        <param name="max">" ${TOP_DYNAMIXEL_VELOCITY}"</param>
-      </command_interface>
-      <command_interface name="effort">
-        <param name="min">"-${TOP_DYNAMIXEL_EFFORT}"</param>
-        <param name="max">" ${TOP_DYNAMIXEL_EFFORT}"</param>
-      </command_interface> -->
-      <state_interface name="position"/>
-      <state_interface name="velocity"/>
-      <!-- <state_interface name="effort"/> -->
+      <xacro:if value="$(arg use_gazebo)">
+        <command_interface name="velocity">
+          <param name="min">"-${BASE_DYNAMIXEL_VELOCITY}"</param>
+          <param name="max">" ${BASE_DYNAMIXEL_VELOCITY}"</param>
+        </command_interface>
+        <command_interface name="effort">
+          <param name="min">"-${BASE_DYNAMIXEL_EFFORT}"</param>
+          <param name="max">" ${BASE_DYNAMIXEL_EFFORT}"</param>
+        </command_interface>
+      </xacro:if>
+      <state_interface name="position" />
+      <state_interface name="velocity" />
+      <xacro:if value="$(arg use_gazebo)">
+        <state_interface name="effort" />
+      </xacro:if>
     </joint>
-    <!-- <joint name="rightdynamixeltop_to_rightdriving_joint">
-      <param name="id">5</param>
-      <command_interface name="position">
-        <param name="min">"${TOP_DYNAMIXEL_UPPER}"</param>
-        <param name="max">"${TOP_DYNAMIXEL_LOWER}"</param>
-      </command_interface>
-      <state_interface name="position"/>
-      <state_interface name="velocity"/>
-    </joint> -->
+    <xacro:if value="$(arg use_gazebo)">
+      <joint name="${RIGHTDYNAMIXELTOP_TO_RIGHTDRIVING_JOINT_NAME}">
+        <param name="id">5</param>
+        <command_interface name="position">
+          <param name="min">"${TOP_DYNAMIXEL_UPPER}"</param>
+          <param name="max">"${TOP_DYNAMIXEL_LOWER}"</param>
+        </command_interface>
+        <command_interface name="velocity">
+          <param name="min">"-${TOP_DYNAMIXEL_VELOCITY}"</param>
+          <param name="max">" ${TOP_DYNAMIXEL_VELOCITY}"</param>
+        </command_interface>
+        <command_interface name="effort">
+          <param name="min">"-${TOP_DYNAMIXEL_EFFORT}"</param>
+          <param name="max">" ${TOP_DYNAMIXEL_EFFORT}"</param>
+        </command_interface>
+        <state_interface name="position" />
+        <state_interface name="velocity" />
+        <state_interface name="effort" />
+      </joint>
+    </xacro:if>
     <!-- BOTTOM DYNAMIXEL TO MISUMI LN -->
-    <joint name="leftdynamixelbottom_to_leftmisumiln_joint">
+    <joint name="${LEFT_DYNAMIXELBOT_TO_LEFTMISUMILN_JOINT_NAME}">
       <param name="id">3</param>
       <command_interface name="position">
@@ -80,25 +107,40 @@
         <param name="max">${BOT_DYNAMIXEL_UPPER}</param>
       </command_interface>
-      <!-- <command_interface name="velocity">
-        <param name="min">"-${BOT_DYNAMIXEL_VELOCITY}"</param>
-        <param name="max">" ${BOT_DYNAMIXEL_VELOCITY}"</param>
-      </command_interface>
-      <command_interface name="effort">
-        <param name="min">"-${BOT_DYNAMIXEL_EFFORT}"</param>
-        <param name="max">" ${BOT_DYNAMIXEL_EFFORT}"</param>
-      </command_interface> -->
-      <state_interface name="position"/>
-      <state_interface name="velocity"/>
-      <!-- <state_interface name="effort"/> -->
+      <xacro:if value="$(arg use_gazebo)">
+        <command_interface name="velocity">
+          <param name="min">"-${BOT_DYNAMIXEL_VELOCITY}"</param>
+          <param name="max">" ${BOT_DYNAMIXEL_VELOCITY}"</param>
+        </command_interface>
+        <command_interface name="effort">
+          <param name="min">"-${BOT_DYNAMIXEL_EFFORT}"</param>
+          <param name="max">" ${BOT_DYNAMIXEL_EFFORT}"</param>
+        </command_interface>
+      </xacro:if>
+      <state_interface name="position" />
+      <state_interface name="velocity" />
+      <xacro:if value="$(arg use_gazebo)">
+        <state_interface name="effort" />
+      </xacro:if>
     </joint>
-    <!-- <joint name="rightdynamixelbottom_to_rightmisumiln_joint">
-      <param name="id">6</param>
-      <command_interface name="position">
-        <param name="min">"${BOT_DYNAMIXEL_UPPER}"</param>
-        <param name="max">"${BOT_DYNAMIXEL_LOWER}"</param>
-      </command_interface>
-      <state_interface name="position"/>
-      <state_interface name="velocity"/>
-    </joint> -->
+    <xacro:if value="$(arg use_gazebo)">
+      <joint name="${RIGHT_DYNAMIXELBOT_TO_RIGHTMISUMILN_JOINT_NAME}">
+        <param name="id">6</param>
+        <command_interface name="position">
+          <param name="min">"${BOT_DYNAMIXEL_UPPER}"</param>
+          <param name="max">"${BOT_DYNAMIXEL_LOWER}"</param>
+        </command_interface>
+        <command_interface name="velocity">
+          <param name="min">"-${BOT_DYNAMIXEL_VELOCITY}"</param>
+          <param name="max">" ${BOT_DYNAMIXEL_VELOCITY}"</param>
+        </command_interface>
+        <command_interface name="effort">
+          <param name="min">"-${BOT_DYNAMIXEL_EFFORT}"</param>
+          <param name="max">" ${BOT_DYNAMIXEL_EFFORT}"</param>
+        </command_interface>
+        <state_interface name="position" />
+        <state_interface name="velocity" />
+        <state_interface name="effort" />
+      </joint>
+    </xacro:if>
   </ros2_control>
 </robot>

Commit message: reorganized joints in control file

File: spacediver_ros2_control/description/ros2_control/spacediver_ros2_control.xacro (robot description, xacro)
@@ -37,27 +37,30 @@
       </xacro:if>
     </joint>
-    <xacro:unless value="$(arg single_arm)">
-      <joint name="${BASE_TO_RIGHTSHOULDER_JOINT_NAME}">
-        <param name="id">4</param>
-        <command_interface name="position">
-          <param name="min">"${BASE_DYNAMIXEL_UPPER}"</param>
-          <param name="max">"${BASE_DYNAMIXEL_LOWER}"</param>
-        </command_interface>
+    <!-- BOTTOM DYNAMIXEL TO MISUMI LN -->
+    <joint name="${LEFT_DYNAMIXELBOT_TO_LEFTMISUMILN_JOINT_NAME}">
+      <param name="id">2</param>
+      <command_interface name="position">
+        <param name="min">${BOT_DYNAMIXEL_LOWER}</param>
+        <param name="max">${BOT_DYNAMIXEL_UPPER}</param>
+      </command_interface>
+      <xacro:if value="$(arg use_gazebo)">
         <command_interface name="velocity">
-          <param name="min">"-${BASE_DYNAMIXEL_VELOCITY}"</param>
-          <param name="max">" ${BASE_DYNAMIXEL_VELOCITY}"</param>
+          <param name="min">"-${BOT_DYNAMIXEL_VELOCITY}"</param>
+          <param name="max">" ${BOT_DYNAMIXEL_VELOCITY}"</param>
         </command_interface>
         <command_interface name="effort">
-          <param name="min">"-${BASE_DYNAMIXEL_EFFORT}"</param>
-          <param name="max">" ${BASE_DYNAMIXEL_EFFORT}"</param>
+          <param name="min">"-${BOT_DYNAMIXEL_EFFORT}"</param>
+          <param name="max">" ${BOT_DYNAMIXEL_EFFORT}"</param>
         </command_interface>
-        <state_interface name="position" />
-        <state_interface name="velocity" />
+      </xacro:if>
+      <state_interface name="position" />
+      <state_interface name="velocity" />
+      <xacro:if value="$(arg use_gazebo)">
         <state_interface name="effort" />
-      </joint>
-    </xacro:unless>
+      </xacro:if>
+    </joint>
     <!-- TOP DYNAMIXEL TO DRIVING LINK -->
     <joint name="${LEFTDYNAMIXELTOP_TO_LEFTDRIVING_JOINT_NAME}">
-      <param name="id">2</param>
+      <param name="id">3</param>
       <command_interface name="position">
         <param name="min">${TOP_DYNAMIXEL_LOWER}</param>
@@ -81,6 +84,42 @@
     </joint>
     <xacro:unless value="$(arg single_arm)">
+      <joint name="${BASE_TO_RIGHTSHOULDER_JOINT_NAME}">
+        <param name="id">4</param>
+        <command_interface name="position">
+          <param name="min">"${BASE_DYNAMIXEL_UPPER}"</param>
+          <param name="max">"${BASE_DYNAMIXEL_LOWER}"</param>
+        </command_interface>
+        <command_interface name="velocity">
+          <param name="min">"-${BASE_DYNAMIXEL_VELOCITY}"</param>
+          <param name="max">" ${BASE_DYNAMIXEL_VELOCITY}"</param>
+        </command_interface>
+        <command_interface name="effort">
+          <param name="min">"-${BASE_DYNAMIXEL_EFFORT}"</param>
+          <param name="max">" ${BASE_DYNAMIXEL_EFFORT}"</param>
+        </command_interface>
+        <state_interface name="position" />
+        <state_interface name="velocity" />
+        <state_interface name="effort" />
+      </joint>
+      <joint name="${RIGHT_DYNAMIXELBOT_TO_RIGHTMISUMILN_JOINT_NAME}">
+        <param name="id">5</param>
+        <command_interface name="position">
+          <param name="min">"${BOT_DYNAMIXEL_UPPER}"</param>
+          <param name="max">"${BOT_DYNAMIXEL_LOWER}"</param>
+        </command_interface>
+        <command_interface name="velocity">
+          <param name="min">"-${BOT_DYNAMIXEL_VELOCITY}"</param>
+          <param name="max">" ${BOT_DYNAMIXEL_VELOCITY}"</param>
+        </command_interface>
+        <command_interface name="effort">
+          <param name="min">"-${BOT_DYNAMIXEL_EFFORT}"</param>
+          <param name="max">" ${BOT_DYNAMIXEL_EFFORT}"</param>
+        </command_interface>
+        <state_interface name="position" />
+        <state_interface name="velocity" />
+        <state_interface name="effort" />
+      </joint>
       <joint name="${RIGHTDYNAMIXELTOP_TO_RIGHTDRIVING_JOINT_NAME}">
-        <param name="id">5</param>
+        <param name="id">6</param>
         <command_interface name="position">
           <param name="min">"${TOP_DYNAMIXEL_UPPER}"</param>
@@ -100,47 +139,4 @@
       </joint>
     </xacro:unless>
-    <!-- BOTTOM DYNAMIXEL TO MISUMI LN -->
-    <joint name="${LEFT_DYNAMIXELBOT_TO_LEFTMISUMILN_JOINT_NAME}">
-      <param name="id">3</param>
-      <command_interface name="position">
-        <param name="min">${BOT_DYNAMIXEL_LOWER}</param>
-        <param name="max">${BOT_DYNAMIXEL_UPPER}</param>
-      </command_interface>
-      <xacro:if value="$(arg use_gazebo)">
-        <command_interface name="velocity">
-          <param name="min">"-${BOT_DYNAMIXEL_VELOCITY}"</param>
-          <param name="max">" ${BOT_DYNAMIXEL_VELOCITY}"</param>
-        </command_interface>
-        <command_interface name="effort">
-          <param name="min">"-${BOT_DYNAMIXEL_EFFORT}"</param>
-          <param name="max">" ${BOT_DYNAMIXEL_EFFORT}"</param>
-        </command_interface>
-      </xacro:if>
-      <state_interface name="position" />
-      <state_interface name="velocity" />
-      <xacro:if value="$(arg use_gazebo)">
-        <state_interface name="effort" />
-      </xacro:if>
-    </joint>
-    <xacro:unless value="$(arg single_arm)">
-      <joint name="${RIGHT_DYNAMIXELBOT_TO_RIGHTMISUMILN_JOINT_NAME}">
-        <param name="id">6</param>
-        <command_interface name="position">
-          <param name="min">"${BOT_DYNAMIXEL_UPPER}"</param>
-          <param name="max">"${BOT_DYNAMIXEL_LOWER}"</param>
-        </command_interface>
-        <command_interface name="velocity">
-          <param name="min">"-${BOT_DYNAMIXEL_VELOCITY}"</param>
-          <param name="max">" ${BOT_DYNAMIXEL_VELOCITY}"</param>
-        </command_interface>
-        <command_interface name="effort">
-          <param name="min">"-${BOT_DYNAMIXEL_EFFORT}"</param>
-          <param name="max">" ${BOT_DYNAMIXEL_EFFORT}"</param>
-        </command_interface>
-        <state_interface name="position" />
-        <state_interface name="velocity" />
-        <state_interface name="effort" />
-      </joint>
-    </xacro:unless>
   </ros2_control>
 </robot>
