Commit message: Update launch file and model paths for gazebo simulation

File: spacediver_ros2_control/description/gazebo/models/spacediver.sdf.xacro (robot description, xacro)
@@ -1,4 +1,4 @@
 <?xml version="1.0" ?>
-<sdf version="1.5">
+<sdf version="1.5" xmlns:xacro="http://ros.org/wiki/xacro">
   <model name="my1stmodel">
     <static>false</static>
@@ -8,5 +8,5 @@
           <box>
             <size>3 2 5</size>
-          </gox>
+          </box>
         </geometry>
         <surface>
@@ -23,5 +23,5 @@
           <box>
             <size>3 2 5</size>
-          </gox>
+          </box>
         </geometry>
         <material>
@@ -33,4 +33,19 @@
       </visual>
     </link>
+    <!-- ros_control plugin -->
+    <!-- <plugin filename="libgazebo_ros2_control.so" name="gazebo_ros2_control">
+      <parameters>$(find spacediver_ros2_control)/bringup/config/spacediver_controllers.yaml</parameters>
+    </plugin> -->
+    <!-- get true robot position plugin -->
+    <!-- <plugin filename="libgazebo_ros_p3d.so" name="base_truth" >
+      <ros>
+        <namespace>odm</namespace>
+        <remapping>odom:=base</remapping>
+      </ros>
+      <frame_name>world</frame_name>
+      <body_name>base_link</body_name>
+      <update_rate>50.0</update_rate>
+      <always_on>true</always_on>
+    </plugin> -->
   </model>
 </sdf>

File: spacediver_ros2_control/description/urdf/spacediver.urdf.xacro (robot description, xacro)
@@ -17,7 +17,3 @@
   <!-- ros2 control plugin -->
   <xacro:include filename="$(find spacediver_ros2_control)/description/ros2_control/spacediver_ros2_control.xacro" />
-  <!-- pluging for ros2 control -->
-  <xacro:if value="$(arg use_gazebo)">
-    <xacro:include filename="$(find spacediver_ros2_control)/description/gazebo/spacediver_gazebo_ros2.xacro" />
-  </xacro:if>
 </robot>

Commit message: Update .gitignore to ignore *.sdf files ``

File: spacediver_ros2_control/description/gazebo/models/spacediver.sdf.xacro (robot description, xacro)
@@ -1,11 +1,13 @@
 <?xml version="1.0" ?>
 <sdf version="1.5" xmlns:xacro="http://ros.org/wiki/xacro">
+  <xacro:include filename="$(find spacediver_ros2_control)/description/urdf/macros/properties.xacro"/>
   <model name="my1stmodel">
     <static>false</static>
-    <link name="link">
+    <link name="base_link">
+      <!-- <pose>0 0 0 0 0 0</pose> -->
       <collision name="collision">
         <geometry>
           <box>
-            <size>3 2 5</size>
+            <size>${BASE_X} ${BASE_Y} ${BASE_Z}</size>
           </box>
         </geometry>
@@ -22,5 +24,5 @@
         <geometry>
           <box>
-            <size>3 2 5</size>
+            <size>${BASE_X} ${BASE_Y} ${BASE_Z}</size>
           </box>
         </geometry>
@@ -33,8 +35,55 @@
       </visual>
     </link>
+    <!-- <link name=link1>
+      <pose>0 0 3 0 0 0</pose>
+      <collision name="collision">
+        <geometry>
+          <box>
+            <size>${LINK_1_X} ${LINK_1_Y} ${LINK_1_Z}</size>
+          </box>
+        </geometry>
+        <surface>
+          <friction>
+            <ode>
+              <mu>100</mu>
+              <mu2>50</mu2>
+            </ode>
+          </friction>
+        </surface>
+      </collision>
+      <visual name="visual">
+        <geometry>
+          <box>
+            <size>${LINK_1_X} ${LINK_1_Y} ${LINK_1_Z}</size>
+          </box>
+        </geometry>
+        <material>
+          <script>
+            <uri>file://media/materials/scripts/gazebo.material</uri>
+            <name>Gazebo/Red</name>
+          </script>
+        </material>
+      </visual>
+    </link> -->
+    <!-- <joint name="active_joint_la" type="revolute">
+      <parent>base_link</parent>
+      <child>link1</child>
+      <axis>
+        <xyz>0 0 1</xyz>
+        <limit>
+          <lower>${ACTIVE_JOINT_LA_LOWER}</lower>
+          <upper>${ACTIVE_JOINT_LA_UPPER}</upper>
+          <effort>${ACTIVE_JOINT_LA_EFFORT}</effort>
+          <velocity>${ACTIVE_JOINT_LA_VELOCITY}</velocity>
+        </limit>
+      </axis>
+      <dynamics>
+        <damping>0.7</damping>
+      </dynamics>
+    </joint> -->
     <!-- ros_control plugin -->
-    <!-- <plugin filename="libgazebo_ros2_control.so" name="gazebo_ros2_control">
+    <plugin filename="libgazebo_ros2_control.so" name="gazebo_ros2_control">
       <parameters>$(find spacediver_ros2_control)/bringup/config/spacediver_controllers.yaml</parameters>
-    </plugin> -->
+    </plugin>
     <!-- get true robot position plugin -->
     <!-- <plugin filename="libgazebo_ros_p3d.so" name="base_truth" >

File: spacediver_ros2_control/description/urdf/parts/spacediver_base.xacro (robot description, xacro)
@@ -2,6 +2,5 @@
 <!-- import xacro reffering here https://gbiggs.github.io/rosjp_urdf_tutorial_text/manipulator_urdf.html -->
 <robot xmlns:xacro="http://ros.org/wiki/xacro">
-  <xacro:property name="BASE_LINK_NAME" value="base_link" />
-  <link name="${BASE_LINK_NAME}">
+  <link name="base_link">
     <visual>
       <origin xyz="0 0 0" rpy="0 0 0"/>

File: spacediver_ros2_control/description/urdf/spacediver.urdf.xacro (robot description, xacro)
@@ -12,5 +12,5 @@
   <!-- Left Arm -->
   <xacro:include filename="$(find spacediver_ros2_control)/description/urdf/parts/spacediver_left_arm.xacro" />
-  <xacro:left_arm base_name="${BASE_LINK_NAME}">
+  <xacro:left_arm base_name="base_link">
     <origin xyz="0 0 ${BASE_Z/2}" rpy="0 0 0"/>
   </xacro:left_arm>

Commit message: add joint to sdf

File: spacediver_ros2_control/description/gazebo/models/spacediver.sdf.xacro (robot description, xacro)
@@ -35,6 +35,6 @@
       </visual>
     </link>
-    <!-- <link name=link1>
-      <pose>0 0 3 0 0 0</pose>
+    <link name="link_1">
+      <pose>0 0 ${BASE_Z}</pose>
       <collision name="collision">
         <geometry>
@@ -61,25 +61,22 @@
           <script>
             <uri>file://media/materials/scripts/gazebo.material</uri>
-            <name>Gazebo/Red</name>
+            <name>Gazebo/Grey</name>
           </script>
         </material>
       </visual>
-    </link> -->
-    <!-- <joint name="active_joint_la" type="revolute">
+    </link>
+    <joint name="active_joint_la" type="revolute">
       <parent>base_link</parent>
-      <child>link1</child>
+      <child>link_1</child>
       <axis>
         <xyz>0 0 1</xyz>
-        <limit>
-          <lower>${ACTIVE_JOINT_LA_LOWER}</lower>
-          <upper>${ACTIVE_JOINT_LA_UPPER}</upper>
-          <effort>${ACTIVE_JOINT_LA_EFFORT}</effort>
-          <velocity>${ACTIVE_JOINT_LA_VELOCITY}</velocity>
-        </limit>
       </axis>
-      <dynamics>
-        <damping>0.7</damping>
-      </dynamics>
-    </joint> -->
+      <limit>
+        <lower>${ACTIVE_JOINT_LA_LOWER}</lower>
+        <upper>${ACTIVE_JOINT_LA_UPPER}</upper>
+        <effort>${ACTIVE_JOINT_LA_EFFORT}</effort>
+        <velocity>${ACTIVE_JOINT_LA_VELOCITY}</velocity>
+      </limit>
+    </joint>
     <!-- ros_control plugin -->
     <plugin filename="libgazebo_ros2_control.so" name="gazebo_ros2_control">

Commit message: Refactor include paths in c_cpp_properties.json

File: spacediver_ros2_control/description/gazebo/models/spacediver.sdf.xacro (robot description, xacro)
@@ -73,4 +73,66 @@
       </visual>
     </link>
+    <link name="link_2">
+      <pose>0 0 ${BASE_Z/2}</pose>
+      <collision name="collision">
+        <geometry>
+          <box>
+            <size>${LINK_1_X} ${LINK_1_Y} ${LINK_1_Z}</size>
+          </box>
+        </geometry>
+        <surface>
+          <friction>
+            <ode>
+              <mu>100</mu>
+              <mu2>50</mu2>
+            </ode>
+          </friction>
+        </surface>
+      </collision>
+      <visual name="visual">
+        <geometry>
+          <box>
+            <size>${LINK_1_X} ${LINK_1_Y} ${LINK_1_Z}</size>
+          </box>
+        </geometry>
+        <material>
+          <script>
+            <uri>file://media/materials/scripts/gazebo.material</uri>
+            <name>Gazebo/Red</name>
+          </script>
+        </material>
+      </visual>
+    </link>
+    <link name="link_3">
+      <pose>0 0 ${BASE_Z/2}</pose>
+      <collision name="collision">
+        <geometry>
+          <box>
+            <size>${LINK_1_X} ${LINK_1_Y} ${LINK_1_Z}</size>
+          </box>
+        </geometry>
+        <surface>
+          <friction>
+            <ode>
+              <mu>100</mu>
+              <mu2>50</mu2>
+            </ode>
+          </friction>
+        </surface>
+      </collision>
+      <visual name="visual">
+        <geometry>
+          <box>
+            <size>${LINK_1_X} ${LINK_1_Y} ${LINK_1_Z}</size>
+          </box>
+        </geometry>
+        <material>
+          <script>
+            <uri>file://media/materials/scripts/gazebo.material</uri>
+            <name>Gazebo/Red</name>
+          </script>
+        </material>
+      </visual>
+    </link>
     <joint name="active_joint_la" type="revolute">
       <parent>base_link</parent>
@@ -86,4 +148,30 @@
       </limit>
     </joint>
+    <joint name="active_joint_lb" type="revolute">
+      <parent>link_1</parent>
+      <child>link_2</child>
+      <axis>
+        <xyz>0 1 0</xyz>
+      </axis>
+      <limit>
+        <lower>${ACTIVE_JOINT_LB_LOWER}</lower>
+        <upper>${ACTIVE_JOINT_LB_UPPER}</upper>
+        <effort>${ACTIVE_JOINT_LB_EFFORT}</effort>
+        <velocity>${ACTIVE_JOINT_LB_VELOCITY}</velocity>
+      </limit>
+    </joint>
+    <joint name="active_joint_lc" type="revolute">
+      <parent>link_2</parent>
+      <child>link_3</child>
+      <axis>
+        <xyz>0 1 0</xyz>
+      </axis>
+      <limit>
+        <lower>${ACTIVE_JOINT_LC_LOWER}</lower>
+        <upper>${ACTIVE_JOINT_LC_UPPER}</upper>
+        <effort>${ACTIVE_JOINT_LC_EFFORT}</effort>
+        <velocity>${ACTIVE_JOINT_LC_VELOCITY}</velocity>
+      </limit>
+    </joint>
   </model>
 </sdf>
