Commit message: updated links of sdf file and corresponding properties to render one arm

File: spacediver_ros2_control/description/gazebo/models/spacediver.sdf.xacro (robot description, xacro)
@@ -42,10 +42,38 @@
       </visual>
     </link>
-    <link name="link_1">
-      <pose>0 0 ${BASE_Z/2}</pose>
-      <collision name="collision">
-        <geometry>
-          <box>
-            <size>${LINK_1_X} ${LINK_1_Y} ${LINK_1_Z}</size>
+    <link name="left_shoulder_plate">
+      <pose>
+        ${SHOULDER_PLATE_POS_X} ${SHOULDER_PLATE_POS_Y} ${SHOULDER_PLATE_POS_Z}
+        ${SHOULDER_PLATE_ROT_X} ${SHOULDER_PLATE_ROT_Y} ${SHOULDER_PLATE_ROT_Z}
+      </pose>
+      <collision name="collision">
+        <geometry>
+          <mesh>
+            <uri>model://spacediver/meshes/shoulder_plate.STL</uri>
+          </mesh>
+        </geometry>
+      </collision>
+      <visual name="visual">
+        <geometry>
+          <mesh>
+            <uri>model://spacediver/meshes/shoulder_plate.STL</uri>
+          </mesh>
+        </geometry>
+        <!-- <material>
+          <script>
+            <uri>file://media/materials/scripts/gazebo.material</uri>
+            <name>Gazebo/Grey</name>
+          </script>
+        </material> -->
+      </visual>
+    </link>
+    <link name="left_dynamixel_top">
+      <pose>
+        ${DYNAMIXEL_LEFT_TOP_POS_X} ${DYNAMIXEL_LEFT_TOP_POS_Y} ${DYNAMIXEL_LEFT_TOP_POS_Z}
+      </pose>
+      <collision name="collision">
+        <geometry>
+          <box>
+            <size>${DYNAMIXEL_X} ${DYNAMIXEL_Y} ${DYNAMIXEL_Z}</size>
           </box>
         </geometry>
@@ -62,21 +90,23 @@
         <geometry>
           <box>
-            <size>${LINK_1_X} ${LINK_1_Y} ${LINK_1_Z}</size>
-          </box>
-        </geometry>
-        <material>
-          <script>
-            <uri>file://media/materials/scripts/gazebo.material</uri>
-            <name>Gazebo/Red</name>
-          </script>
-        </material>
-      </visual>
-    </link>
-    <link name="link_2">
-      <pose>0 0 ${BASE_Z/2+LINK_1_X}</pose>
-      <collision name="collision">
-        <geometry>
-          <box>
-            <size>${LINK_2_X} ${LINK_2_Y} ${LINK_2_Z}</size>
+            <size>${DYNAMIXEL_X} ${DYNAMIXEL_Y} ${DYNAMIXEL_Z}</size>
+          </box>
+        </geometry>
+        <material>
+          <script>
+            <uri>file://media/materials/scripts/gazebo.material</uri>
+            <name>Gazebo/Blue</name>
+          </script>
+        </material>
+      </visual>
+    </link>
+    <link name="left_dynamixel_bottom">
+      <pose>
+        ${DYNAMIXEL_LEFT_BOT_POS_X} ${DYNAMIXEL_LEFT_BOT_POS_Y} ${DYNAMIXEL_LEFT_BOT_POS_Z}
+      </pose>
+      <collision name="collision">
+        <geometry>
+          <box>
+            <size>${DYNAMIXEL_X} ${DYNAMIXEL_Y} ${DYNAMIXEL_Z}</size>
           </box>
         </geometry>
@@ -93,6 +123,32 @@
         <geometry>
           <box>
-            <size>${LINK_2_X} ${LINK_2_Y} ${LINK_2_Z}</size>
-          </box>
+            <size>${DYNAMIXEL_X} ${DYNAMIXEL_Y} ${DYNAMIXEL_Z}</size>
+          </box>
+        </geometry>
+        <material>
+          <script>
+            <uri>file://media/materials/scripts/gazebo.material</uri>
+            <name>Gazebo/Blue</name>
+          </script>
+        </material>
+      </visual>
+    </link>
+    <link name="misumi_ln">
+      <pose>
+        ${MISUMILN_POS_X} ${MISUMILN_POS_Y} ${MISUMILN_POS_Z}
+        0 0 ${MISUMILN_ROT_Z}
+      </pose>
+      <collision name="collision">
+        <geometry>
+          <mesh>
+            <uri>model://spacediver/meshes/Link_MISUMI_LNMS16-10-200.STL</uri>
+          </mesh>
+        </geometry>
+      </collision>
+      <visual name="visual">
+        <geometry>
+          <mesh>
+            <uri>model://spacediver/meshes/Link_MISUMI_LNMS16-10-200.STL</uri>
+          </mesh>
         </geometry>
         <material>
@@ -104,26 +160,46 @@
       </visual>
     </link>
-    <link name="link_3">
-      <pose>0 0 ${BASE_Z/2+LINK_1_X+LINK_2_X}</pose>
-      <collision name="collision">
-        <geometry>
-          <box>
-            <size>${LINK_3_X} ${LINK_3_Y} ${LINK_3_Z}</size>
-          </box>
-        </geometry>
-        <surface>
-          <friction>
-            <ode>
-              <mu>100</mu>
-              <mu2>50</mu2>
-            </ode>
-          </friction>
-        </surface>
-      </collision>
-      <visual name="visual">
-        <geometry>
-          <box>
-            <size>${LINK_3_X} ${LINK_3_Y} ${LINK_3_Z}</size>
-          </box>
+    <link name="driving_link">
+      <pose>
+        ${DRIVING_POS_X} ${DRIVING_POS_Y} ${DRIVING_POS_Z}
+      </pose>
+      <collision name="collision">
+        <geometry>
+          <mesh>
+            <uri>model://spacediver/meshes/upper_arm_driving_link.STL</uri>
+          </mesh>
+        </geometry>
+      </collision>
+      <visual name="visual">
+        <geometry>
+          <mesh>
+            <uri>model://spacediver/meshes/upper_arm_driving_link.STL</uri>
+          </mesh>
+        </geometry>
+        <material>
+          <script>
+            <uri>file://media/materials/scripts/gazebo.material</uri>
+            <name>Gazebo/Green</name>
+          </script>
+        </material>
+      </visual>
+    </link>
+    <link name="driven_link">
+      <pose>
+        ${DRIVEN_POS_X} ${DRIVEN_POS_Y} ${DRIVEN_POS_Z}
+        0 0 ${DRIVEN_ROT_Z}
+      </pose>
+      <collision name="collision">
+        <geometry>
+          <mesh>
+            <uri>model://spacediver/meshes/upper_arm_driven_link.STL</uri>
+          </mesh>
+        </geometry>
+      </collision>
+      <visual name="visual">
+        <geometry>
+          <mesh>
+            <uri>model://spacediver/meshes/upper_arm_driven_link.STL</uri>
+          </mesh>
         </geometry>
         <material>
@@ -135,42 +211,43 @@
       </visual>
     </link>
-    <joint name="active_joint_la" type="revolute">
-      <parent>base_link</parent>
-      <child>link_1</child>
+    <link name="misumi_ft">
+      <pose>
+        ${MISUMIFT_POS_X} ${MISUMIFT_POS_Y} ${MISUMIFT_POS_Z}
+        0 0 ${MISUMIFT_ROT_Z}
+      </pose>
+      <collision name="collision">
+        <geometry>
+          <mesh>
+            <uri>model://spacediver/meshes/Misumi_LNFTS10-P10-V10-L200-S50-W18-T9.STL</uri>
+          </mesh>
+        </geometry>
+      </collision>
+      <visual name="visual">
+        <geometry>
+          <mesh>
+            <uri>model://spacediver/meshes/Misumi_LNFTS10-P10-V10-L200-S50-W18-T9.STL</uri>
+          </mesh>
+        </geometry>
+        <material>
+          <script>
+            <uri>file://media/materials/scripts/gazebo.material</uri>
+            <name>Gazebo/Green</name>
+          </script>
+        </material>
+      </visual>
+    </link>
+    <joint name="dynamixel_to_driving_joint" type="revolute">
+      <parent>left_dynamixel_top</parent>
+      <child>driving_link</child>
       <axis>
-        <xyz>0 1 0</xyz>
+        <xyz>0 0 1</xyz>
       </axis>
-      <limit>
-        <lower>${ACTIVE_JOINT_LA_LOWER}</lower>
-        <upper>${ACTIVE_JOINT_LA_UPPER}</upper>
-        <effort>${ACTIVE_JOINT_LA_EFFORT}</effort>
-        <velocity>${ACTIVE_JOINT_LA_VELOCITY}</velocity>
-      </limit>
     </joint>
-    <joint name="active_joint_lb" type="revolute">
-      <parent>link_1</parent>
-      <child>link_2</child>
+    <joint name="driving_to_driven_joint" type="revolute">
+      <parent>driving_link</parent>
+      <child>driven_link</child>
       <axis>
-        <xyz>0 1 1</xyz>
+        <xyz>0 0 1</xyz>
       </axis>
-      <limit>
-        <lower>${ACTIVE_JOINT_LB_LOWER}</lower>
-        <upper>${ACTIVE_JOINT_LB_UPPER}</upper>
-        <effort>${ACTIVE_JOINT_LB_EFFORT}</effort>
-        <velocity>${ACTIVE_JOINT_LB_VELOCITY}</velocity>
-      </limit>
-    </joint>
-    <joint name="active_joint_lc" type="revolute">
-      <parent>link_2</parent>
-      <child>link_3</child>
-      <axis>
-        <xyz>1 1 0</xyz>
-      </axis>
-      <limit>
-        <lower>${ACTIVE_JOINT_LC_LOWER}</lower>
-        <upper>${ACTIVE_JOINT_LC_UPPER}</upper>
-        <effort>${ACTIVE_JOINT_LC_EFFORT}</effort>
-        <velocity>${ACTIVE_JOINT_LC_VELOCITY}</velocity>
-      </limit>
     </joint>
   </model>

File: spacediver_ros2_control/description/urdf/macros/properties.xacro (robot description, xacro)
@@ -2,9 +2,71 @@
 <robot xmlns:xacro="http://ros.org/wiki/xacro">
   <xacro:property name="PI" value="3.1415926535"/>
-  <xacro:property name="BASE_X" value="0.5"/>
-  <xacro:property name="BASE_Y" value="0.5"/>
-  <xacro:property name="BASE_Z" value="0.5"/>
+  <xacro:property name="BASE_X" value="0.18"/>
+  <xacro:property name="BASE_Y" value="0.0585"/>
+  <xacro:property name="BASE_Z" value="0.0415"/>
   <xacro:property name="BASE_MASS" value="50"/>
   <xacro:property name="BASE_INERTIA_Z" value="0.13526810"/>
+  <xacro:property name="BASE_TO_SHOULDER_PLATE_X" value="0.0045"/>
+  <xacro:property name="SHOULDER_PLATE_X" value="0.03"/>
+  <xacro:property name="SHOULDER_PLATE_Y" value="0.0585"/>
+  <xacro:property name="SHOULDER_PLATE_Z" value="0.148"/>
+  <xacro:property name="SHOULDER_PLATE_ROT_X" value="${-PI/2}"/>
+  <xacro:property name="SHOULDER_PLATE_ROT_Y" value="0"/>
+  <xacro:property name="SHOULDER_PLATE_ROT_Z" value="${-PI/2}"/>
+  <xacro:property name="SHOULDER_PLATE_POS_X" value="${BASE_X/2 + 0.0045}"/>
+  <xacro:property name="SHOULDER_PLATE_POS_Y" value="${SHOULDER_PLATE_Y/2}"/>
+  <xacro:property name="SHOULDER_PLATE_POS_Z" value="${SHOULDER_PLATE_Z/2}"/>
+  <xacro:property name="DYNAMIXEL_X" value="0.0335"/>
+  <xacro:property name="DYNAMIXEL_Y" value="0.0585"/>
+  <xacro:property name="DYNAMIXEL_Z" value="0.044"/>
+  <xacro:property name="DYNAMIXEL_JOINTB_X" value="0"/>
+  <xacro:property name="DYNAMIXEL_JOINTB_Y" value="${DYNAMIXEL_Y - 0.04475}"/>
+  <xacro:property name="DYNAMIXEL_LEFT_TOP_POS_X" value="${SHOULDER_PLATE_POS_X + SHOULDER_PLATE_X + DYNAMIXEL_X/2}"/>
+  <xacro:property name="DYNAMIXEL_LEFT_TOP_POS_Y" value="${SHOULDER_PLATE_POS_Y - SHOULDER_PLATE_Y/2}"/>
+  <xacro:property name="DYNAMIXEL_LEFT_TOP_POS_Z" value="${SHOULDER_PLATE_POS_Z - DYNAMIXEL_Z/2}"/>
+  <xacro:property name="DYNAMIXEL_LEFT_BOT_POS_X" value="${SHOULDER_PLATE_POS_X + SHOULDER_PLATE_X + DYNAMIXEL_X/2}"/>
+  <xacro:property name="DYNAMIXEL_LEFT_BOT_POS_Y" value="${SHOULDER_PLATE_POS_Y - SHOULDER_PLATE_Y/2}"/>
+  <xacro:property name="DYNAMIXEL_LEFT_BOT_POS_Z" value="${SHOULDER_PLATE_POS_Z - SHOULDER_PLATE_Z + DYNAMIXEL_Z/2}"/>
+  <xacro:property name="MISUMILN_X" value="0.032"/>
+  <xacro:property name="MISUMILN_Y" value="0.225"/>
+  <xacro:property name="MISUMILN_Z" value="0.009"/>
+  <xacro:property name="MISUMILN_ROT_Z" value="${-PI/2}"/>
+  <xacro:property name="MISUMILN_JOINTA_X" value="0.016"/>
+  <xacro:property name="MISUMILN_JOINTA_Y" value="0.012"/>
+  <xacro:property name="MISUMILN_POS_X" value="${DYNAMIXEL_LEFT_BOT_POS_X - MISUMILN_JOINTA_X}"/>
+  <xacro:property name="MISUMILN_POS_Y" value="${DYNAMIXEL_LEFT_BOT_POS_Y - DYNAMIXEL_JOINTB_Y + MISUMILN_JOINTA_Y}"/>
+  <xacro:property name="MISUMILN_POS_Z" value="${DYNAMIXEL_LEFT_BOT_POS_Z + DYNAMIXEL_Z/2 + 0.0045}"/>
+  <xacro:property name="DRIVING_X" value="0.076"/>
+  <xacro:property name="DRIVING_Y" value="0.026"/>
+  <xacro:property name="DRIVING_Z" value="0.004"/>
+  <xacro:property name="DRIVING_JOINTA_X" value="0.013"/>
+  <xacro:property name="DRIVING_JOINTA_Y" value="0.013"/>
+  <xacro:property name="DRIVING_POS_X" value="${DYNAMIXEL_LEFT_TOP_POS_X - DRIVING_JOINTA_X}"/>
+  <xacro:property name="DRIVING_POS_Y" value="${DYNAMIXEL_LEFT_TOP_POS_Y - DYNAMIXEL_JOINTB_Y - DRIVING_JOINTA_Y}"/>
+  <xacro:property name="DRIVING_POS_Z" value="${DYNAMIXEL_LEFT_TOP_POS_Z - DYNAMIXEL_Z/2 - DRIVING_Z - 0.0045}"/>
+  <xacro:property name="DRIVING_JOINTB_X" value="0.063"/>
+  <xacro:property name="DRIVING_JOINTB_Y" value="0.013"/>
+  <xacro:property name="DRIVEN_X" value="0.026"/>
+  <xacro:property name="DRIVEN_Y" value="0.226"/>
+  <xacro:property name="DRIVEN_Z" value="0.004"/>
+  <xacro:property name="DRIVEN_ROT_Z" value="${-PI/2}"/>
+  <xacro:property name="DRIVEN_JOINTA_X" value="0.013"/>
+  <xacro:property name="DRIVEN_JOINTA_Y" value="0.013"/>
+  <xacro:property name="DRIVEN_POS_X" value="${DRIVING_POS_X + DRIVING_JOINTB_X - DRIVEN_JOINTA_X}"/>
+  <xacro:property name="DRIVEN_POS_Y" value="${DRIVING_POS_Y + DRIVING_JOINTB_Y + DRIVEN_JOINTA_Y}"/>
+  <xacro:property name="DRIVEN_POS_Z" value="${DRIVING_POS_Z - DRIVING_Z - 0.01}"/>
+  <xacro:property name="DRIVEN_JOINTB_X" value="0.013"/>
+  <xacro:property name="DRIVEN_JOINTB_Y" value="0.213"/>
+  <xacro:property name="MISUMIFT_X" value="0.268"/>
+  <xacro:property name="MISUMIFT_Y" value="0.018"/>
+  <xacro:property name="MISUMIFT_Z" value="0.009"/>
+  <xacro:property name="MISUMIFT_ROT_Z" value="${-PI}"/>
+  <xacro:property name="MISUMIFT_JOINTA_X" value="0.009"/>
+  <xacro:property name="MISUMIFT_JOINTA_Y" value="0.009"/>
+  <xacro:property name="MISUMIFT_JOINTB_X" value="0.059"/>
+  <xacro:property name="MISUMIFT_JOINTB_Y" value="0.009"/>
+  <xacro:property name="MISUMIFT_POS_X" value="${DRIVEN_POS_X + DRIVEN_JOINTB_X + MISUMIFT_JOINTA_X}"/>
+  <xacro:property name="MISUMIFT_POS_Y" value="${DRIVEN_POS_Y - DRIVEN_JOINTB_Y + MISUMIFT_JOINTA_Y}"/>
+  <xacro:property name="MISUMIFT_POS_Z" value="${DRIVEN_POS_Z - MISUMIFT_Z - 0.005}"/>
   <xacro:property name="ACTIVE_JOINT_LA_LOWER" value="-${PI}"/>
   <xacro:property name="ACTIVE_JOINT_LA_UPPER" value=" ${PI}"/>

Commit message: added joints to arm links relative to child link

File: spacediver_ros2_control/description/gazebo/models/spacediver.sdf.xacro (robot description, xacro)
@@ -237,7 +237,20 @@
       </visual>
     </link>
+    <joint name="dynamixel_to_misumiln_joint" type="revolute">
+      <parent>left_dynamixel_bottom</parent>
+      <child>misumi_ln</child>
+      <pose>
+        ${MISUMILN_JOINTA_Y} ${MISUMILN_JOINTA_X} ${MISUMILN_JOINTA_Z}
+      </pose>
+      <axis>
+        <xyz>0 0 1</xyz>
+      </axis>
+    </joint>
     <joint name="dynamixel_to_driving_joint" type="revolute">
       <parent>left_dynamixel_top</parent>
       <child>driving_link</child>
+      <pose>
+        ${DRIVING_JOINTA_X} ${DRIVING_JOINTA_Y} ${DRIVING_JOINTA_Z}
+      </pose>
       <axis>
         <xyz>0 0 1</xyz>
@@ -247,4 +260,27 @@
       <parent>driving_link</parent>
       <child>driven_link</child>
+      <pose>
+        ${DRIVEN_JOINTA_X} ${DRIVEN_JOINTA_Y} ${DRIVEN_JOINTA_Z}
+      </pose>
+      <axis>
+        <xyz>0 0 1</xyz>
+      </axis>
+    </joint>
+    <joint name="driven_to_misumift_joint" type="revolute">
+      <parent>driven_link</parent>
+      <child>misumi_ft</child>
+      <pose>
+        ${MISUMIFT_JOINTA_X} ${MISUMIFT_JOINTA_Y} ${MISUMIFT_JOINTA_Z}
+      </pose>
+      <axis>
+        <xyz>0 0 1</xyz>
+      </axis>
+    </joint>
+    <joint name="misumiln_to_misumift_joint" type="revolute">
+      <parent>misumi_ln</parent>
+      <child>misumi_ft</child>
+      <pose>
+        ${MISUMIFT_JOINTB_X} ${MISUMIFT_JOINTB_Y} ${MISUMIFT_JOINTB_Z}
+      </pose>
       <axis>
         <xyz>0 0 1</xyz>

File: spacediver_ros2_control/description/urdf/macros/properties.xacro (robot description, xacro)
@@ -34,4 +34,5 @@
   <xacro:property name="MISUMILN_JOINTA_X" value="0.016"/>
   <xacro:property name="MISUMILN_JOINTA_Y" value="0.012"/>
+  <xacro:property name="MISUMILN_JOINTA_Z" value="${0.01 + MISUMILN_Z/2}"/>
   <xacro:property name="MISUMILN_POS_X" value="${DYNAMIXEL_LEFT_BOT_POS_X - MISUMILN_JOINTA_X}"/>
   <xacro:property name="MISUMILN_POS_Y" value="${DYNAMIXEL_LEFT_BOT_POS_Y - DYNAMIXEL_JOINTB_Y + MISUMILN_JOINTA_Y}"/>
@@ -42,4 +43,5 @@
   <xacro:property name="DRIVING_JOINTA_X" value="0.013"/>
   <xacro:property name="DRIVING_JOINTA_Y" value="0.013"/>
+  <xacro:property name="DRIVING_JOINTA_Z" value="${DRIVING_Z/2}"/>
   <xacro:property name="DRIVING_POS_X" value="${DYNAMIXEL_LEFT_TOP_POS_X - DRIVING_JOINTA_X}"/>
   <xacro:property name="DRIVING_POS_Y" value="${DYNAMIXEL_LEFT_TOP_POS_Y - DYNAMIXEL_JOINTB_Y - DRIVING_JOINTA_Y}"/>
@@ -53,4 +55,5 @@
   <xacro:property name="DRIVEN_JOINTA_X" value="0.013"/>
   <xacro:property name="DRIVEN_JOINTA_Y" value="0.013"/>
+  <xacro:property name="DRIVEN_JOINTA_Z" value="${DRIVEN_Z/2}"/>
   <xacro:property name="DRIVEN_POS_X" value="${DRIVING_POS_X + DRIVING_JOINTB_X - DRIVEN_JOINTA_X}"/>
   <xacro:property name="DRIVEN_POS_Y" value="${DRIVING_POS_Y + DRIVING_JOINTB_Y + DRIVEN_JOINTA_Y}"/>
@@ -64,6 +67,8 @@
   <xacro:property name="MISUMIFT_JOINTA_X" value="0.009"/>
   <xacro:property name="MISUMIFT_JOINTA_Y" value="0.009"/>
+  <xacro:property name="MISUMIFT_JOINTA_Z" value="${MISUMIFT_Z/2}"/>
   <xacro:property name="MISUMIFT_JOINTB_X" value="0.059"/>
   <xacro:property name="MISUMIFT_JOINTB_Y" value="0.009"/>
+  <xacro:property name="MISUMIFT_JOINTB_Z" value="${MISUMIFT_Z/2}"/>
   <xacro:property name="MISUMIFT_POS_X" value="${DRIVEN_POS_X + DRIVEN_JOINTB_X + MISUMIFT_JOINTA_X}"/>
   <xacro:property name="MISUMIFT_POS_Y" value="${DRIVEN_POS_Y - DRIVEN_JOINTB_Y + MISUMIFT_JOINTA_Y}"/>

Commit message: added fixed joints for base-plate and plate-dynamixels

File: spacediver_ros2_control/description/gazebo/models/spacediver.sdf.xacro (robot description, xacro)
@@ -237,4 +237,16 @@
       </visual>
     </link>
+    <joint name="base_to_leftshoulderplate_joint" type="fixed">
+      <parent>base_link</parent>
+      <child>left_shoulder_plate</child>
+    </joint>
+    <joint name="leftshoulderplate_to_leftdynamixeltop_joint" type="fixed">
+      <parent>left_shoulder_plate</parent>
+      <child>left_dynamixel_top</child>
+    </joint>
+    <joint name="leftshoulderplate_to_leftdynamixelbottom_joint" type="fixed">
+      <parent>left_shoulder_plate</parent>
+      <child>left_dynamixel_bottom</child>
+    </joint>
     <joint name="dynamixel_to_misumiln_joint" type="revolute">
       <parent>left_dynamixel_bottom</parent>

Commit message: rotated initial pose to avoid intersection of arms' misumift's

File: spacediver_ros2_control/description/gazebo/models/spacediver.sdf.xacro (robot description, xacro)
@@ -163,4 +163,5 @@
       <pose>
         ${DRIVING_POS_X} ${DRIVING_POS_Y} ${DRIVING_POS_Z}
+        0 0 ${DRIVING_ROT_Z}
       </pose>
       <collision name="collision">

File: spacediver_ros2_control/description/urdf/macros/properties.xacro (robot description, xacro)
@@ -1,5 +1,6 @@
 <?xml version="1.0"?>
 <robot xmlns:xacro="http://ros.org/wiki/xacro">
-  <xacro:property name="PI" value="3.1415926535"/>
+  <xacro:property name="PI" value="${math.pi}"/>
+  <xacro:property name="ROT" value="${PI/6}"/>
   <xacro:property name="BASE_X" value="0.18"/>
   <xacro:property name="BASE_Y" value="0.0585"/>
@@ -31,10 +32,10 @@
   <xacro:property name="MISUMILN_Y" value="0.225"/>
   <xacro:property name="MISUMILN_Z" value="0.009"/>
-  <xacro:property name="MISUMILN_ROT_Z" value="${-PI/2}"/>
+  <xacro:property name="MISUMILN_ROT_Z" value="${-PI/2+ROT}"/>
   <xacro:property name="MISUMILN_JOINTA_X" value="0.016"/>
   <xacro:property name="MISUMILN_JOINTA_Y" value="0.012"/>
   <xacro:property name="MISUMILN_JOINTA_Z" value="${0.01 + MISUMILN_Z/2}"/>
-  <xacro:property name="MISUMILN_POS_X" value="${DYNAMIXEL_LEFT_BOT_POS_X - MISUMILN_JOINTA_X}"/>
-  <xacro:property name="MISUMILN_POS_Y" value="${DYNAMIXEL_LEFT_BOT_POS_Y - DYNAMIXEL_JOINTB_Y + MISUMILN_JOINTA_Y}"/>
+  <xacro:property name="MISUMILN_POS_X" value="${DYNAMIXEL_LEFT_BOT_POS_X + math.cos(ROT)*(-MISUMILN_JOINTA_X) - math.sin(ROT)*(MISUMILN_JOINTA_Y)}"/>
+  <xacro:property name="MISUMILN_POS_Y" value="${DYNAMIXEL_LEFT_BOT_POS_Y - DYNAMIXEL_JOINTB_Y + math.sin(ROT)*(-MISUMILN_JOINTA_X) + math.cos(ROT)*(MISUMILN_JOINTA_Y)}"/>
   <xacro:property name="MISUMILN_POS_Z" value="${DYNAMIXEL_LEFT_BOT_POS_Z + DYNAMIXEL_Z/2 + 0.0045}"/>
   <xacro:property name="DRIVING_X" value="0.076"/>
@@ -44,4 +45,5 @@
   <xacro:property name="DRIVING_JOINTA_Y" value="0.013"/>
   <xacro:property name="DRIVING_JOINTA_Z" value="${DRIVING_Z/2}"/>
+  <xacro:property name="DRIVING_ROT_Z" value="${0}"/>
   <xacro:property name="DRIVING_POS_X" value="${DYNAMIXEL_LEFT_TOP_POS_X - DRIVING_JOINTA_X}"/>
   <xacro:property name="DRIVING_POS_Y" value="${DYNAMIXEL_LEFT_TOP_POS_Y - DYNAMIXEL_JOINTB_Y - DRIVING_JOINTA_Y}"/>
@@ -52,10 +54,10 @@
   <xacro:property name="DRIVEN_Y" value="0.226"/>
   <xacro:property name="DRIVEN_Z" value="0.004"/>
-  <xacro:property name="DRIVEN_ROT_Z" value="${-PI/2}"/>
+  <xacro:property name="DRIVEN_ROT_Z" value="${-PI/2+ROT}"/>
   <xacro:property name="DRIVEN_JOINTA_X" value="0.013"/>
   <xacro:property name="DRIVEN_JOINTA_Y" value="0.013"/>
   <xacro:property name="DRIVEN_JOINTA_Z" value="${DRIVEN_Z/2}"/>
-  <xacro:property name="DRIVEN_POS_X" value="${DRIVING_POS_X + DRIVING_JOINTB_X - DRIVEN_JOINTA_X}"/>
-  <xacro:property name="DRIVEN_POS_Y" value="${DRIVING_POS_Y + DRIVING_JOINTB_Y + DRIVEN_JOINTA_Y}"/>
+  <xacro:property name="DRIVEN_POS_X" value="${DRIVING_POS_X + DRIVING_JOINTB_X + math.cos(ROT)*(-DRIVEN_JOINTA_X) - math.sin(ROT)*(DRIVEN_JOINTA_Y)}"/>
+  <xacro:property name="DRIVEN_POS_Y" value="${DRIVING_POS_Y + DRIVING_JOINTB_Y + math.sin(ROT)*(-DRIVEN_JOINTA_X) + math.cos(ROT)*(DRIVEN_JOINTA_Y)}"/>
   <xacro:property name="DRIVEN_POS_Z" value="${DRIVING_POS_Z - DRIVING_Z - 0.01}"/>
   <xacro:property name="DRIVEN_JOINTB_X" value="0.013"/>
@@ -64,5 +66,5 @@
   <xacro:property name="MISUMIFT_Y" value="0.018"/>
   <xacro:property name="MISUMIFT_Z" value="0.009"/>
-  <xacro:property name="MISUMIFT_ROT_Z" value="${-PI}"/>
+  <xacro:property name="MISUMIFT_ROT_Z" value="${PI}"/>
   <xacro:property name="MISUMIFT_JOINTA_X" value="0.009"/>
   <xacro:property name="MISUMIFT_JOINTA_Y" value="0.009"/>
@@ -71,6 +73,6 @@
   <xacro:property name="MISUMIFT_JOINTB_Y" value="0.009"/>
   <xacro:property name="MISUMIFT_JOINTB_Z" value="${MISUMIFT_Z/2}"/>
-  <xacro:property name="MISUMIFT_POS_X" value="${DRIVEN_POS_X + DRIVEN_JOINTB_X + MISUMIFT_JOINTA_X}"/>
-  <xacro:property name="MISUMIFT_POS_Y" value="${DRIVEN_POS_Y - DRIVEN_JOINTB_Y + MISUMIFT_JOINTA_Y}"/>
+  <xacro:property name="MISUMIFT_POS_X" value="${DRIVEN_POS_X + math.cos(ROT)*(DRIVEN_JOINTB_X) - math.sin(ROT)*(-DRIVEN_JOINTB_Y) + MISUMIFT_JOINTA_X}"/>
+  <xacro:property name="MISUMIFT_POS_Y" value="${DRIVEN_POS_Y + math.sin(ROT)*(DRIVEN_JOINTB_X) + math.cos(ROT)*(-DRIVEN_JOINTB_Y) + MISUMIFT_JOINTA_Y}"/>
   <xacro:property name="MISUMIFT_POS_Z" value="${DRIVEN_POS_Z - MISUMIFT_Z - 0.005}"/>
   <xacro:property name="ACTIVE_JOINT_LA_LOWER" value="-${PI}"/>
