Commit message: added right arm links and joints

File: spacediver_ros2_control/description/gazebo/models/spacediver.sdf.xacro (robot description, xacro)
@@ -42,4 +42,5 @@
       </visual>
     </link>
+    <!-- SHOULDER PLATES -->
     <link name="left_shoulder_plate">
       <pose>
@@ -68,7 +69,34 @@
       </visual>
     </link>
+    <link name="right_shoulder_plate">
+      <pose>
+        ${-SHOULDER_PLATE_POS_X} ${SHOULDER_PLATE_POS_Y} ${-SHOULDER_PLATE_POS_Z}
+        ${PI/2} ${0} ${-PI/2}
+      </pose>
+      <collision name="collision">
+        <geometry>
+          <mesh>
+            <uri>model://spacediver/meshes/shoulder_plate.STL</uri>
+          </mesh>
+        </geometry>
+      </collision>
+      <visual name="visual">
+        <geometry>
+          <mesh>
+            <uri>model://spacediver/meshes/shoulder_plate.STL</uri>
+          </mesh>
+        </geometry>
+        <!-- <material>
+          <script>
+            <uri>file://media/materials/scripts/gazebo.material</uri>
+            <name>Gazebo/Grey</name>
+          </script>
+        </material> -->
+      </visual>
+    </link>
+    <!-- DYNAMIXELS -->
     <link name="left_dynamixel_top">
       <pose>
-        ${DYNAMIXEL_LEFT_TOP_POS_X} ${DYNAMIXEL_LEFT_TOP_POS_Y} ${DYNAMIXEL_LEFT_TOP_POS_Z}
+        ${DYNAMIXEL_TOP_POS_X} ${DYNAMIXEL_TOP_POS_Y} ${DYNAMIXEL_TOP_POS_Z}
       </pose>
       <collision name="collision">
@@ -101,7 +129,7 @@
       </visual>
     </link>
-    <link name="left_dynamixel_bottom">
-      <pose>
-        ${DYNAMIXEL_LEFT_BOT_POS_X} ${DYNAMIXEL_LEFT_BOT_POS_Y} ${DYNAMIXEL_LEFT_BOT_POS_Z}
+    <link name="right_dynamixel_top">
+      <pose>
+        ${-DYNAMIXEL_TOP_POS_X} ${DYNAMIXEL_TOP_POS_Y} ${DYNAMIXEL_TOP_POS_Z}
       </pose>
       <collision name="collision">
@@ -134,5 +162,72 @@
       </visual>
     </link>
-    <link name="misumi_ln">
+    <link name="left_dynamixel_bottom">
+      <pose>
+        ${DYNAMIXEL_BOT_POS_X} ${DYNAMIXEL_BOT_POS_Y} ${DYNAMIXEL_BOT_POS_Z}
+      </pose>
+      <collision name="collision">
+        <geometry>
+          <box>
+            <size>${DYNAMIXEL_X} ${DYNAMIXEL_Y} ${DYNAMIXEL_Z}</size>
+          </box>
+        </geometry>
+        <surface>
+          <friction>
+            <ode>
+              <mu>100</mu>
+              <mu2>50</mu2>
+            </ode>
+          </friction>
+        </surface>
+      </collision>
+      <visual name="visual">
+        <geometry>
+          <box>
+            <size>${DYNAMIXEL_X} ${DYNAMIXEL_Y} ${DYNAMIXEL_Z}</size>
+          </box>
+        </geometry>
+        <material>
+          <script>
+            <uri>file://media/materials/scripts/gazebo.material</uri>
+            <name>Gazebo/Blue</name>
+          </script>
+        </material>
+      </visual>
+    </link>
+    <link name="right_dynamixel_bottom">
+      <pose>
+        ${-DYNAMIXEL_BOT_POS_X} ${DYNAMIXEL_BOT_POS_Y} ${DYNAMIXEL_BOT_POS_Z}
+      </pose>
+      <collision name="collision">
+        <geometry>
+          <box>
+            <size>${DYNAMIXEL_X} ${DYNAMIXEL_Y} ${DYNAMIXEL_Z}</size>
+          </box>
+        </geometry>
+        <surface>
+          <friction>
+            <ode>
+              <mu>100</mu>
+              <mu2>50</mu2>
+            </ode>
+          </friction>
+        </surface>
+      </collision>
+      <visual name="visual">
+        <geometry>
+          <box>
+            <size>${DYNAMIXEL_X} ${DYNAMIXEL_Y} ${DYNAMIXEL_Z}</size>
+          </box>
+        </geometry>
+        <material>
+          <script>
+            <uri>file://media/materials/scripts/gazebo.material</uri>
+            <name>Gazebo/Blue</name>
+          </script>
+        </material>
+      </visual>
+    </link>
+    <!-- MISUMI LN (lower link) -->
+    <link name="left_misumi_ln">
       <pose>
         ${MISUMILN_POS_X} ${MISUMILN_POS_Y} ${MISUMILN_POS_Z}
@@ -160,5 +255,32 @@
       </visual>
     </link>
-    <link name="driving_link">
+    <link name="right_misumi_ln">
+      <pose>
+        ${R_MISUMILN_POS_X} ${R_MISUMILN_POS_Y} ${R_MISUMILN_POS_Z}
+        0 0 ${R_MISUMILN_ROT_Z}
+      </pose>
+      <collision name="collision">
+        <geometry>
+          <mesh>
+            <uri>model://spacediver/meshes/Link_MISUMI_LNMS16-10-200.STL</uri>
+          </mesh>
+        </geometry>
+      </collision>
+      <visual name="visual">
+        <geometry>
+          <mesh>
+            <uri>model://spacediver/meshes/Link_MISUMI_LNMS16-10-200.STL</uri>
+          </mesh>
+        </geometry>
+        <material>
+          <script>
+            <uri>file://media/materials/scripts/gazebo.material</uri>
+            <name>Gazebo/Red</name>
+          </script>
+        </material>
+      </visual>
+    </link>
+    <!-- DRIVING LINK -->
+    <link name="left_driving_link">
       <pose>
         ${DRIVING_POS_X} ${DRIVING_POS_Y} ${DRIVING_POS_Z}
@@ -186,5 +308,32 @@
       </visual>
     </link>
-    <link name="driven_link">
+    <link name="right_driving_link">
+      <pose>
+        ${R_DRIVING_POS_X} ${R_DRIVING_POS_Y} ${R_DRIVING_POS_Z}
+        0 0 ${R_DRIVING_ROT_Z}
+      </pose>
+      <collision name="collision">
+        <geometry>
+          <mesh>
+            <uri>model://spacediver/meshes/upper_arm_driving_link.STL</uri>
+          </mesh>
+        </geometry>
+      </collision>
+      <visual name="visual">
+        <geometry>
+          <mesh>
+            <uri>model://spacediver/meshes/upper_arm_driving_link.STL</uri>
+          </mesh>
+        </geometry>
+        <material>
+          <script>
+            <uri>file://media/materials/scripts/gazebo.material</uri>
+            <name>Gazebo/Green</name>
+          </script>
+        </material>
+      </visual>
+    </link>
+    <!-- DRIVEN LINK -->
+    <link name="left_driven_link">
       <pose>
         ${DRIVEN_POS_X} ${DRIVEN_POS_Y} ${DRIVEN_POS_Z}
@@ -212,5 +361,32 @@
       </visual>
     </link>
-    <link name="misumi_ft">
+    <link name="right_driven_link">
+      <pose>
+        ${R_DRIVEN_POS_X} ${R_DRIVEN_POS_Y} ${R_DRIVEN_POS_Z}
+        0 0 ${R_DRIVEN_ROT_Z}
+      </pose>
+      <collision name="collision">
+        <geometry>
+          <mesh>
+            <uri>model://spacediver/meshes/upper_arm_driven_link.STL</uri>
+          </mesh>
+        </geometry>
+      </collision>
+      <visual name="visual">
+        <geometry>
+          <mesh>
+            <uri>model://spacediver/meshes/upper_arm_driven_link.STL</uri>
+          </mesh>
+        </geometry>
+        <material>
+          <script>
+            <uri>file://media/materials/scripts/gazebo.material</uri>
+            <name>Gazebo/Red</name>
+          </script>
+        </material>
+      </visual>
+    </link>
+    <!-- MISUMI FT (final link) -->
+    <link name="left_misumi_ft">
       <pose>
         ${MISUMIFT_POS_X} ${MISUMIFT_POS_Y} ${MISUMIFT_POS_Z}
@@ -238,19 +414,58 @@
       </visual>
     </link>
+    <link name="right_misumi_ft">
+      <pose>
+        ${R_MISUMIFT_POS_X} ${R_MISUMIFT_POS_Y} ${R_MISUMIFT_POS_Z}
+        0 0 ${R_MISUMIFT_ROT_Z}
+      </pose>
+      <collision name="collision">
+        <geometry>
+          <mesh>
+            <uri>model://spacediver/meshes/Misumi_LNFTS10-P10-V10-L200-S50-W18-T9.STL</uri>
+          </mesh>
+        </geometry>
+      </collision>
+      <visual name="visual">
+        <geometry>
+          <mesh>
+            <uri>model://spacediver/meshes/Misumi_LNFTS10-P10-V10-L200-S50-W18-T9.STL</uri>
+          </mesh>
+        </geometry>
+        <material>
+          <script>
+            <uri>file://media/materials/scripts/gazebo.material</uri>
+            <name>Gazebo/Green</name>
+          </script>
+        </material>
+      </visual>
+    </link>
+    <!-- JOINTS -->
     <joint name="base_to_leftshoulderplate_joint" type="fixed">
       <parent>base_link</parent>
       <child>left_shoulder_plate</child>
     </joint>
+    <joint name="base_to_rightshoulderplate_joint" type="fixed">
+      <parent>base_link</parent>
+      <child>right_shoulder_plate</child>
+    </joint>
     <joint name="leftshoulderplate_to_leftdynamixeltop_joint" type="fixed">
       <parent>left_shoulder_plate</parent>
       <child>left_dynamixel_top</child>
     </joint>
+    <joint name="rightshoulderplate_to_rightdynamixeltop_joint" type="fixed">
+      <parent>right_shoulder_plate</parent>
+      <child>right_dynamixel_top</child>
+    </joint>
     <joint name="leftshoulderplate_to_leftdynamixelbottom_joint" type="fixed">
       <parent>left_shoulder_plate</parent>
       <child>left_dynamixel_bottom</child>
     </joint>
-    <joint name="dynamixel_to_misumiln_joint" type="revolute">
+    <joint name="rightshoulderplate_to_rightdynamixelbottom_joint" type="fixed">
+      <parent>right_shoulder_plate</parent>
+      <child>right_dynamixel_bottom</child>
+    </joint>
+    <joint name="leftdynamixelbottom_to_leftmisumiln_joint" type="revolute">
       <parent>left_dynamixel_bottom</parent>
-      <child>misumi_ln</child>
+      <child>left_misumi_ln</child>
       <pose>
         ${MISUMILN_JOINTA_Y} ${MISUMILN_JOINTA_X} ${MISUMILN_JOINTA_Z}
@@ -260,7 +475,17 @@
       </axis>
     </joint>
-    <joint name="dynamixel_to_driving_joint" type="revolute">
+    <joint name="rightdynamixelbottom_to_rightmisumiln_joint" type="revolute">
+      <parent>right_dynamixel_bottom</parent>
+      <child>right_misumi_ln</child>
+      <pose>
+        ${MISUMILN_JOINTA_Y} ${MISUMILN_JOINTA_X} ${MISUMILN_JOINTA_Z}
+      </pose>
+      <axis>
+        <xyz>0 0 1</xyz>
+      </axis>
+    </joint>
+    <joint name="leftdynamixeltop_to_leftdriving_joint" type="revolute">
       <parent>left_dynamixel_top</parent>
-      <child>driving_link</child>
+      <child>left_driving_link</child>
       <pose>
         ${DRIVING_JOINTA_X} ${DRIVING_JOINTA_Y} ${DRIVING_JOINTA_Z}
@@ -270,7 +495,17 @@
       </axis>
     </joint>
-    <joint name="driving_to_driven_joint" type="revolute">
-      <parent>driving_link</parent>
-      <child>driven_link</child>
+    <joint name="rightdynamixeltop_to_rightdriving_joint" type="revolute">
+      <parent>right_dynamixel_top</parent>
+      <child>right_driving_link</child>
+      <pose>
+        ${DRIVING_JOINTA_X} ${DRIVING_JOINTA_Y} ${DRIVING_JOINTA_Z}
+      </pose>
+      <axis>
+        <xyz>0 0 1</xyz>
+      </axis>
+    </joint>
+    <joint name="leftdriving_to_leftdriven_joint" type="revolute">
+      <parent>left_driving_link</parent>
+      <child>left_driven_link</child>
       <pose>
         ${DRIVEN_JOINTA_X} ${DRIVEN_JOINTA_Y} ${DRIVEN_JOINTA_Z}
@@ -280,7 +515,17 @@
       </axis>
     </joint>
-    <joint name="driven_to_misumift_joint" type="revolute">
-      <parent>driven_link</parent>
-      <child>misumi_ft</child>
+    <joint name="rightdriving_to_rightdriven_joint" type="revolute">
+      <parent>right_driving_link</parent>
+      <child>right_driven_link</child>
+      <pose>
+        ${DRIVEN_JOINTA_X} ${DRIVEN_JOINTA_Y} ${DRIVEN_JOINTA_Z}
+      </pose>
+      <axis>
+        <xyz>0 0 1</xyz>
+      </axis>
+    </joint>
+    <joint name="leftdriven_to_leftmisumift_joint" type="revolute">
+      <parent>left_driven_link</parent>
+      <child>left_misumi_ft</child>
       <pose>
         ${MISUMIFT_JOINTA_X} ${MISUMIFT_JOINTA_Y} ${MISUMIFT_JOINTA_Z}
@@ -290,7 +535,27 @@
       </axis>
     </joint>
-    <joint name="misumiln_to_misumift_joint" type="revolute">
-      <parent>misumi_ln</parent>
-      <child>misumi_ft</child>
+    <joint name="rightdriven_to_rightmisumift_joint" type="revolute">
+      <parent>right_driven_link</parent>
+      <child>right_misumi_ft</child>
+      <pose>
+        ${MISUMIFT_JOINTA_X} ${MISUMIFT_JOINTA_Y} ${MISUMIFT_JOINTA_Z}
+      </pose>
+      <axis>
+        <xyz>0 0 1</xyz>
+      </axis>
+    </joint>
+    <joint name="leftmisumiln_to_leftmisumift_joint" type="revolute">
+      <parent>left_misumi_ln</parent>
+      <child>left_misumi_ft</child>
+      <pose>
+        ${MISUMIFT_JOINTB_X} ${MISUMIFT_JOINTB_Y} ${MISUMIFT_JOINTB_Z}
+      </pose>
+      <axis>
+        <xyz>0 0 1</xyz>
+      </axis>
+    </joint>
+    <joint name="rightmisumiln_to_rightmisumift_joint" type="revolute">
+      <parent>right_misumi_ln</parent>
+      <child>right_misumi_ft</child>
       <pose>
         ${MISUMIFT_JOINTB_X} ${MISUMIFT_JOINTB_Y} ${MISUMIFT_JOINTB_Z}

File: spacediver_ros2_control/description/urdf/macros/properties.xacro (robot description, xacro)
@@ -8,5 +8,5 @@
   <xacro:property name="BASE_MASS" value="50"/>
   <xacro:property name="BASE_INERTIA_Z" value="0.13526810"/>
-  <xacro:property name="BASE_TO_SHOULDER_PLATE_X" value="0.0045"/>
+  <!-- SHOULDER PLATE -->
   <xacro:property name="SHOULDER_PLATE_X" value="0.03"/>
   <xacro:property name="SHOULDER_PLATE_Y" value="0.0585"/>
@@ -18,4 +18,5 @@
   <xacro:property name="SHOULDER_PLATE_POS_Y" value="${SHOULDER_PLATE_Y/2}"/>
   <xacro:property name="SHOULDER_PLATE_POS_Z" value="${SHOULDER_PLATE_Z/2}"/>
+  <!-- DYNAMIXEL -->
   <xacro:property name="DYNAMIXEL_X" value="0.0335"/>
   <xacro:property name="DYNAMIXEL_Y" value="0.0585"/>
@@ -23,20 +24,28 @@
   <xacro:property name="DYNAMIXEL_JOINTB_X" value="0"/>
   <xacro:property name="DYNAMIXEL_JOINTB_Y" value="${DYNAMIXEL_Y - 0.04475}"/>
-  <xacro:property name="DYNAMIXEL_LEFT_TOP_POS_X" value="${SHOULDER_PLATE_POS_X + SHOULDER_PLATE_X + DYNAMIXEL_X/2}"/>
-  <xacro:property name="DYNAMIXEL_LEFT_TOP_POS_Y" value="${SHOULDER_PLATE_POS_Y - SHOULDER_PLATE_Y/2}"/>
-  <xacro:property name="DYNAMIXEL_LEFT_TOP_POS_Z" value="${SHOULDER_PLATE_POS_Z - DYNAMIXEL_Z/2}"/>
-  <xacro:property name="DYNAMIXEL_LEFT_BOT_POS_X" value="${SHOULDER_PLATE_POS_X + SHOULDER_PLATE_X + DYNAMIXEL_X/2}"/>
-  <xacro:property name="DYNAMIXEL_LEFT_BOT_POS_Y" value="${SHOULDER_PLATE_POS_Y - SHOULDER_PLATE_Y/2}"/>
-  <xacro:property name="DYNAMIXEL_LEFT_BOT_POS_Z" value="${SHOULDER_PLATE_POS_Z - SHOULDER_PLATE_Z + DYNAMIXEL_Z/2}"/>
+  <xacro:property name="DYNAMIXEL_TOP_POS_X" value="${SHOULDER_PLATE_POS_X + SHOULDER_PLATE_X + DYNAMIXEL_X/2}"/>
+  <xacro:property name="DYNAMIXEL_TOP_POS_Y" value="${SHOULDER_PLATE_POS_Y - SHOULDER_PLATE_Y/2}"/>
+  <xacro:property name="DYNAMIXEL_TOP_POS_Z" value="${SHOULDER_PLATE_POS_Z - DYNAMIXEL_Z/2}"/>
+  <xacro:property name="DYNAMIXEL_BOT_POS_X" value="${SHOULDER_PLATE_POS_X + SHOULDER_PLATE_X + DYNAMIXEL_X/2}"/>
+  <xacro:property name="DYNAMIXEL_BOT_POS_Y" value="${SHOULDER_PLATE_POS_Y - SHOULDER_PLATE_Y/2}"/>
+  <xacro:property name="DYNAMIXEL_BOT_POS_Z" value="${SHOULDER_PLATE_POS_Z - SHOULDER_PLATE_Z + DYNAMIXEL_Z/2}"/>
+  <!-- MIUSMI LN (LOWER LINK) -->
   <xacro:property name="MISUMILN_X" value="0.032"/>
   <xacro:property name="MISUMILN_Y" value="0.225"/>
   <xacro:property name="MISUMILN_Z" value="0.009"/>
-  <xacro:property name="MISUMILN_ROT_Z" value="${-PI/2+ROT}"/>
   <xacro:property name="MISUMILN_JOINTA_X" value="0.016"/>
   <xacro:property name="MISUMILN_JOINTA_Y" value="0.012"/>
   <xacro:property name="MISUMILN_JOINTA_Z" value="${0.01 + MISUMILN_Z/2}"/>
-  <xacro:property name="MISUMILN_POS_X" value="${DYNAMIXEL_LEFT_BOT_POS_X + math.cos(ROT)*(-MISUMILN_JOINTA_X) - math.sin(ROT)*(MISUMILN_JOINTA_Y)}"/>
-  <xacro:property name="MISUMILN_POS_Y" value="${DYNAMIXEL_LEFT_BOT_POS_Y - DYNAMIXEL_JOINTB_Y + math.sin(ROT)*(-MISUMILN_JOINTA_X) + math.cos(ROT)*(MISUMILN_JOINTA_Y)}"/>
-  <xacro:property name="MISUMILN_POS_Z" value="${DYNAMIXEL_LEFT_BOT_POS_Z + DYNAMIXEL_Z/2 + 0.0045}"/>
+  <!-- LEFT -->
+  <xacro:property name="MISUMILN_ROT_Z" value="${-PI/2+ROT}"/>
+  <xacro:property name="MISUMILN_POS_X" value="${DYNAMIXEL_BOT_POS_X + math.cos(ROT)*(-MISUMILN_JOINTA_X) - math.sin(ROT)*(MISUMILN_JOINTA_Y)}"/>
+  <xacro:property name="MISUMILN_POS_Y" value="${DYNAMIXEL_BOT_POS_Y - DYNAMIXEL_JOINTB_Y + math.sin(ROT)*(-MISUMILN_JOINTA_X) + math.cos(ROT)*(MISUMILN_JOINTA_Y)}"/>
+  <xacro:property name="MISUMILN_POS_Z" value="${DYNAMIXEL_BOT_POS_Z + DYNAMIXEL_Z/2 + 0.0045}"/>
+  <!-- RIGHT -->
+  <xacro:property name="R_MISUMILN_ROT_Z" value="${-PI/2-ROT}"/>
+  <xacro:property name="R_MISUMILN_POS_X" value="${-DYNAMIXEL_BOT_POS_X + math.cos(-ROT)*(-MISUMILN_JOINTA_X) - math.sin(-ROT)*(MISUMILN_JOINTA_Y)}"/>
+  <xacro:property name="R_MISUMILN_POS_Y" value="${DYNAMIXEL_BOT_POS_Y - DYNAMIXEL_JOINTB_Y + math.sin(-ROT)*(-MISUMILN_JOINTA_X) + math.cos(-ROT)*(MISUMILN_JOINTA_Y)}"/>
+  <xacro:property name="R_MISUMILN_POS_Z" value="${DYNAMIXEL_BOT_POS_Z + DYNAMIXEL_Z/2 + 0.0045}"/>
+  <!-- DRIVING LINK -->
   <xacro:property name="DRIVING_X" value="0.076"/>
   <xacro:property name="DRIVING_Y" value="0.026"/>
@@ -45,26 +54,39 @@
   <xacro:property name="DRIVING_JOINTA_Y" value="0.013"/>
   <xacro:property name="DRIVING_JOINTA_Z" value="${DRIVING_Z/2}"/>
+  <!-- LEFT -->
   <xacro:property name="DRIVING_ROT_Z" value="${0}"/>
-  <xacro:property name="DRIVING_POS_X" value="${DYNAMIXEL_LEFT_TOP_POS_X - DRIVING_JOINTA_X}"/>
-  <xacro:property name="DRIVING_POS_Y" value="${DYNAMIXEL_LEFT_TOP_POS_Y - DYNAMIXEL_JOINTB_Y - DRIVING_JOINTA_Y}"/>
-  <xacro:property name="DRIVING_POS_Z" value="${DYNAMIXEL_LEFT_TOP_POS_Z - DYNAMIXEL_Z/2 - DRIVING_Z - 0.0045}"/>
+  <xacro:property name="DRIVING_POS_X" value="${DYNAMIXEL_TOP_POS_X - DRIVING_JOINTA_X}"/>
+  <xacro:property name="DRIVING_POS_Y" value="${DYNAMIXEL_TOP_POS_Y - DYNAMIXEL_JOINTB_Y - DRIVING_JOINTA_Y}"/>
+  <xacro:property name="DRIVING_POS_Z" value="${DYNAMIXEL_TOP_POS_Z - DYNAMIXEL_Z/2 - DRIVING_Z - 0.0045}"/>
+  <!-- RIGHT -->
+  <xacro:property name="R_DRIVING_ROT_Z" value="${PI}"/>
+  <xacro:property name="R_DRIVING_POS_X" value="${-DYNAMIXEL_TOP_POS_X + DRIVING_JOINTA_X}"/>
+  <xacro:property name="R_DRIVING_POS_Y" value="${DYNAMIXEL_TOP_POS_Y - DYNAMIXEL_JOINTB_Y + DRIVING_JOINTA_Y}"/>
+  <xacro:property name="R_DRIVING_POS_Z" value="${DYNAMIXEL_TOP_POS_Z - DYNAMIXEL_Z/2 - DRIVING_Z - 0.0045}"/>
   <xacro:property name="DRIVING_JOINTB_X" value="0.063"/>
   <xacro:property name="DRIVING_JOINTB_Y" value="0.013"/>
+  <!-- DRIVEN LINK -->
   <xacro:property name="DRIVEN_X" value="0.026"/>
   <xacro:property name="DRIVEN_Y" value="0.226"/>
   <xacro:property name="DRIVEN_Z" value="0.004"/>
-  <xacro:property name="DRIVEN_ROT_Z" value="${-PI/2+ROT}"/>
   <xacro:property name="DRIVEN_JOINTA_X" value="0.013"/>
   <xacro:property name="DRIVEN_JOINTA_Y" value="0.013"/>
   <xacro:property name="DRIVEN_JOINTA_Z" value="${DRIVEN_Z/2}"/>
+  <!-- LEFT -->
+  <xacro:property name="DRIVEN_ROT_Z" value="${-PI/2+ROT}"/>
   <xacro:property name="DRIVEN_POS_X" value="${DRIVING_POS_X + DRIVING_JOINTB_X + math.cos(ROT)*(-DRIVEN_JOINTA_X) - math.sin(ROT)*(DRIVEN_JOINTA_Y)}"/>
   <xacro:property name="DRIVEN_POS_Y" value="${DRIVING_POS_Y + DRIVING_JOINTB_Y + math.sin(ROT)*(-DRIVEN_JOINTA_X) + math.cos(ROT)*(DRIVEN_JOINTA_Y)}"/>
   <xacro:property name="DRIVEN_POS_Z" value="${DRIVING_POS_Z - DRIVING_Z - 0.01}"/>
+  <!-- RIGHT -->
+  <xacro:property name="R_DRIVEN_ROT_Z" value="${-PI/2-ROT}"/>
+  <xacro:property name="R_DRIVEN_POS_X" value="${-DRIVING_POS_X - DRIVING_JOINTB_X + math.cos(-ROT)*(-DRIVEN_JOINTA_X) - math.sin(-ROT)*(DRIVEN_JOINTA_Y)}"/>
+  <xacro:property name="R_DRIVEN_POS_Y" value="${DRIVING_POS_Y + DRIVING_JOINTB_Y + math.sin(-ROT)*(-DRIVEN_JOINTA_X) + math.cos(-ROT)*(DRIVEN_JOINTA_Y)}"/>
+  <xacro:property name="R_DRIVEN_POS_Z" value="${DRIVING_POS_Z - DRIVING_Z - 0.01}"/>
   <xacro:property name="DRIVEN_JOINTB_X" value="0.013"/>
   <xacro:property name="DRIVEN_JOINTB_Y" value="0.213"/>
+  <!-- MISUMI FT (final link) -->
   <xacro:property name="MISUMIFT_X" value="0.268"/>
   <xacro:property name="MISUMIFT_Y" value="0.018"/>
   <xacro:property name="MISUMIFT_Z" value="0.009"/>
-  <xacro:property name="MISUMIFT_ROT_Z" value="${PI}"/>
   <xacro:property name="MISUMIFT_JOINTA_X" value="0.009"/>
   <xacro:property name="MISUMIFT_JOINTA_Y" value="0.009"/>
@@ -73,7 +95,14 @@
   <xacro:property name="MISUMIFT_JOINTB_Y" value="0.009"/>
   <xacro:property name="MISUMIFT_JOINTB_Z" value="${MISUMIFT_Z/2}"/>
+  <!-- LEFT -->
+  <xacro:property name="MISUMIFT_ROT_Z" value="${PI}"/>
   <xacro:property name="MISUMIFT_POS_X" value="${DRIVEN_POS_X + math.cos(ROT)*(DRIVEN_JOINTB_X) - math.sin(ROT)*(-DRIVEN_JOINTB_Y) + MISUMIFT_JOINTA_X}"/>
   <xacro:property name="MISUMIFT_POS_Y" value="${DRIVEN_POS_Y + math.sin(ROT)*(DRIVEN_JOINTB_X) + math.cos(ROT)*(-DRIVEN_JOINTB_Y) + MISUMIFT_JOINTA_Y}"/>
   <xacro:property name="MISUMIFT_POS_Z" value="${DRIVEN_POS_Z - MISUMIFT_Z - 0.005}"/>
+  <!-- RIGHT -->
+  <xacro:property name="R_MISUMIFT_ROT_Z" value="${0}"/>
+  <xacro:property name="R_MISUMIFT_POS_X" value="${-DRIVEN_POS_X + math.cos(-ROT)*(-DRIVEN_JOINTB_X) - math.sin(-ROT)*(-DRIVEN_JOINTB_Y) - MISUMIFT_JOINTA_X}"/>
+  <xacro:property name="R_MISUMIFT_POS_Y" value="${DRIVEN_POS_Y + math.sin(-ROT)*(-DRIVEN_JOINTB_X) + math.cos(-ROT)*(-DRIVEN_JOINTB_Y) - MISUMIFT_JOINTA_Y}"/>
+  <xacro:property name="R_MISUMIFT_POS_Z" value="${DRIVEN_POS_Z - MISUMIFT_Z - 0.005}"/>
   <xacro:property name="ACTIVE_JOINT_LA_LOWER" value="-${PI}"/>
   <xacro:property name="ACTIVE_JOINT_LA_UPPER" value=" ${PI}"/>
