Commit message: redefined left and right

File: spacediver_ros2_control/description/gazebo/models/spacediver.sdf.xacro (robot description, xacro)
@@ -231,6 +231,6 @@
     <link name="left_misumi_ln">
       <pose>
-        ${MISUMILN_POS_X} ${MISUMILN_POS_Y} ${MISUMILN_POS_Z}
-        0 0 ${MISUMILN_ROT_Z}
+        ${L_MISUMILN_POS_X} ${L_MISUMILN_POS_Y} ${L_MISUMILN_POS_Z}
+        0 0 ${L_MISUMILN_ROT_Z}
       </pose>
       <collision name="collision">
@@ -284,6 +284,6 @@
     <link name="left_driving_link">
       <pose>
-        ${DRIVING_POS_X} ${DRIVING_POS_Y} ${DRIVING_POS_Z}
-        0 0 ${DRIVING_ROT_Z}
+        ${L_DRIVING_POS_X} ${L_DRIVING_POS_Y} ${L_DRIVING_POS_Z}
+        0 0 ${L_DRIVING_ROT_Z}
       </pose>
       <collision name="collision">
@@ -337,6 +337,6 @@
     <link name="left_driven_link">
       <pose>
-        ${DRIVEN_POS_X} ${DRIVEN_POS_Y} ${DRIVEN_POS_Z}
-        0 0 ${DRIVEN_ROT_Z}
+        ${L_DRIVEN_POS_X} ${L_DRIVEN_POS_Y} ${L_DRIVEN_POS_Z}
+        0 0 ${L_DRIVEN_ROT_Z}
       </pose>
       <collision name="collision">
@@ -390,6 +390,6 @@
     <link name="left_misumi_ft">
       <pose>
-        ${MISUMIFT_POS_X} ${MISUMIFT_POS_Y} ${MISUMIFT_POS_Z}
-        0 0 ${MISUMIFT_ROT_Z}
+        ${L_MISUMIFT_POS_X} ${L_MISUMIFT_POS_Y} ${L_MISUMIFT_POS_Z}
+        0 0 ${L_MISUMIFT_ROT_Z}
       </pose>
       <collision name="collision">

File: spacediver_ros2_control/description/urdf/macros/properties.xacro (robot description, xacro)
@@ -38,8 +38,8 @@
   <xacro:property name="MISUMILN_JOINTA_Z" value="${0.01 + MISUMILN_Z/2}"/>
   <!-- LEFT -->
-  <xacro:property name="MISUMILN_ROT_Z" value="${-PI/2+ROT}"/>
-  <xacro:property name="MISUMILN_POS_X" value="${DYNAMIXEL_BOT_POS_X + math.cos(ROT)*(-MISUMILN_JOINTA_X) - math.sin(ROT)*(MISUMILN_JOINTA_Y)}"/>
-  <xacro:property name="MISUMILN_POS_Y" value="${DYNAMIXEL_BOT_POS_Y - DYNAMIXEL_JOINTB_Y + math.sin(ROT)*(-MISUMILN_JOINTA_X) + math.cos(ROT)*(MISUMILN_JOINTA_Y)}"/>
-  <xacro:property name="MISUMILN_POS_Z" value="${DYNAMIXEL_BOT_POS_Z + DYNAMIXEL_Z/2 + 0.0045}"/>
+  <xacro:property name="L_MISUMILN_ROT_Z" value="${-PI/2+ROT}"/>
+  <xacro:property name="L_MISUMILN_POS_X" value="${DYNAMIXEL_BOT_POS_X + math.cos(ROT)*(-MISUMILN_JOINTA_X) - math.sin(ROT)*(MISUMILN_JOINTA_Y)}"/>
+  <xacro:property name="L_MISUMILN_POS_Y" value="${DYNAMIXEL_BOT_POS_Y - DYNAMIXEL_JOINTB_Y + math.sin(ROT)*(-MISUMILN_JOINTA_X) + math.cos(ROT)*(MISUMILN_JOINTA_Y)}"/>
+  <xacro:property name="L_MISUMILN_POS_Z" value="${DYNAMIXEL_BOT_POS_Z + DYNAMIXEL_Z/2 + 0.0045}"/>
   <!-- RIGHT -->
   <xacro:property name="R_MISUMILN_ROT_Z" value="${-PI/2-ROT}"/>
@@ -55,8 +55,8 @@
   <xacro:property name="DRIVING_JOINTA_Z" value="${DRIVING_Z/2}"/>
   <!-- LEFT -->
-  <xacro:property name="DRIVING_ROT_Z" value="${0}"/>
-  <xacro:property name="DRIVING_POS_X" value="${DYNAMIXEL_TOP_POS_X - DRIVING_JOINTA_X}"/>
-  <xacro:property name="DRIVING_POS_Y" value="${DYNAMIXEL_TOP_POS_Y - DYNAMIXEL_JOINTB_Y - DRIVING_JOINTA_Y}"/>
-  <xacro:property name="DRIVING_POS_Z" value="${DYNAMIXEL_TOP_POS_Z - DYNAMIXEL_Z/2 - DRIVING_Z - 0.0045}"/>
+  <xacro:property name="L_DRIVING_ROT_Z" value="${0}"/>
+  <xacro:property name="L_DRIVING_POS_X" value="${DYNAMIXEL_TOP_POS_X - DRIVING_JOINTA_X}"/>
+  <xacro:property name="L_DRIVING_POS_Y" value="${DYNAMIXEL_TOP_POS_Y - DYNAMIXEL_JOINTB_Y - DRIVING_JOINTA_Y}"/>
+  <xacro:property name="L_DRIVING_POS_Z" value="${DYNAMIXEL_TOP_POS_Z - DYNAMIXEL_Z/2 - DRIVING_Z - 0.0045}"/>
   <!-- RIGHT -->
   <xacro:property name="R_DRIVING_ROT_Z" value="${PI}"/>
@@ -74,13 +74,13 @@
   <xacro:property name="DRIVEN_JOINTA_Z" value="${DRIVEN_Z/2}"/>
   <!-- LEFT -->
-  <xacro:property name="DRIVEN_ROT_Z" value="${-PI/2+ROT}"/>
-  <xacro:property name="DRIVEN_POS_X" value="${DRIVING_POS_X + DRIVING_JOINTB_X + math.cos(ROT)*(-DRIVEN_JOINTA_X) - math.sin(ROT)*(DRIVEN_JOINTA_Y)}"/>
-  <xacro:property name="DRIVEN_POS_Y" value="${DRIVING_POS_Y + DRIVING_JOINTB_Y + math.sin(ROT)*(-DRIVEN_JOINTA_X) + math.cos(ROT)*(DRIVEN_JOINTA_Y)}"/>
-  <xacro:property name="DRIVEN_POS_Z" value="${DRIVING_POS_Z - DRIVING_Z - 0.01}"/>
+  <xacro:property name="L_DRIVEN_ROT_Z" value="${-PI/2+ROT}"/>
+  <xacro:property name="L_DRIVEN_POS_X" value="${L_DRIVING_POS_X + DRIVING_JOINTB_X + math.cos(ROT)*(-DRIVEN_JOINTA_X) - math.sin(ROT)*(DRIVEN_JOINTA_Y)}"/>
+  <xacro:property name="L_DRIVEN_POS_Y" value="${L_DRIVING_POS_Y + DRIVING_JOINTB_Y + math.sin(ROT)*(-DRIVEN_JOINTA_X) + math.cos(ROT)*(DRIVEN_JOINTA_Y)}"/>
+  <xacro:property name="L_DRIVEN_POS_Z" value="${L_DRIVING_POS_Z - DRIVING_Z - 0.01}"/>
   <!-- RIGHT -->
   <xacro:property name="R_DRIVEN_ROT_Z" value="${-PI/2-ROT}"/>
-  <xacro:property name="R_DRIVEN_POS_X" value="${-DRIVING_POS_X - DRIVING_JOINTB_X + math.cos(-ROT)*(-DRIVEN_JOINTA_X) - math.sin(-ROT)*(DRIVEN_JOINTA_Y)}"/>
-  <xacro:property name="R_DRIVEN_POS_Y" value="${DRIVING_POS_Y + DRIVING_JOINTB_Y + math.sin(-ROT)*(-DRIVEN_JOINTA_X) + math.cos(-ROT)*(DRIVEN_JOINTA_Y)}"/>
-  <xacro:property name="R_DRIVEN_POS_Z" value="${DRIVING_POS_Z - DRIVING_Z - 0.01}"/>
+  <xacro:property name="R_DRIVEN_POS_X" value="${R_DRIVING_POS_X - DRIVING_JOINTB_X + math.cos(-ROT)*(-DRIVEN_JOINTA_X) - math.sin(-ROT)*(DRIVEN_JOINTA_Y)}"/>
+  <xacro:property name="R_DRIVEN_POS_Y" value="${R_DRIVING_POS_Y - DRIVING_JOINTB_Y + math.sin(-ROT)*(-DRIVEN_JOINTA_X) + math.cos(-ROT)*(DRIVEN_JOINTA_Y)}"/>
+  <xacro:property name="R_DRIVEN_POS_Z" value="${R_DRIVING_POS_Z - DRIVING_Z - 0.01}"/>
   <xacro:property name="DRIVEN_JOINTB_X" value="0.013"/>
   <xacro:property name="DRIVEN_JOINTB_Y" value="0.213"/>
@@ -96,13 +96,13 @@
   <xacro:property name="MISUMIFT_JOINTB_Z" value="${MISUMIFT_Z/2}"/>
   <!-- LEFT -->
-  <xacro:property name="MISUMIFT_ROT_Z" value="${PI}"/>
-  <xacro:property name="MISUMIFT_POS_X" value="${DRIVEN_POS_X + math.cos(ROT)*(DRIVEN_JOINTB_X) - math.sin(ROT)*(-DRIVEN_JOINTB_Y) + MISUMIFT_JOINTA_X}"/>
-  <xacro:property name="MISUMIFT_POS_Y" value="${DRIVEN_POS_Y + math.sin(ROT)*(DRIVEN_JOINTB_X) + math.cos(ROT)*(-DRIVEN_JOINTB_Y) + MISUMIFT_JOINTA_Y}"/>
-  <xacro:property name="MISUMIFT_POS_Z" value="${DRIVEN_POS_Z - MISUMIFT_Z - 0.005}"/>
+  <xacro:property name="L_MISUMIFT_ROT_Z" value="${PI}"/>
+  <xacro:property name="L_MISUMIFT_POS_X" value="${L_DRIVEN_POS_X + math.cos(ROT)*(DRIVEN_JOINTB_X) - math.sin(ROT)*(-DRIVEN_JOINTB_Y) + MISUMIFT_JOINTA_X}"/>
+  <xacro:property name="L_MISUMIFT_POS_Y" value="${L_DRIVEN_POS_Y + math.sin(ROT)*(DRIVEN_JOINTB_X) + math.cos(ROT)*(-DRIVEN_JOINTB_Y) + MISUMIFT_JOINTA_Y}"/>
+  <xacro:property name="L_MISUMIFT_POS_Z" value="${L_DRIVEN_POS_Z - MISUMIFT_Z - 0.005}"/>
   <!-- RIGHT -->
   <xacro:property name="R_MISUMIFT_ROT_Z" value="${0}"/>
-  <xacro:property name="R_MISUMIFT_POS_X" value="${-DRIVEN_POS_X + math.cos(-ROT)*(-DRIVEN_JOINTB_X) - math.sin(-ROT)*(-DRIVEN_JOINTB_Y) - MISUMIFT_JOINTA_X}"/>
-  <xacro:property name="R_MISUMIFT_POS_Y" value="${DRIVEN_POS_Y + math.sin(-ROT)*(-DRIVEN_JOINTB_X) + math.cos(-ROT)*(-DRIVEN_JOINTB_Y) - MISUMIFT_JOINTA_Y}"/>
-  <xacro:property name="R_MISUMIFT_POS_Z" value="${DRIVEN_POS_Z - MISUMIFT_Z - 0.005}"/>
+  <xacro:property name="R_MISUMIFT_POS_X" value="${R_DRIVEN_POS_X + math.cos(-ROT)*(DRIVEN_JOINTB_X) - math.sin(-ROT)*(-DRIVEN_JOINTB_Y) - MISUMIFT_JOINTA_X}"/>
+  <xacro:property name="R_MISUMIFT_POS_Y" value="${R_DRIVEN_POS_Y + math.sin(-ROT)*(DRIVEN_JOINTB_X) + math.cos(-ROT)*(-DRIVEN_JOINTB_Y) - MISUMIFT_JOINTA_Y}"/>
+  <xacro:property name="R_MISUMIFT_POS_Z" value="${R_DRIVEN_POS_Z - MISUMIFT_Z - 0.005}"/>
   <xacro:property name="ACTIVE_JOINT_LA_LOWER" value="-${PI}"/>
   <xacro:property name="ACTIVE_JOINT_LA_UPPER" value=" ${PI}"/>

Commit message: left and right have same z coordinates

File: spacediver_ros2_control/description/gazebo/models/spacediver.sdf.xacro (robot description, xacro)
@@ -231,5 +231,5 @@
     <link name="left_misumi_ln">
       <pose>
-        ${L_MISUMILN_POS_X} ${L_MISUMILN_POS_Y} ${L_MISUMILN_POS_Z}
+        ${L_MISUMILN_POS_X} ${L_MISUMILN_POS_Y} ${MISUMILN_POS_Z}
         0 0 ${L_MISUMILN_ROT_Z}
       </pose>
@@ -257,5 +257,5 @@
     <link name="right_misumi_ln">
       <pose>
-        ${R_MISUMILN_POS_X} ${R_MISUMILN_POS_Y} ${R_MISUMILN_POS_Z}
+        ${R_MISUMILN_POS_X} ${R_MISUMILN_POS_Y} ${MISUMILN_POS_Z}
         0 0 ${R_MISUMILN_ROT_Z}
       </pose>
@@ -284,5 +284,5 @@
     <link name="left_driving_link">
       <pose>
-        ${L_DRIVING_POS_X} ${L_DRIVING_POS_Y} ${L_DRIVING_POS_Z}
+        ${L_DRIVING_POS_X} ${L_DRIVING_POS_Y} ${DRIVING_POS_Z}
         0 0 ${L_DRIVING_ROT_Z}
       </pose>
@@ -310,5 +310,5 @@
     <link name="right_driving_link">
       <pose>
-        ${R_DRIVING_POS_X} ${R_DRIVING_POS_Y} ${R_DRIVING_POS_Z}
+        ${R_DRIVING_POS_X} ${R_DRIVING_POS_Y} ${DRIVING_POS_Z}
         0 0 ${R_DRIVING_ROT_Z}
       </pose>
@@ -337,5 +337,5 @@
     <link name="left_driven_link">
       <pose>
-        ${L_DRIVEN_POS_X} ${L_DRIVEN_POS_Y} ${L_DRIVEN_POS_Z}
+        ${L_DRIVEN_POS_X} ${L_DRIVEN_POS_Y} ${DRIVEN_POS_Z}
         0 0 ${L_DRIVEN_ROT_Z}
       </pose>
@@ -363,5 +363,5 @@
     <link name="right_driven_link">
       <pose>
-        ${R_DRIVEN_POS_X} ${R_DRIVEN_POS_Y} ${R_DRIVEN_POS_Z}
+        ${R_DRIVEN_POS_X} ${R_DRIVEN_POS_Y} ${DRIVEN_POS_Z}
         0 0 ${R_DRIVEN_ROT_Z}
       </pose>
@@ -390,5 +390,5 @@
     <link name="left_misumi_ft">
       <pose>
-        ${L_MISUMIFT_POS_X} ${L_MISUMIFT_POS_Y} ${L_MISUMIFT_POS_Z}
+        ${L_MISUMIFT_POS_X} ${L_MISUMIFT_POS_Y} ${MISUMIFT_POS_Z}
         0 0 ${L_MISUMIFT_ROT_Z}
       </pose>
@@ -416,5 +416,5 @@
     <link name="right_misumi_ft">
       <pose>
-        ${R_MISUMIFT_POS_X} ${R_MISUMIFT_POS_Y} ${R_MISUMIFT_POS_Z}
+        ${R_MISUMIFT_POS_X} ${R_MISUMIFT_POS_Y} ${MISUMIFT_POS_Z}
         0 0 ${R_MISUMIFT_ROT_Z}
       </pose>

File: spacediver_ros2_control/description/urdf/macros/properties.xacro (robot description, xacro)
@@ -41,10 +41,9 @@
   <xacro:property name="L_MISUMILN_POS_X" value="${DYNAMIXEL_BOT_POS_X + math.cos(ROT)*(-MISUMILN_JOINTA_X) - math.sin(ROT)*(MISUMILN_JOINTA_Y)}"/>
   <xacro:property name="L_MISUMILN_POS_Y" value="${DYNAMIXEL_BOT_POS_Y - DYNAMIXEL_JOINTB_Y + math.sin(ROT)*(-MISUMILN_JOINTA_X) + math.cos(ROT)*(MISUMILN_JOINTA_Y)}"/>
-  <xacro:property name="L_MISUMILN_POS_Z" value="${DYNAMIXEL_BOT_POS_Z + DYNAMIXEL_Z/2 + 0.0045}"/>
   <!-- RIGHT -->
   <xacro:property name="R_MISUMILN_ROT_Z" value="${-PI/2-ROT}"/>
   <xacro:property name="R_MISUMILN_POS_X" value="${-DYNAMIXEL_BOT_POS_X + math.cos(-ROT)*(-MISUMILN_JOINTA_X) - math.sin(-ROT)*(MISUMILN_JOINTA_Y)}"/>
   <xacro:property name="R_MISUMILN_POS_Y" value="${DYNAMIXEL_BOT_POS_Y - DYNAMIXEL_JOINTB_Y + math.sin(-ROT)*(-MISUMILN_JOINTA_X) + math.cos(-ROT)*(MISUMILN_JOINTA_Y)}"/>
-  <xacro:property name="R_MISUMILN_POS_Z" value="${DYNAMIXEL_BOT_POS_Z + DYNAMIXEL_Z/2 + 0.0045}"/>
+  <xacro:property name="MISUMILN_POS_Z" value="${DYNAMIXEL_BOT_POS_Z + DYNAMIXEL_Z/2 + 0.0045}"/>
   <!-- DRIVING LINK -->
   <xacro:property name="DRIVING_X" value="0.076"/>
@@ -58,10 +57,9 @@
   <xacro:property name="L_DRIVING_POS_X" value="${DYNAMIXEL_TOP_POS_X - DRIVING_JOINTA_X}"/>
   <xacro:property name="L_DRIVING_POS_Y" value="${DYNAMIXEL_TOP_POS_Y - DYNAMIXEL_JOINTB_Y - DRIVING_JOINTA_Y}"/>
-  <xacro:property name="L_DRIVING_POS_Z" value="${DYNAMIXEL_TOP_POS_Z - DYNAMIXEL_Z/2 - DRIVING_Z - 0.0045}"/>
   <!-- RIGHT -->
   <xacro:property name="R_DRIVING_ROT_Z" value="${PI}"/>
   <xacro:property name="R_DRIVING_POS_X" value="${-DYNAMIXEL_TOP_POS_X + DRIVING_JOINTA_X}"/>
   <xacro:property name="R_DRIVING_POS_Y" value="${DYNAMIXEL_TOP_POS_Y - DYNAMIXEL_JOINTB_Y + DRIVING_JOINTA_Y}"/>
-  <xacro:property name="R_DRIVING_POS_Z" value="${DYNAMIXEL_TOP_POS_Z - DYNAMIXEL_Z/2 - DRIVING_Z - 0.0045}"/>
+  <xacro:property name="DRIVING_POS_Z" value="${DYNAMIXEL_TOP_POS_Z - DYNAMIXEL_Z/2 - DRIVING_Z - 0.0045}"/>
   <xacro:property name="DRIVING_JOINTB_X" value="0.063"/>
   <xacro:property name="DRIVING_JOINTB_Y" value="0.013"/>
@@ -77,10 +75,9 @@
   <xacro:property name="L_DRIVEN_POS_X" value="${L_DRIVING_POS_X + DRIVING_JOINTB_X + math.cos(ROT)*(-DRIVEN_JOINTA_X) - math.sin(ROT)*(DRIVEN_JOINTA_Y)}"/>
   <xacro:property name="L_DRIVEN_POS_Y" value="${L_DRIVING_POS_Y + DRIVING_JOINTB_Y + math.sin(ROT)*(-DRIVEN_JOINTA_X) + math.cos(ROT)*(DRIVEN_JOINTA_Y)}"/>
-  <xacro:property name="L_DRIVEN_POS_Z" value="${L_DRIVING_POS_Z - DRIVING_Z - 0.01}"/>
   <!-- RIGHT -->
   <xacro:property name="R_DRIVEN_ROT_Z" value="${-PI/2-ROT}"/>
   <xacro:property name="R_DRIVEN_POS_X" value="${R_DRIVING_POS_X - DRIVING_JOINTB_X + math.cos(-ROT)*(-DRIVEN_JOINTA_X) - math.sin(-ROT)*(DRIVEN_JOINTA_Y)}"/>
   <xacro:property name="R_DRIVEN_POS_Y" value="${R_DRIVING_POS_Y - DRIVING_JOINTB_Y + math.sin(-ROT)*(-DRIVEN_JOINTA_X) + math.cos(-ROT)*(DRIVEN_JOINTA_Y)}"/>
-  <xacro:property name="R_DRIVEN_POS_Z" value="${R_DRIVING_POS_Z - DRIVING_Z - 0.01}"/>
+  <xacro:property name="DRIVEN_POS_Z" value="${DRIVING_POS_Z - DRIVING_Z - 0.01}"/>
   <xacro:property name="DRIVEN_JOINTB_X" value="0.013"/>
   <xacro:property name="DRIVEN_JOINTB_Y" value="0.213"/>
@@ -99,10 +96,9 @@
   <xacro:property name="L_MISUMIFT_POS_X" value="${L_DRIVEN_POS_X + math.cos(ROT)*(DRIVEN_JOINTB_X) - math.sin(ROT)*(-DRIVEN_JOINTB_Y) + MISUMIFT_JOINTA_X}"/>
   <xacro:property name="L_MISUMIFT_POS_Y" value="${L_DRIVEN_POS_Y + math.sin(ROT)*(DRIVEN_JOINTB_X) + math.cos(ROT)*(-DRIVEN_JOINTB_Y) + MISUMIFT_JOINTA_Y}"/>
-  <xacro:property name="L_MISUMIFT_POS_Z" value="${L_DRIVEN_POS_Z - MISUMIFT_Z - 0.005}"/>
   <!-- RIGHT -->
   <xacro:property name="R_MISUMIFT_ROT_Z" value="${0}"/>
   <xacro:property name="R_MISUMIFT_POS_X" value="${R_DRIVEN_POS_X + math.cos(-ROT)*(DRIVEN_JOINTB_X) - math.sin(-ROT)*(-DRIVEN_JOINTB_Y) - MISUMIFT_JOINTA_X}"/>
   <xacro:property name="R_MISUMIFT_POS_Y" value="${R_DRIVEN_POS_Y + math.sin(-ROT)*(DRIVEN_JOINTB_X) + math.cos(-ROT)*(-DRIVEN_JOINTB_Y) - MISUMIFT_JOINTA_Y}"/>
-  <xacro:property name="R_MISUMIFT_POS_Z" value="${R_DRIVEN_POS_Z - MISUMIFT_Z - 0.005}"/>
+  <xacro:property name="MISUMIFT_POS_Z" value="${DRIVEN_POS_Z - MISUMIFT_Z - 0.005}"/>
   <xacro:property name="ACTIVE_JOINT_LA_LOWER" value="-${PI}"/>
   <xacro:property name="ACTIVE_JOINT_LA_UPPER" value=" ${PI}"/>

Commit message: updated meshes with updated origins

File: spacediver_ros2_control/description/gazebo/models/spacediver.sdf.xacro (robot description, xacro)
@@ -46,5 +46,4 @@
       <pose>
         ${SHOULDER_PLATE_POS_X} ${SHOULDER_PLATE_POS_Y} ${SHOULDER_PLATE_POS_Z}
-        ${SHOULDER_PLATE_ROT_X} ${SHOULDER_PLATE_ROT_Y} ${SHOULDER_PLATE_ROT_Z}
       </pose>
       <collision name="collision">
@@ -72,5 +71,5 @@
       <pose>
         ${-SHOULDER_PLATE_POS_X} ${SHOULDER_PLATE_POS_Y} ${-SHOULDER_PLATE_POS_Z}
-        ${PI/2} ${0} ${-PI/2}
+        ${R_SHOULDER_PLATE_ROT_X} ${R_SHOULDER_PLATE_ROT_Y} ${R_SHOULDER_PLATE_ROT_Z}
       </pose>
       <collision name="collision">

File: spacediver_ros2_control/description/urdf/macros/properties.xacro (robot description, xacro)
@@ -11,11 +11,13 @@
   <xacro:property name="SHOULDER_PLATE_X" value="0.03"/>
   <xacro:property name="SHOULDER_PLATE_Y" value="0.0585"/>
+  <xacro:property name="SHOULDER_PLATE_Y_ADD" value="0.00275"/>
   <xacro:property name="SHOULDER_PLATE_Z" value="0.148"/>
-  <xacro:property name="SHOULDER_PLATE_ROT_X" value="${-PI/2}"/>
-  <xacro:property name="SHOULDER_PLATE_ROT_Y" value="0"/>
-  <xacro:property name="SHOULDER_PLATE_ROT_Z" value="${-PI/2}"/>
   <xacro:property name="SHOULDER_PLATE_POS_X" value="${BASE_X/2 + 0.0045}"/>
-  <xacro:property name="SHOULDER_PLATE_POS_Y" value="${SHOULDER_PLATE_Y/2}"/>
-  <xacro:property name="SHOULDER_PLATE_POS_Z" value="${SHOULDER_PLATE_Z/2}"/>
+  <xacro:property name="SHOULDER_PLATE_POS_Y" value="${-SHOULDER_PLATE_Y_ADD - SHOULDER_PLATE_Y/2}"/>
+  <xacro:property name="SHOULDER_PLATE_POS_Z" value="${-SHOULDER_PLATE_Z/2}"/>
+  <!-- RIGHT -->
+  <xacro:property name="R_SHOULDER_PLATE_ROT_X" value="${PI}"/>
+  <xacro:property name="R_SHOULDER_PLATE_ROT_Y" value="${0}"/>
+  <xacro:property name="R_SHOULDER_PLATE_ROT_Z" value="${PI}"/>
   <!-- DYNAMIXEL -->
   <xacro:property name="DYNAMIXEL_X" value="0.0335"/>
@@ -25,9 +27,9 @@
   <xacro:property name="DYNAMIXEL_JOINTB_Y" value="${DYNAMIXEL_Y - 0.04475}"/>
   <xacro:property name="DYNAMIXEL_TOP_POS_X" value="${SHOULDER_PLATE_POS_X + SHOULDER_PLATE_X + DYNAMIXEL_X/2}"/>
-  <xacro:property name="DYNAMIXEL_TOP_POS_Y" value="${SHOULDER_PLATE_POS_Y - SHOULDER_PLATE_Y/2}"/>
-  <xacro:property name="DYNAMIXEL_TOP_POS_Z" value="${SHOULDER_PLATE_POS_Z - DYNAMIXEL_Z/2}"/>
+  <xacro:property name="DYNAMIXEL_TOP_POS_Y" value="${SHOULDER_PLATE_POS_Y + SHOULDER_PLATE_Y_ADD + SHOULDER_PLATE_Y/2}"/>
+  <xacro:property name="DYNAMIXEL_TOP_POS_Z" value="${SHOULDER_PLATE_POS_Z + SHOULDER_PLATE_Z - DYNAMIXEL_Z/2}"/>
   <xacro:property name="DYNAMIXEL_BOT_POS_X" value="${SHOULDER_PLATE_POS_X + SHOULDER_PLATE_X + DYNAMIXEL_X/2}"/>
-  <xacro:property name="DYNAMIXEL_BOT_POS_Y" value="${SHOULDER_PLATE_POS_Y - SHOULDER_PLATE_Y/2}"/>
-  <xacro:property name="DYNAMIXEL_BOT_POS_Z" value="${SHOULDER_PLATE_POS_Z - SHOULDER_PLATE_Z + DYNAMIXEL_Z/2}"/>
+  <xacro:property name="DYNAMIXEL_BOT_POS_Y" value="${SHOULDER_PLATE_POS_Y + SHOULDER_PLATE_Y_ADD + SHOULDER_PLATE_Y/2}"/>
+  <xacro:property name="DYNAMIXEL_BOT_POS_Z" value="${SHOULDER_PLATE_POS_Z+ DYNAMIXEL_Z/2}"/>
   <!-- MIUSMI LN (LOWER LINK) -->
   <xacro:property name="MISUMILN_X" value="0.032"/>

Commit message: dynamixels have same x and y's

File: spacediver_ros2_control/description/gazebo/models/spacediver.sdf.xacro (robot description, xacro)
@@ -97,5 +97,5 @@
     <link name="left_dynamixel_top">
       <pose>
-        ${DYNAMIXEL_TOP_POS_X} ${DYNAMIXEL_TOP_POS_Y} ${DYNAMIXEL_TOP_POS_Z}
+        ${DYNAMIXEL_POS_X} ${DYNAMIXEL_POS_Y} ${DYNAMIXEL_TOP_POS_Z}
       </pose>
       <collision name="collision">
@@ -130,5 +130,5 @@
     <link name="right_dynamixel_top">
       <pose>
-        ${-DYNAMIXEL_TOP_POS_X} ${DYNAMIXEL_TOP_POS_Y} ${DYNAMIXEL_TOP_POS_Z}
+        ${-DYNAMIXEL_POS_X} ${DYNAMIXEL_POS_Y} ${DYNAMIXEL_TOP_POS_Z}
       </pose>
       <collision name="collision">
@@ -163,5 +163,5 @@
     <link name="left_dynamixel_bottom">
       <pose>
-        ${DYNAMIXEL_BOT_POS_X} ${DYNAMIXEL_BOT_POS_Y} ${DYNAMIXEL_BOT_POS_Z}
+        ${DYNAMIXEL_POS_X} ${DYNAMIXEL_POS_Y} ${DYNAMIXEL_BOT_POS_Z}
       </pose>
       <collision name="collision">
@@ -196,5 +196,5 @@
     <link name="right_dynamixel_bottom">
       <pose>
-        ${-DYNAMIXEL_BOT_POS_X} ${DYNAMIXEL_BOT_POS_Y} ${DYNAMIXEL_BOT_POS_Z}
+        ${-DYNAMIXEL_POS_X} ${DYNAMIXEL_POS_Y} ${DYNAMIXEL_BOT_POS_Z}
       </pose>
       <collision name="collision">

File: spacediver_ros2_control/description/urdf/macros/properties.xacro (robot description, xacro)
@@ -26,10 +26,8 @@
   <xacro:property name="DYNAMIXEL_JOINTB_X" value="0"/>
   <xacro:property name="DYNAMIXEL_JOINTB_Y" value="${DYNAMIXEL_Y - 0.04475}"/>
-  <xacro:property name="DYNAMIXEL_TOP_POS_X" value="${SHOULDER_PLATE_POS_X + SHOULDER_PLATE_X + DYNAMIXEL_X/2}"/>
-  <xacro:property name="DYNAMIXEL_TOP_POS_Y" value="${SHOULDER_PLATE_POS_Y + SHOULDER_PLATE_Y_ADD + SHOULDER_PLATE_Y/2}"/>
+  <xacro:property name="DYNAMIXEL_POS_X" value="${SHOULDER_PLATE_POS_X + SHOULDER_PLATE_X + DYNAMIXEL_X/2}"/>
+  <xacro:property name="DYNAMIXEL_POS_Y" value="${SHOULDER_PLATE_POS_Y + SHOULDER_PLATE_Y_ADD + SHOULDER_PLATE_Y/2}"/>
   <xacro:property name="DYNAMIXEL_TOP_POS_Z" value="${SHOULDER_PLATE_POS_Z + SHOULDER_PLATE_Z - DYNAMIXEL_Z/2}"/>
-  <xacro:property name="DYNAMIXEL_BOT_POS_X" value="${SHOULDER_PLATE_POS_X + SHOULDER_PLATE_X + DYNAMIXEL_X/2}"/>
-  <xacro:property name="DYNAMIXEL_BOT_POS_Y" value="${SHOULDER_PLATE_POS_Y + SHOULDER_PLATE_Y_ADD + SHOULDER_PLATE_Y/2}"/>
-  <xacro:property name="DYNAMIXEL_BOT_POS_Z" value="${SHOULDER_PLATE_POS_Z+ DYNAMIXEL_Z/2}"/>
+  <xacro:property name="DYNAMIXEL_BOT_POS_Z" value="${SHOULDER_PLATE_POS_Z + DYNAMIXEL_Z/2}"/>
   <!-- MIUSMI LN (LOWER LINK) -->
   <xacro:property name="MISUMILN_X" value="0.032"/>
@@ -41,10 +39,10 @@
   <!-- LEFT -->
   <xacro:property name="L_MISUMILN_ROT_Z" value="${-PI/2+ROT}"/>
-  <xacro:property name="L_MISUMILN_POS_X" value="${DYNAMIXEL_BOT_POS_X + math.cos(ROT)*(-MISUMILN_JOINTA_X) - math.sin(ROT)*(MISUMILN_JOINTA_Y)}"/>
-  <xacro:property name="L_MISUMILN_POS_Y" value="${DYNAMIXEL_BOT_POS_Y - DYNAMIXEL_JOINTB_Y + math.sin(ROT)*(-MISUMILN_JOINTA_X) + math.cos(ROT)*(MISUMILN_JOINTA_Y)}"/>
+  <xacro:property name="L_MISUMILN_POS_X" value="${DYNAMIXEL_POS_X + math.cos(ROT)*(-MISUMILN_JOINTA_X) - math.sin(ROT)*(MISUMILN_JOINTA_Y)}"/>
+  <xacro:property name="L_MISUMILN_POS_Y" value="${DYNAMIXEL_POS_Y - DYNAMIXEL_JOINTB_Y + math.sin(ROT)*(-MISUMILN_JOINTA_X) + math.cos(ROT)*(MISUMILN_JOINTA_Y)}"/>
   <!-- RIGHT -->
   <xacro:property name="R_MISUMILN_ROT_Z" value="${-PI/2-ROT}"/>
-  <xacro:property name="R_MISUMILN_POS_X" value="${-DYNAMIXEL_BOT_POS_X + math.cos(-ROT)*(-MISUMILN_JOINTA_X) - math.sin(-ROT)*(MISUMILN_JOINTA_Y)}"/>
-  <xacro:property name="R_MISUMILN_POS_Y" value="${DYNAMIXEL_BOT_POS_Y - DYNAMIXEL_JOINTB_Y + math.sin(-ROT)*(-MISUMILN_JOINTA_X) + math.cos(-ROT)*(MISUMILN_JOINTA_Y)}"/>
+  <xacro:property name="R_MISUMILN_POS_X" value="${-DYNAMIXEL_POS_X + math.cos(-ROT)*(-MISUMILN_JOINTA_X) - math.sin(-ROT)*(MISUMILN_JOINTA_Y)}"/>
+  <xacro:property name="R_MISUMILN_POS_Y" value="${DYNAMIXEL_POS_Y - DYNAMIXEL_JOINTB_Y + math.sin(-ROT)*(-MISUMILN_JOINTA_X) + math.cos(-ROT)*(MISUMILN_JOINTA_Y)}"/>
   <xacro:property name="MISUMILN_POS_Z" value="${DYNAMIXEL_BOT_POS_Z + DYNAMIXEL_Z/2 + 0.0045}"/>
   <!-- DRIVING LINK -->
@@ -57,10 +55,10 @@
   <!-- LEFT -->
   <xacro:property name="L_DRIVING_ROT_Z" value="${0}"/>
-  <xacro:property name="L_DRIVING_POS_X" value="${DYNAMIXEL_TOP_POS_X - DRIVING_JOINTA_X}"/>
-  <xacro:property name="L_DRIVING_POS_Y" value="${DYNAMIXEL_TOP_POS_Y - DYNAMIXEL_JOINTB_Y - DRIVING_JOINTA_Y}"/>
+  <xacro:property name="L_DRIVING_POS_X" value="${DYNAMIXEL_POS_X - DRIVING_JOINTA_X}"/>
+  <xacro:property name="L_DRIVING_POS_Y" value="${DYNAMIXEL_POS_Y - DYNAMIXEL_JOINTB_Y - DRIVING_JOINTA_Y}"/>
   <!-- RIGHT -->
   <xacro:property name="R_DRIVING_ROT_Z" value="${PI}"/>
-  <xacro:property name="R_DRIVING_POS_X" value="${-DYNAMIXEL_TOP_POS_X + DRIVING_JOINTA_X}"/>
-  <xacro:property name="R_DRIVING_POS_Y" value="${DYNAMIXEL_TOP_POS_Y - DYNAMIXEL_JOINTB_Y + DRIVING_JOINTA_Y}"/>
+  <xacro:property name="R_DRIVING_POS_X" value="${-DYNAMIXEL_POS_X + DRIVING_JOINTA_X}"/>
+  <xacro:property name="R_DRIVING_POS_Y" value="${DYNAMIXEL_POS_Y - DYNAMIXEL_JOINTB_Y + DRIVING_JOINTA_Y}"/>
   <xacro:property name="DRIVING_POS_Z" value="${DYNAMIXEL_TOP_POS_Z - DYNAMIXEL_Z/2 - DRIVING_Z - 0.0045}"/>
   <xacro:property name="DRIVING_JOINTB_X" value="0.063"/>
