Commit message: updated shoulder plate mesh and pos

File: spacediver_ros2_control/description/gazebo/models/spacediver.sdf.xacro (robot description, xacro)
@@ -46,4 +46,5 @@
       <pose>
         ${SHOULDER_PLATE_POS_X} ${SHOULDER_PLATE_POS_Y} ${SHOULDER_PLATE_POS_Z}
+        0 0 ${L_SHOULDER_PLATE_ROT_Z}
       </pose>
       <collision name="collision">

File: spacediver_ros2_control/description/urdf/macros/properties.xacro (robot description, xacro)
@@ -14,10 +14,12 @@
   <xacro:property name="SHOULDER_PLATE_Z" value="0.148"/>
   <xacro:property name="SHOULDER_PLATE_POS_X" value="${BASE_X/2 + 0.0045}"/>
-  <xacro:property name="SHOULDER_PLATE_POS_Y" value="${-SHOULDER_PLATE_Y_ADD - SHOULDER_PLATE_Y/2}"/>
+  <xacro:property name="SHOULDER_PLATE_POS_Y" value="${SHOULDER_PLATE_Y/2}"/>
   <xacro:property name="SHOULDER_PLATE_POS_Z" value="${-SHOULDER_PLATE_Z/2}"/>
+  <!-- LEFT -->
+  <xacro:property name="L_SHOULDER_PLATE_ROT_Z" value="${-PI/2}"/>
   <!-- RIGHT -->
   <xacro:property name="R_SHOULDER_PLATE_ROT_X" value="${PI}"/>
   <xacro:property name="R_SHOULDER_PLATE_ROT_Y" value="${0}"/>
-  <xacro:property name="R_SHOULDER_PLATE_ROT_Z" value="${PI}"/>
+  <xacro:property name="R_SHOULDER_PLATE_ROT_Z" value="${-PI/2}"/>
   <!-- DYNAMIXEL -->
   <xacro:property name="DYNAMIXEL_X" value="0.0335"/>
@@ -27,5 +29,5 @@
   <xacro:property name="DYNAMIXEL_JOINTB_Y" value="${DYNAMIXEL_Y - 0.04475}"/>
   <xacro:property name="DYNAMIXEL_POS_X" value="${SHOULDER_PLATE_POS_X + SHOULDER_PLATE_X + DYNAMIXEL_X/2}"/>
-  <xacro:property name="DYNAMIXEL_POS_Y" value="${SHOULDER_PLATE_POS_Y + SHOULDER_PLATE_Y_ADD + SHOULDER_PLATE_Y/2}"/>
+  <xacro:property name="DYNAMIXEL_POS_Y" value="${SHOULDER_PLATE_POS_Y - SHOULDER_PLATE_Y/2}"/>
   <xacro:property name="DYNAMIXEL_TOP_POS_Z" value="${SHOULDER_PLATE_POS_Z + SHOULDER_PLATE_Z - DYNAMIXEL_Z/2}"/>
   <xacro:property name="DYNAMIXEL_BOT_POS_Z" value="${SHOULDER_PLATE_POS_Z + DYNAMIXEL_Z/2}"/>

Commit message: base to shoulder plate revolute joint

File: spacediver_ros2_control/description/gazebo/models/spacediver.sdf.xacro (robot description, xacro)
@@ -441,11 +441,23 @@
     </link>
     <!-- JOINTS -->
-    <joint name="base_to_leftshoulderplate_joint" type="fixed">
+    <joint name="base_to_leftshoulderplate_joint" type="revolute">
       <parent>base_link</parent>
       <child>left_shoulder_plate</child>
-    </joint>
-    <joint name="base_to_rightshoulderplate_joint" type="fixed">
+      <pose>
+        ${SHOULDER_PLATE_JOINTA_X} ${SHOULDER_PLATE_JOINTA_Y} ${SHOULDER_PLATE_JOINTA_Z}
+      </pose>
+      <axis>
+        <xyz>0 1 0</xyz>
+      </axis>
+    </joint>
+    <joint name="base_to_rightshoulderplate_joint" type="revolute">
       <parent>base_link</parent>
       <child>right_shoulder_plate</child>
+      <pose>
+        ${SHOULDER_PLATE_JOINTA_X} ${SHOULDER_PLATE_JOINTA_Y} ${SHOULDER_PLATE_JOINTA_Z}
+      </pose>
+      <axis>
+        <xyz>0 1 0</xyz>
+      </axis>
     </joint>
     <joint name="leftshoulderplate_to_leftdynamixeltop_joint" type="fixed">

File: spacediver_ros2_control/description/urdf/macros/properties.xacro (robot description, xacro)
@@ -13,4 +13,7 @@
   <xacro:property name="SHOULDER_PLATE_Y_ADD" value="0.00275"/>
   <xacro:property name="SHOULDER_PLATE_Z" value="0.148"/>
+  <xacro:property name="SHOULDER_PLATE_JOINTA_X" value="${0.04475}"/>
+  <xacro:property name="SHOULDER_PLATE_JOINTA_Y" value="${0.005}"/>
+  <xacro:property name="SHOULDER_PLATE_JOINTA_Z" value="${SHOULDER_PLATE_Z/2}"/>
   <xacro:property name="SHOULDER_PLATE_POS_X" value="${BASE_X/2 + 0.0045}"/>
   <xacro:property name="SHOULDER_PLATE_POS_Y" value="${SHOULDER_PLATE_Y/2}"/>
@@ -38,5 +41,5 @@
   <xacro:property name="MISUMILN_JOINTA_X" value="0.016"/>
   <xacro:property name="MISUMILN_JOINTA_Y" value="0.012"/>
-  <xacro:property name="MISUMILN_JOINTA_Z" value="${0.01 + MISUMILN_Z/2}"/>
+  <xacro:property name="MISUMILN_JOINTA_Z" value="${MISUMILN_Z/2}"/>
   <!-- LEFT -->
   <xacro:property name="L_MISUMILN_ROT_Z" value="${-PI/2+ROT}"/>

Commit message: Add properties about the joint position, velocity, and effort limit for each active joint, which is a dynamixel joint.

File: spacediver_ros2_control/description/gazebo/models/spacediver.sdf.xacro (robot description, xacro)
@@ -477,4 +477,24 @@
       <child>right_dynamixel_bottom</child>
     </joint>
+    <joint name="leftdynamixeltop_to_leftdriving_joint" type="revolute">
+      <parent>left_dynamixel_top</parent>
+      <child>left_driving_link</child>
+      <pose>
+        ${DRIVING_JOINTA_X} ${DRIVING_JOINTA_Y} ${DRIVING_JOINTA_Z}
+      </pose>
+      <axis>
+        <xyz>0 0 1</xyz>
+      </axis>
+    </joint>
+    <joint name="rightdynamixeltop_to_rightdriving_joint" type="revolute">
+      <parent>right_dynamixel_top</parent>
+      <child>right_driving_link</child>
+      <pose>
+        ${DRIVING_JOINTA_X} ${DRIVING_JOINTA_Y} ${DRIVING_JOINTA_Z}
+      </pose>
+      <axis>
+        <xyz>0 0 1</xyz>
+      </axis>
+    </joint>
     <joint name="leftdynamixelbottom_to_leftmisumiln_joint" type="revolute">
       <parent>left_dynamixel_bottom</parent>
@@ -497,24 +517,4 @@
       </axis>
     </joint>
-    <joint name="leftdynamixeltop_to_leftdriving_joint" type="revolute">
-      <parent>left_dynamixel_top</parent>
-      <child>left_driving_link</child>
-      <pose>
-        ${DRIVING_JOINTA_X} ${DRIVING_JOINTA_Y} ${DRIVING_JOINTA_Z}
-      </pose>
-      <axis>
-        <xyz>0 0 1</xyz>
-      </axis>
-    </joint>
-    <joint name="rightdynamixeltop_to_rightdriving_joint" type="revolute">
-      <parent>right_dynamixel_top</parent>
-      <child>right_driving_link</child>
-      <pose>
-        ${DRIVING_JOINTA_X} ${DRIVING_JOINTA_Y} ${DRIVING_JOINTA_Z}
-      </pose>
-      <axis>
-        <xyz>0 0 1</xyz>
-      </axis>
-    </joint>
     <joint name="leftdriving_to_leftdriven_joint" type="revolute">
       <parent>left_driving_link</parent>

File: spacediver_ros2_control/description/ros2_control/spacediver_ros2_control.xacro (robot description, xacro)
@@ -12,4 +12,110 @@
       </hardware>
     </xacro:unless>
+    <!-- BASE TO LEFT SHOULDER PLATE -->
+    <joint name="base_to_leftshoulderplate_joint">
+      <command_interface name="position">
+        <param name="min">"${BASE_DYNAMIXEL_LOWER}"</param>
+        <param name="max">"${BASE_DYNAMIXEL_UPPER}"</param>
+      </command_interface>
+      <command_interface name="velocity">
+        <param name="min">"-${BASE_DYNAMIXEL_VELOCITY}"</param>
+        <param name="max">" ${BASE_DYNAMIXEL_VELOCITY}"</param>
+      </command_interface>
+      <command_interface name="effort">
+        <param name="min">"-${BASE_DYNAMIXEL_EFFORT}"</param>
+        <param name="max">" ${BASE_DYNAMIXEL_EFFORT}"</param>
+      </command_interface>
+      <state_interface name="position"/>
+      <state_interface name="velocity"/>
+      <state_interface name="effort"/>
+    </joint>
+    <!-- BASE TO RIGHT SHOULDER PLATE -->
+    <joint name="base_to_rightshoulderplate_joint">
+      <command_interface name="position">
+        <param name="min">"${BASE_DYNAMIXEL_UPPER}"</param>
+        <param name="max">"${BASE_DYNAMIXEL_LOWER}"</param>
+      </command_interface>
+      <command_interface name="velocity">
+        <param name="min">"-${BASE_DYNAMIXEL_VELOCITY}"</param>
+        <param name="max">" ${BASE_DYNAMIXEL_VELOCITY}"</param>
+      </command_interface>
+      <command_interface name="effort">
+        <param name="min">"-${BASE_DYNAMIXEL_EFFORT}"</param>
+        <param name="max">" ${BASE_DYNAMIXEL_EFFORT}"</param>
+      </command_interface>
+      <state_interface name="position"/>
+      <state_interface name="velocity"/>
+      <state_interface name="effort"/>
+    </joint>
+    <!-- TOP DYNAMIXEL TO DRIVING LINK -->
+    <joint name="leftdynamixeltop_to_leftdriving_joint">
+      <command_interface name="position">
+        <param name="min">"${TOP_DYNAMIXEL_LOWER}"</param>
+        <param name="max">"${TOP_DYNAMIXEL_UPPER}"</param>
+      </command_interface>
+      <command_interface name="velocity">
+        <param name="min">"-${TOP_DYNAMIXEL_VELOCITY}"</param>
+        <param name="max">" ${TOP_DYNAMIXEL_VELOCITY}"</param>
+      </command_interface>
+      <command_interface name="effort">
+        <param name="min">"-${TOP_DYNAMIXEL_EFFORT}"</param>
+        <param name="max">" ${TOP_DYNAMIXEL_EFFORT}"</param>
+      </command_interface>
+      <state_interface name="position"/>
+      <state_interface name="velocity"/>
+      <state_interface name="effort"/>
+    </joint>
+    <joint name="rightdynamixeltop_to_rightdriving_joint">
+      <command_interface name="position">
+        <param name="min">"${TOP_DYNAMIXEL_UPPER}"</param>
+        <param name="max">"${TOP_DYNAMIXEL_LOWER}"</param>
+      </command_interface>
+      <command_interface name="velocity">
+        <param name="min">"-${TOP_DYNAMIXEL_VELOCITY}"</param>
+        <param name="max">" ${TOP_DYNAMIXEL_VELOCITY}"</param>
+      </command_interface>
+      <command_interface name="effort">
+        <param name="min">"-${TOP_DYNAMIXEL_EFFORT}"</param>
+        <param name="max">" ${TOP_DYNAMIXEL_EFFORT}"</param>
+      </command_interface>
+      <state_interface name="position"/>
+      <state_interface name="velocity"/>
+      <state_interface name="effort"/>
+    </joint>
+    <!-- BOTTOM DYNAMIXEL TO MISUMI LN -->
+    <joint name="leftdynamixelbottom_to_leftmisumiln_joint">
+      <command_interface name="position">
+        <param name="min">"${BOT_DYNAMIXEL_LOWER}"</param>
+        <param name="max">"${BOT_DYNAMIXEL_UPPER}"</param>
+      </command_interface>
+      <command_interface name="velocity">
+        <param name="min">"-${BOT_DYNAMIXEL_VELOCITY}"</param>
+        <param name="max">" ${BOT_DYNAMIXEL_VELOCITY}"</param>
+      </command_interface>
+      <command_interface name="effort">
+        <param name="min">"-${BOT_DYNAMIXEL_EFFORT}"</param>
+        <param name="max">" ${BOT_DYNAMIXEL_EFFORT}"</param>
+      </command_interface>
+      <state_interface name="position"/>
+      <state_interface name="velocity"/>
+      <state_interface name="effort"/>
+    </joint>
+    <joint name="rightdynamixelbottom_to_rightmisumiln_joint">
+      <command_interface name="position">
+        <param name="min">"${BOT_DYNAMIXEL_UPPER}"</param>
+        <param name="max">"${BOT_DYNAMIXEL_LOWER}"</param>
+      </command_interface>
+      <command_interface name="velocity">
+        <param name="min">"-${BOT_DYNAMIXEL_VELOCITY}"</param>
+        <param name="max">" ${BOT_DYNAMIXEL_VELOCITY}"</param>
+      </command_interface>
+      <command_interface name="effort">
+        <param name="min">"-${BOT_DYNAMIXEL_EFFORT}"</param>
+        <param name="max">" ${BOT_DYNAMIXEL_EFFORT}"</param>
+      </command_interface>
+      <state_interface name="position"/>
+      <state_interface name="velocity"/>
+      <state_interface name="effort"/>
+    </joint>
     <!-- Joint 1 -->
     <joint name="active_joint_la">

File: spacediver_ros2_control/description/urdf/macros/properties.xacro (robot description, xacro)
@@ -3,4 +3,6 @@
   <xacro:property name="PI" value="${math.pi}"/>
   <xacro:property name="ROT" value="${PI/6}"/>
+  <xacro:property name="RPM" value="30"/>
+  <!-- BASE -->
   <xacro:property name="BASE_X" value="0.18"/>
   <xacro:property name="BASE_Y" value="0.0585"/>
@@ -8,4 +10,9 @@
   <xacro:property name="BASE_MASS" value="50"/>
   <xacro:property name="BASE_INERTIA_Z" value="0.13526810"/>
+  <!-- JOINT -->
+  <xacro:property name="BASE_DYNAMIXEL_LOWER" value="-${PI}"/>
+  <xacro:property name="BASE_DYNAMIXEL_UPPER" value=" ${PI}"/>
+  <xacro:property name="BASE_DYNAMIXEL_VELOCITY" value="${(RPM) * 2*(PI)/60}"/>
+  <xacro:property name="BASE_DYNAMIXEL_EFFORT" value="1"/>
   <!-- SHOULDER PLATE -->
   <xacro:property name="SHOULDER_PLATE_X" value="0.03"/>
@@ -29,10 +36,19 @@
   <xacro:property name="DYNAMIXEL_Y" value="0.0585"/>
   <xacro:property name="DYNAMIXEL_Z" value="0.044"/>
-  <xacro:property name="DYNAMIXEL_JOINTB_X" value="0"/>
-  <xacro:property name="DYNAMIXEL_JOINTB_Y" value="${DYNAMIXEL_Y - 0.04475}"/>
   <xacro:property name="DYNAMIXEL_POS_X" value="${SHOULDER_PLATE_POS_X + SHOULDER_PLATE_X + DYNAMIXEL_X/2}"/>
   <xacro:property name="DYNAMIXEL_POS_Y" value="${SHOULDER_PLATE_POS_Y - SHOULDER_PLATE_Y/2}"/>
   <xacro:property name="DYNAMIXEL_TOP_POS_Z" value="${SHOULDER_PLATE_POS_Z + SHOULDER_PLATE_Z - DYNAMIXEL_Z/2}"/>
   <xacro:property name="DYNAMIXEL_BOT_POS_Z" value="${SHOULDER_PLATE_POS_Z + DYNAMIXEL_Z/2}"/>
+  <!-- JOINT -->
+  <xacro:property name="DYNAMIXEL_JOINTB_X" value="0"/>
+  <xacro:property name="DYNAMIXEL_JOINTB_Y" value="${DYNAMIXEL_Y - 0.04475}"/>
+  <xacro:property name="TOP_DYNAMIXEL_LOWER" value="-${PI}"/>
+  <xacro:property name="TOP_DYNAMIXEL_UPPER" value=" ${PI}"/>
+  <xacro:property name="TOP_DYNAMIXEL_VELOCITY" value="${(RPM) * 2*(PI)/60}"/>
+  <xacro:property name="TOP_DYNAMIXEL_EFFORT" value="1"/>
+  <xacro:property name="BOT_DYNAMIXEL_LOWER" value="-${PI}"/>
+  <xacro:property name="BOT_DYNAMIXEL_UPPER" value=" ${PI}"/>
+  <xacro:property name="BOT_DYNAMIXEL_VELOCITY" value="${(RPM) * 2*(PI)/60}"/>
+  <xacro:property name="BOT_DYNAMIXEL_EFFORT" value="1"/>
   <!-- MIUSMI LN (LOWER LINK) -->
   <xacro:property name="MISUMILN_X" value="0.032"/>
