Commit message: Feature/create robot model sdf (#3)
Created robot model sdf

- added mesh files (.STL) for the shoulder plate and arm links
- created script to automate mesh transfer to gazebo models directory on local machine
- updated sdf file with new link structure
- added joints relative to the child links
- xacro properties file includes the variable names and values

---------

Co-authored-by: akiyoshi <uchida.akiyoshi.s3@dc.tohoku.ac.jp>

File: spacediver_ros2_control/description/gazebo/models/spacediver.sdf.xacro (robot description, xacro)
@@ -42,10 +42,66 @@
       </visual>
     </link>
-    <link name="link_1">
-      <pose>0 0 ${BASE_Z/2}</pose>
-      <collision name="collision">
-        <geometry>
-          <box>
-            <size>${LINK_1_X} ${LINK_1_Y} ${LINK_1_Z}</size>
+    <!-- SHOULDER PLATES -->
+    <link name="left_shoulder_plate">
+      <pose>
+        ${SHOULDER_PLATE_POS_X} ${SHOULDER_PLATE_POS_Y} ${SHOULDER_PLATE_POS_Z}
+        0 0 ${L_SHOULDER_PLATE_ROT_Z}
+      </pose>
+      <collision name="collision">
+        <geometry>
+          <mesh>
+            <uri>model://spacediver/meshes/shoulder_plate.STL</uri>
+          </mesh>
+        </geometry>
+      </collision>
+      <visual name="visual">
+        <geometry>
+          <mesh>
+            <uri>model://spacediver/meshes/shoulder_plate.STL</uri>
+          </mesh>
+        </geometry>
+        <!-- <material>
+          <script>
+            <uri>file://media/materials/scripts/gazebo.material</uri>
+            <name>Gazebo/Grey</name>
+          </script>
+        </material> -->
+      </visual>
+    </link>
+    <link name="right_shoulder_plate">
+      <pose>
+        ${-SHOULDER_PLATE_POS_X} ${SHOULDER_PLATE_POS_Y} ${-SHOULDER_PLATE_POS_Z}
+        ${R_SHOULDER_PLATE_ROT_X} ${R_SHOULDER_PLATE_ROT_Y} ${R_SHOULDER_PLATE_ROT_Z}
+      </pose>
+      <collision name="collision">
+        <geometry>
+          <mesh>
+            <uri>model://spacediver/meshes/shoulder_plate.STL</uri>
+          </mesh>
+        </geometry>
+      </collision>
+      <visual name="visual">
+        <geometry>
+          <mesh>
+            <uri>model://spacediver/meshes/shoulder_plate.STL</uri>
+          </mesh>
+        </geometry>
+        <!-- <material>
+          <script>
+            <uri>file://media/materials/scripts/gazebo.material</uri>
+            <name>Gazebo/Grey</name>
+          </script>
+        </material> -->
+      </visual>
+    </link>
+    <!-- DYNAMIXELS -->
+    <link name="left_dynamixel_top">
+      <pose>
+        ${DYNAMIXEL_POS_X} ${DYNAMIXEL_POS_Y} ${DYNAMIXEL_TOP_POS_Z}
+      </pose>
+      <collision name="collision">
+        <geometry>
+          <box>
+            <size>${DYNAMIXEL_X} ${DYNAMIXEL_Y} ${DYNAMIXEL_Z}</size>
           </box>
         </geometry>
@@ -62,21 +118,23 @@
         <geometry>
           <box>
-            <size>${LINK_1_X} ${LINK_1_Y} ${LINK_1_Z}</size>
-          </box>
-        </geometry>
-        <material>
-          <script>
-            <uri>file://media/materials/scripts/gazebo.material</uri>
-            <name>Gazebo/Red</name>
-          </script>
-        </material>
-      </visual>
-    </link>
-    <link name="link_2">
-      <pose>0 0 ${BASE_Z/2+LINK_1_X}</pose>
-      <collision name="collision">
-        <geometry>
-          <box>
-            <size>${LINK_2_X} ${LINK_2_Y} ${LINK_2_Z}</size>
+            <size>${DYNAMIXEL_X} ${DYNAMIXEL_Y} ${DYNAMIXEL_Z}</size>
+          </box>
+        </geometry>
+        <material>
+          <script>
+            <uri>file://media/materials/scripts/gazebo.material</uri>
+            <name>Gazebo/Blue</name>
+          </script>
+        </material>
+      </visual>
+    </link>
+    <link name="right_dynamixel_top">
+      <pose>
+        ${-DYNAMIXEL_POS_X} ${DYNAMIXEL_POS_Y} ${DYNAMIXEL_TOP_POS_Z}
+      </pose>
+      <collision name="collision">
+        <geometry>
+          <box>
+            <size>${DYNAMIXEL_X} ${DYNAMIXEL_Y} ${DYNAMIXEL_Z}</size>
           </box>
         </geometry>
@@ -93,21 +151,23 @@
         <geometry>
           <box>
-            <size>${LINK_2_X} ${LINK_2_Y} ${LINK_2_Z}</size>
-          </box>
-        </geometry>
-        <material>
-          <script>
-            <uri>file://media/materials/scripts/gazebo.material</uri>
-            <name>Gazebo/Red</name>
-          </script>
-        </material>
-      </visual>
-    </link>
-    <link name="link_3">
-      <pose>0 0 ${BASE_Z/2+LINK_1_X+LINK_2_X}</pose>
-      <collision name="collision">
-        <geometry>
-          <box>
-            <size>${LINK_3_X} ${LINK_3_Y} ${LINK_3_Z}</size>
+            <size>${DYNAMIXEL_X} ${DYNAMIXEL_Y} ${DYNAMIXEL_Z}</size>
+          </box>
+        </geometry>
+        <material>
+          <script>
+            <uri>file://media/materials/scripts/gazebo.material</uri>
+            <name>Gazebo/Blue</name>
+          </script>
+        </material>
+      </visual>
+    </link>
+    <link name="left_dynamixel_bottom">
+      <pose>
+        ${DYNAMIXEL_POS_X} ${DYNAMIXEL_POS_Y} ${DYNAMIXEL_BOT_POS_Z}
+      </pose>
+      <collision name="collision">
+        <geometry>
+          <box>
+            <size>${DYNAMIXEL_X} ${DYNAMIXEL_Y} ${DYNAMIXEL_Z}</size>
           </box>
         </geometry>
@@ -124,6 +184,66 @@
         <geometry>
           <box>
-            <size>${LINK_3_X} ${LINK_3_Y} ${LINK_3_Z}</size>
-          </box>
+            <size>${DYNAMIXEL_X} ${DYNAMIXEL_Y} ${DYNAMIXEL_Z}</size>
+          </box>
+        </geometry>
+        <material>
+          <script>
+            <uri>file://media/materials/scripts/gazebo.material</uri>
+            <name>Gazebo/Blue</name>
+          </script>
+        </material>
+      </visual>
+    </link>
+    <link name="right_dynamixel_bottom">
+      <pose>
+        ${-DYNAMIXEL_POS_X} ${DYNAMIXEL_POS_Y} ${DYNAMIXEL_BOT_POS_Z}
+      </pose>
+      <collision name="collision">
+        <geometry>
+          <box>
+            <size>${DYNAMIXEL_X} ${DYNAMIXEL_Y} ${DYNAMIXEL_Z}</size>
+          </box>
+        </geometry>
+        <surface>
+          <friction>
+            <ode>
+              <mu>100</mu>
+              <mu2>50</mu2>
+            </ode>
+          </friction>
+        </surface>
+      </collision>
+      <visual name="visual">
+        <geometry>
+          <box>
+            <size>${DYNAMIXEL_X} ${DYNAMIXEL_Y} ${DYNAMIXEL_Z}</size>
+          </box>
+        </geometry>
+        <material>
+          <script>
+            <uri>file://media/materials/scripts/gazebo.material</uri>
+            <name>Gazebo/Blue</name>
+          </script>
+        </material>
+      </visual>
+    </link>
+    <!-- MISUMI LN (lower link) -->
+    <link name="left_misumi_ln">
+      <pose>
+        ${L_MISUMILN_POS_X} ${L_MISUMILN_POS_Y} ${MISUMILN_POS_Z}
+        0 0 ${L_MISUMILN_ROT_Z}
+      </pose>
+      <collision name="collision">
+        <geometry>
+          <mesh>
+            <uri>model://spacediver/meshes/Link_MISUMI_LNMS16-10-200.STL</uri>
+          </mesh>
+        </geometry>
+      </collision>
+      <visual name="visual">
+        <geometry>
+          <mesh>
+            <uri>model://spacediver/meshes/Link_MISUMI_LNMS16-10-200.STL</uri>
+          </mesh>
         </geometry>
         <material>
@@ -135,42 +255,325 @@
       </visual>
     </link>
-    <joint name="active_joint_la" type="revolute">
+    <link name="right_misumi_ln">
+      <pose>
+        ${R_MISUMILN_POS_X} ${R_MISUMILN_POS_Y} ${MISUMILN_POS_Z}
+        0 0 ${R_MISUMILN_ROT_Z}
+      </pose>
+      <collision name="collision">
+        <geometry>
+          <mesh>
+            <uri>model://spacediver/meshes/Link_MISUMI_LNMS16-10-200.STL</uri>
+          </mesh>
+        </geometry>
+      </collision>
+      <visual name="visual">
+        <geometry>
+          <mesh>
+            <uri>model://spacediver/meshes/Link_MISUMI_LNMS16-10-200.STL</uri>
+          </mesh>
+        </geometry>
+        <material>
+          <script>
+            <uri>file://media/materials/scripts/gazebo.material</uri>
+            <name>Gazebo/Red</name>
+          </script>
+        </material>
+      </visual>
+    </link>
+    <!-- DRIVING LINK -->
+    <link name="left_driving_link">
+      <pose>
+        ${L_DRIVING_POS_X} ${L_DRIVING_POS_Y} ${DRIVING_POS_Z}
+        0 0 ${L_DRIVING_ROT_Z}
+      </pose>
+      <collision name="collision">
+        <geometry>
+          <mesh>
+            <uri>model://spacediver/meshes/upper_arm_driving_link.STL</uri>
+          </mesh>
+        </geometry>
+      </collision>
+      <visual name="visual">
+        <geometry>
+          <mesh>
+            <uri>model://spacediver/meshes/upper_arm_driving_link.STL</uri>
+          </mesh>
+        </geometry>
+        <material>
+          <script>
+            <uri>file://media/materials/scripts/gazebo.material</uri>
+            <name>Gazebo/Green</name>
+          </script>
+        </material>
+      </visual>
+    </link>
+    <link name="right_driving_link">
+      <pose>
+        ${R_DRIVING_POS_X} ${R_DRIVING_POS_Y} ${DRIVING_POS_Z}
+        0 0 ${R_DRIVING_ROT_Z}
+      </pose>
+      <collision name="collision">
+        <geometry>
+          <mesh>
+            <uri>model://spacediver/meshes/upper_arm_driving_link.STL</uri>
+          </mesh>
+        </geometry>
+      </collision>
+      <visual name="visual">
+        <geometry>
+          <mesh>
+            <uri>model://spacediver/meshes/upper_arm_driving_link.STL</uri>
+          </mesh>
+        </geometry>
+        <material>
+          <script>
+            <uri>file://media/materials/scripts/gazebo.material</uri>
+            <name>Gazebo/Green</name>
+          </script>
+        </material>
+      </visual>
+    </link>
+    <!-- DRIVEN LINK -->
+    <link name="left_driven_link">
+      <pose>
+        ${L_DRIVEN_POS_X} ${L_DRIVEN_POS_Y} ${DRIVEN_POS_Z}
+        0 0 ${L_DRIVEN_ROT_Z}
+      </pose>
+      <collision name="collision">
+        <geometry>
+          <mesh>
+            <uri>model://spacediver/meshes/upper_arm_driven_link.STL</uri>
+          </mesh>
+        </geometry>
+      </collision>
+      <visual name="visual">
+        <geometry>
+          <mesh>
+            <uri>model://spacediver/meshes/upper_arm_driven_link.STL</uri>
+          </mesh>
+        </geometry>
+        <material>
+          <script>
+            <uri>file://media/materials/scripts/gazebo.material</uri>
+            <name>Gazebo/Red</name>
+          </script>
+        </material>
+      </visual>
+    </link>
+    <link name="right_driven_link">
+      <pose>
+        ${R_DRIVEN_POS_X} ${R_DRIVEN_POS_Y} ${DRIVEN_POS_Z}
+        0 0 ${R_DRIVEN_ROT_Z}
+      </pose>
+      <collision name="collision">
+        <geometry>
+          <mesh>
+            <uri>model://spacediver/meshes/upper_arm_driven_link.STL</uri>
+          </mesh>
+        </geometry>
+      </collision>
+      <visual name="visual">
+        <geometry>
+          <mesh>
+            <uri>model://spacediver/meshes/upper_arm_driven_link.STL</uri>
+          </mesh>
+        </geometry>
+        <material>
+          <script>
+            <uri>file://media/materials/scripts/gazebo.material</uri>
+            <name>Gazebo/Red</name>
+          </script>
+        </material>
+      </visual>
+    </link>
+    <!-- MISUMI FT (final link) -->
+    <link name="left_misumi_ft">
+      <pose>
+        ${L_MISUMIFT_POS_X} ${L_MISUMIFT_POS_Y} ${MISUMIFT_POS_Z}
+        0 0 ${L_MISUMIFT_ROT_Z}
+      </pose>
+      <collision name="collision">
+        <geometry>
+          <mesh>
+            <uri>model://spacediver/meshes/Misumi_LNFTS10-P10-V10-L200-S50-W18-T9.STL</uri>
+          </mesh>
+        </geometry>
+      </collision>
+      <visual name="visual">
+        <geometry>
+          <mesh>
+            <uri>model://spacediver/meshes/Misumi_LNFTS10-P10-V10-L200-S50-W18-T9.STL</uri>
+          </mesh>
+        </geometry>
+        <material>
+          <script>
+            <uri>file://media/materials/scripts/gazebo.material</uri>
+            <name>Gazebo/Green</name>
+          </script>
+        </material>
+      </visual>
+    </link>
+    <link name="right_misumi_ft">
+      <pose>
+        ${R_MISUMIFT_POS_X} ${R_MISUMIFT_POS_Y} ${MISUMIFT_POS_Z}
+        0 0 ${R_MISUMIFT_ROT_Z}
+      </pose>
+      <collision name="collision">
+        <geometry>
+          <mesh>
+            <uri>model://spacediver/meshes/Misumi_LNFTS10-P10-V10-L200-S50-W18-T9.STL</uri>
+          </mesh>
+        </geometry>
+      </collision>
+      <visual name="visual">
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
File: spacediver_ros2_control/description/urdf/macros/properties.xacro (robot description, xacro)
@@ -1,10 +1,109 @@
 <?xml version="1.0"?>
 <robot xmlns:xacro="http://ros.org/wiki/xacro">
-  <xacro:property name="PI" value="3.1415926535"/>
-  <xacro:property name="BASE_X" value="0.5"/>
-  <xacro:property name="BASE_Y" value="0.5"/>
-  <xacro:property name="BASE_Z" value="0.5"/>
+  <xacro:property name="PI" value="${math.pi}"/>
+  <xacro:property name="ROT" value="${PI/6}"/>
+  <xacro:property name="BASE_X" value="0.18"/>
+  <xacro:property name="BASE_Y" value="0.0585"/>
+  <xacro:property name="BASE_Z" value="0.0415"/>
   <xacro:property name="BASE_MASS" value="50"/>
   <xacro:property name="BASE_INERTIA_Z" value="0.13526810"/>
+  <!-- SHOULDER PLATE -->
+  <xacro:property name="SHOULDER_PLATE_X" value="0.03"/>
+  <xacro:property name="SHOULDER_PLATE_Y" value="0.0585"/>
+  <xacro:property name="SHOULDER_PLATE_Y_ADD" value="0.00275"/>
+  <xacro:property name="SHOULDER_PLATE_Z" value="0.148"/>
+  <xacro:property name="SHOULDER_PLATE_JOINTA_X" value="${0.04475}"/>
+  <xacro:property name="SHOULDER_PLATE_JOINTA_Y" value="${0.005}"/>
+  <xacro:property name="SHOULDER_PLATE_JOINTA_Z" value="${SHOULDER_PLATE_Z/2}"/>
+  <xacro:property name="SHOULDER_PLATE_POS_X" value="${BASE_X/2 + 0.0045}"/>
+  <xacro:property name="SHOULDER_PLATE_POS_Y" value="${SHOULDER_PLATE_Y/2}"/>
+  <xacro:property name="SHOULDER_PLATE_POS_Z" value="${-SHOULDER_PLATE_Z/2}"/>
+  <!-- LEFT -->
+  <xacro:property name="L_SHOULDER_PLATE_ROT_Z" value="${-PI/2}"/>
+  <!-- RIGHT -->
+  <xacro:property name="R_SHOULDER_PLATE_ROT_X" value="${PI}"/>
+  <xacro:property name="R_SHOULDER_PLATE_ROT_Y" value="${0}"/>
+  <xacro:property name="R_SHOULDER_PLATE_ROT_Z" value="${-PI/2}"/>
+  <!-- DYNAMIXEL -->
+  <xacro:property name="DYNAMIXEL_X" value="0.0335"/>
+  <xacro:property name="DYNAMIXEL_Y" value="0.0585"/>
+  <xacro:property name="DYNAMIXEL_Z" value="0.044"/>
+  <xacro:property name="DYNAMIXEL_JOINTB_X" value="0"/>
+  <xacro:property name="DYNAMIXEL_JOINTB_Y" value="${DYNAMIXEL_Y - 0.04475}"/>
+  <xacro:property name="DYNAMIXEL_POS_X" value="${SHOULDER_PLATE_POS_X + SHOULDER_PLATE_X + DYNAMIXEL_X/2}"/>
+  <xacro:property name="DYNAMIXEL_POS_Y" value="${SHOULDER_PLATE_POS_Y - SHOULDER_PLATE_Y/2}"/>
+  <xacro:property name="DYNAMIXEL_TOP_POS_Z" value="${SHOULDER_PLATE_POS_Z + SHOULDER_PLATE_Z - DYNAMIXEL_Z/2}"/>
+  <xacro:property name="DYNAMIXEL_BOT_POS_Z" value="${SHOULDER_PLATE_POS_Z + DYNAMIXEL_Z/2}"/>
+  <!-- MIUSMI LN (LOWER LINK) -->
+  <xacro:property name="MISUMILN_X" value="0.032"/>
+  <xacro:property name="MISUMILN_Y" value="0.225"/>
+  <xacro:property name="MISUMILN_Z" value="0.009"/>
+  <xacro:property name="MISUMILN_JOINTA_X" value="0.016"/>
+  <xacro:property name="MISUMILN_JOINTA_Y" value="0.012"/>
+  <xacro:property name="MISUMILN_JOINTA_Z" value="${MISUMILN_Z/2}"/>
+  <!-- LEFT -->
+  <xacro:property name="L_MISUMILN_ROT_Z" value="${-PI/2+ROT}"/>
+  <xacro:property name="L_MISUMILN_POS_X" value="${DYNAMIXEL_POS_X + math.cos(ROT)*(-MISUMILN_JOINTA_X) - math.sin(ROT)*(MISUMILN_JOINTA_Y)}"/>
+  <xacro:property name="L_MISUMILN_POS_Y" value="${DYNAMIXEL_POS_Y - DYNAMIXEL_JOINTB_Y + math.sin(ROT)*(-MISUMILN_JOINTA_X) + math.cos(ROT)*(MISUMILN_JOINTA_Y)}"/>
+  <!-- RIGHT -->
+  <xacro:property name="R_MISUMILN_ROT_Z" value="${-PI/2-ROT}"/>
+  <xacro:property name="R_MISUMILN_POS_X" value="${-DYNAMIXEL_POS_X + math.cos(-ROT)*(-MISUMILN_JOINTA_X) - math.sin(-ROT)*(MISUMILN_JOINTA_Y)}"/>
+  <xacro:property name="R_MISUMILN_POS_Y" value="${DYNAMIXEL_POS_Y - DYNAMIXEL_JOINTB_Y + math.sin(-ROT)*(-MISUMILN_JOINTA_X) + math.cos(-ROT)*(MISUMILN_JOINTA_Y)}"/>
+  <xacro:property name="MISUMILN_POS_Z" value="${DYNAMIXEL_BOT_POS_Z + DYNAMIXEL_Z/2 + 0.0145}"/>
+  <!-- DRIVING LINK -->
+  <xacro:property name="DRIVING_X" value="0.076"/>
+  <xacro:property name="DRIVING_Y" value="0.026"/>
+  <xacro:property name="DRIVING_Z" value="0.004"/>
+  <xacro:property name="DRIVING_JOINTA_X" value="0.013"/>
+  <xacro:property name="DRIVING_JOINTA_Y" value="0.013"/>
+  <xacro:property name="DRIVING_JOINTA_Z" value="${DRIVING_Z/2}"/>
+  <!-- LEFT -->
+  <xacro:property name="L_DRIVING_ROT_Z" value="${0}"/>
+  <xacro:property name="L_DRIVING_POS_X" value="${DYNAMIXEL_POS_X - DRIVING_JOINTA_X}"/>
+  <xacro:property name="L_DRIVING_POS_Y" value="${DYNAMIXEL_POS_Y - DYNAMIXEL_JOINTB_Y - DRIVING_JOINTA_Y}"/>
+  <!-- RIGHT -->
+  <xacro:property name="R_DRIVING_ROT_Z" value="${PI}"/>
+  <xacro:property name="R_DRIVING_POS_X" value="${-DYNAMIXEL_POS_X + DRIVING_JOINTA_X}"/>
+  <xacro:property name="R_DRIVING_POS_Y" value="${DYNAMIXEL_POS_Y - DYNAMIXEL_JOINTB_Y + DRIVING_JOINTA_Y}"/>
+  <xacro:property name="DRIVING_POS_Z" value="${DYNAMIXEL_TOP_POS_Z - DYNAMIXEL_Z/2 - DRIVING_Z - 0.0045}"/>
+  <xacro:property name="DRIVING_JOINTB_X" value="0.063"/>
+  <xacro:property name="DRIVING_JOINTB_Y" value="0.013"/>
+  <!-- DRIVEN LINK -->
+  <xacro:property name="DRIVEN_X" value="0.026"/>
+  <xacro:property name="DRIVEN_Y" value="0.226"/>
+  <xacro:property name="DRIVEN_Z" value="0.004"/>
+  <xacro:property name="DRIVEN_JOINTA_X" value="0.013"/>
+  <xacro:property name="DRIVEN_JOINTA_Y" value="0.013"/>
+  <xacro:property name="DRIVEN_JOINTA_Z" value="${DRIVEN_Z/2}"/>
+  <!-- LEFT -->
+  <xacro:property name="L_DRIVEN_ROT_Z" value="${-PI/2+ROT}"/>
+  <xacro:property name="L_DRIVEN_POS_X" value="${L_DRIVING_POS_X + DRIVING_JOINTB_X + math.cos(ROT)*(-DRIVEN_JOINTA_X) - math.sin(ROT)*(DRIVEN_JOINTA_Y)}"/>
+  <xacro:property name="L_DRIVEN_POS_Y" value="${L_DRIVING_POS_Y + DRIVING_JOINTB_Y + math.sin(ROT)*(-DRIVEN_JOINTA_X) + math.cos(ROT)*(DRIVEN_JOINTA_Y)}"/>
+  <!-- RIGHT -->
+  <xacro:property name="R_DRIVEN_ROT_Z" value="${-PI/2-ROT}"/>
+  <xacro:property name="R_DRIVEN_POS_X" value="${R_DRIVING_POS_X - DRIVING_JOINTB_X + math.cos(-ROT)*(-DRIVEN_JOINTA_X) - math.sin(-ROT)*(DRIVEN_JOINTA_Y)}"/>
+  <xacro:property name="R_DRIVEN_POS_Y" value="${R_DRIVING_POS_Y - DRIVING_JOINTB_Y + math.sin(-ROT)*(-DRIVEN_JOINTA_X) + math.cos(-ROT)*(DRIVEN_JOINTA_Y)}"/>
+  <xacro:property name="DRIVEN_POS_Z" value="${DRIVING_POS_Z - DRIVING_Z - 0.01}"/>
+  <xacro:property name="DRIVEN_JOINTB_X" value="0.013"/>
+  <xacro:property name="DRIVEN_JOINTB_Y" value="0.213"/>
+  <!-- MISUMI FT (final link) -->
+  <xacro:property name="MISUMIFT_X" value="0.268"/>
+  <xacro:property name="MISUMIFT_Y" value="0.018"/>
+  <xacro:property name="MISUMIFT_Z" value="0.009"/>
+  <xacro:property name="MISUMIFT_JOINTA_X" value="0.009"/>
+  <xacro:property name="MISUMIFT_JOINTA_Y" value="0.009"/>
+  <xacro:property name="MISUMIFT_JOINTA_Z" value="${MISUMIFT_Z/2}"/>
+  <xacro:property name="MISUMIFT_JOINTB_X" value="0.059"/>
+  <xacro:property name="MISUMIFT_JOINTB_Y" value="0.009"/>
+  <xacro:property name="MISUMIFT_JOINTB_Z" value="${MISUMIFT_Z/2}"/>
+  <!-- LEFT -->
+  <xacro:property name="L_MISUMIFT_ROT_Z" value="${PI}"/>
+  <xacro:property name="L_MISUMIFT_POS_X" value="${L_DRIVEN_POS_X + math.cos(ROT)*(DRIVEN_JOINTB_X) - math.sin(ROT)*(-DRIVEN_JOINTB_Y) + MISUMIFT_JOINTA_X}"/>
+  <xacro:property name="L_MISUMIFT_POS_Y" value="${L_DRIVEN_POS_Y + math.sin(ROT)*(DRIVEN_JOINTB_X) + math.cos(ROT)*(-DRIVEN_JOINTB_Y) + MISUMIFT_JOINTA_Y}"/>
+  <!-- RIGHT -->
+  <xacro:property name="R_MISUMIFT_ROT_Z" value="${0}"/>
+  <xacro:property name="R_MISUMIFT_POS_X" value="${R_DRIVEN_POS_X + math.cos(-ROT)*(DRIVEN_JOINTB_X) - math.sin(-ROT)*(-DRIVEN_JOINTB_Y) - MISUMIFT_JOINTA_X}"/>
+  <xacro:property name="R_MISUMIFT_POS_Y" value="${R_DRIVEN_POS_Y + math.sin(-ROT)*(DRIVEN_JOINTB_X) + math.cos(-ROT)*(-DRIVEN_JOINTB_Y) - MISUMIFT_JOINTA_Y}"/>
+  <xacro:property name="MISUMIFT_POS_Z" value="${DRIVEN_POS_Z - MISUMIFT_Z - 0.005}"/>
   <xacro:property name="ACTIVE_JOINT_LA_LOWER" value="-${PI}"/>
   <xacro:property name="ACTIVE_JOINT_LA_UPPER" value=" ${PI}"/>
