Commit message: removed "plate" from shoulders' link and joint names

File: spacediver_ros2_control/description/gazebo/models/spacediver.sdf.xacro (robot description, xacro)
@@ -43,5 +43,5 @@
     </link>
     <!-- SHOULDER PLATES -->
-    <link name="left_shoulder_plate">
+    <link name="left_shoulder_link">
       <pose>
         ${SHOULDER_PLATE_POS_X} ${SHOULDER_PLATE_POS_Y} ${SHOULDER_PLATE_POS_Z}
@@ -69,5 +69,5 @@
       </visual>
     </link>
-    <link name="right_shoulder_plate">
+    <link name="right_shoulder_link">
       <pose>
         ${-SHOULDER_PLATE_POS_X} ${SHOULDER_PLATE_POS_Y} ${-SHOULDER_PLATE_POS_Z}
@@ -441,7 +441,7 @@
     </link>
     <!-- JOINTS -->
-    <joint name="base_to_leftshoulderplate_joint" type="revolute">
+    <joint name="base_to_leftshoulder_joint" type="revolute">
       <parent>base_link</parent>
-      <child>left_shoulder_plate</child>
+      <child>left_shoulder_link</child>
       <pose>
         ${SHOULDER_PLATE_JOINTA_X} ${SHOULDER_PLATE_JOINTA_Y} ${SHOULDER_PLATE_JOINTA_Z}
@@ -451,7 +451,7 @@
       </axis>
     </joint>
-    <joint name="base_to_rightshoulderplate_joint" type="revolute">
+    <joint name="base_to_rightshoulder_joint" type="revolute">
       <parent>base_link</parent>
-      <child>right_shoulder_plate</child>
+      <child>right_shoulder_link</child>
       <pose>
         ${SHOULDER_PLATE_JOINTA_X} ${SHOULDER_PLATE_JOINTA_Y} ${SHOULDER_PLATE_JOINTA_Z}
@@ -461,18 +461,18 @@
       </axis>
     </joint>
-    <joint name="leftshoulderplate_to_leftdynamixeltop_joint" type="fixed">
-      <parent>left_shoulder_plate</parent>
+    <joint name="leftshoulder_to_leftdynamixeltop_joint" type="fixed">
+      <parent>left_shoulder_link</parent>
       <child>left_dynamixel_top</child>
     </joint>
-    <joint name="rightshoulderplate_to_rightdynamixeltop_joint" type="fixed">
-      <parent>right_shoulder_plate</parent>
+    <joint name="rightshoulder_to_rightdynamixeltop_joint" type="fixed">
+      <parent>right_shoulder_link</parent>
       <child>right_dynamixel_top</child>
     </joint>
-    <joint name="leftshoulderplate_to_leftdynamixelbottom_joint" type="fixed">
-      <parent>left_shoulder_plate</parent>
+    <joint name="leftshoulder_to_leftdynamixelbottom_joint" type="fixed">
+      <parent>left_shoulder_link</parent>
       <child>left_dynamixel_bottom</child>
     </joint>
-    <joint name="rightshoulderplate_to_rightdynamixelbottom_joint" type="fixed">
-      <parent>right_shoulder_plate</parent>
+    <joint name="rightshoulder_to_rightdynamixelbottom_joint" type="fixed">
+      <parent>right_shoulder_link</parent>
       <child>right_dynamixel_bottom</child>
     </joint>

File: spacediver_ros2_control/description/ros2_control/spacediver_ros2_control.xacro (robot description, xacro)
@@ -13,5 +13,5 @@
     </xacro:unless>
     <!-- BASE TO LEFT SHOULDER PLATE -->
-    <joint name="base_to_leftshoulderplate_joint">
+    <joint name="base_to_leftshoulder_joint">
       <command_interface name="position">
         <param name="min">"${BASE_DYNAMIXEL_LOWER}"</param>
@@ -31,5 +31,5 @@
     </joint>
     <!-- BASE TO RIGHT SHOULDER PLATE -->
-    <joint name="base_to_rightshoulderplate_joint">
+    <joint name="base_to_rightshoulder_joint">
       <command_interface name="position">
         <param name="min">"${BASE_DYNAMIXEL_UPPER}"</param>

Commit message: removed "plate" from shoulder properties

File: spacediver_ros2_control/description/gazebo/models/spacediver.sdf.xacro (robot description, xacro)
@@ -45,6 +45,6 @@
     <link name="left_shoulder_link">
       <pose>
-        ${SHOULDER_PLATE_POS_X} ${SHOULDER_PLATE_POS_Y} ${SHOULDER_PLATE_POS_Z}
-        0 0 ${L_SHOULDER_PLATE_ROT_Z}
+        ${SHOULDER_POS_X} ${SHOULDER_POS_Y} ${SHOULDER_POS_Z}
+        0 0 ${L_SHOULDER_ROT_Z}
       </pose>
       <collision name="collision">
@@ -71,6 +71,6 @@
     <link name="right_shoulder_link">
       <pose>
-        ${-SHOULDER_PLATE_POS_X} ${SHOULDER_PLATE_POS_Y} ${-SHOULDER_PLATE_POS_Z}
-        ${R_SHOULDER_PLATE_ROT_X} ${R_SHOULDER_PLATE_ROT_Y} ${R_SHOULDER_PLATE_ROT_Z}
+        ${-SHOULDER_POS_X} ${SHOULDER_POS_Y} ${-SHOULDER_POS_Z}
+        ${R_SHOULDER_ROT_X} ${R_SHOULDER_ROT_Y} ${R_SHOULDER_ROT_Z}
       </pose>
       <collision name="collision">
@@ -445,5 +445,5 @@
       <child>left_shoulder_link</child>
       <pose>
-        ${SHOULDER_PLATE_JOINTA_X} ${SHOULDER_PLATE_JOINTA_Y} ${SHOULDER_PLATE_JOINTA_Z}
+        ${SHOULDER_JOINTA_X} ${SHOULDER_JOINTA_Y} ${SHOULDER_JOINTA_Z}
       </pose>
       <axis>
@@ -455,5 +455,5 @@
       <child>right_shoulder_link</child>
       <pose>
-        ${SHOULDER_PLATE_JOINTA_X} ${SHOULDER_PLATE_JOINTA_Y} ${SHOULDER_PLATE_JOINTA_Z}
+        ${SHOULDER_JOINTA_X} ${SHOULDER_JOINTA_Y} ${SHOULDER_JOINTA_Z}
       </pose>
       <axis>

File: spacediver_ros2_control/description/urdf/macros/properties.xacro (robot description, xacro)
@@ -16,28 +16,28 @@
   <xacro:property name="BASE_DYNAMIXEL_EFFORT" value="1"/>
   <!-- SHOULDER PLATE -->
-  <xacro:property name="SHOULDER_PLATE_X" value="0.03"/>
-  <xacro:property name="SHOULDER_PLATE_Y" value="0.0585"/>
-  <xacro:property name="SHOULDER_PLATE_Y_ADD" value="0.00275"/>
-  <xacro:property name="SHOULDER_PLATE_Z" value="0.148"/>
-  <xacro:property name="SHOULDER_PLATE_JOINTA_X" value="${0.04475}"/>
-  <xacro:property name="SHOULDER_PLATE_JOINTA_Y" value="${0.005}"/>
-  <xacro:property name="SHOULDER_PLATE_JOINTA_Z" value="${SHOULDER_PLATE_Z/2}"/>
-  <xacro:property name="SHOULDER_PLATE_POS_X" value="${BASE_X/2 + 0.0045}"/>
-  <xacro:property name="SHOULDER_PLATE_POS_Y" value="${SHOULDER_PLATE_Y/2}"/>
-  <xacro:property name="SHOULDER_PLATE_POS_Z" value="${-SHOULDER_PLATE_Z/2}"/>
+  <xacro:property name="SHOULDER_X" value="0.03"/>
+  <xacro:property name="SHOULDER_Y" value="0.0585"/>
+  <xacro:property name="SHOULDER_Y_ADD" value="0.00275"/>
+  <xacro:property name="SHOULDER_Z" value="0.148"/>
+  <xacro:property name="SHOULDER_JOINTA_X" value="${0.04475}"/>
+  <xacro:property name="SHOULDER_JOINTA_Y" value="${0.005}"/>
+  <xacro:property name="SHOULDER_JOINTA_Z" value="${SHOULDER_Z/2}"/>
+  <xacro:property name="SHOULDER_POS_X" value="${BASE_X/2 + 0.0045}"/>
+  <xacro:property name="SHOULDER_POS_Y" value="${SHOULDER_Y/2}"/>
+  <xacro:property name="SHOULDER_POS_Z" value="${-SHOULDER_Z/2}"/>
   <!-- LEFT -->
-  <xacro:property name="L_SHOULDER_PLATE_ROT_Z" value="${-PI/2}"/>
+  <xacro:property name="L_SHOULDER_ROT_Z" value="${-PI/2}"/>
   <!-- RIGHT -->
-  <xacro:property name="R_SHOULDER_PLATE_ROT_X" value="${PI}"/>
-  <xacro:property name="R_SHOULDER_PLATE_ROT_Y" value="${0}"/>
-  <xacro:property name="R_SHOULDER_PLATE_ROT_Z" value="${-PI/2}"/>
+  <xacro:property name="R_SHOULDER_ROT_X" value="${PI}"/>
+  <xacro:property name="R_SHOULDER_ROT_Y" value="${0}"/>
+  <xacro:property name="R_SHOULDER_ROT_Z" value="${-PI/2}"/>
   <!-- DYNAMIXEL -->
   <xacro:property name="DYNAMIXEL_X" value="0.0335"/>
   <xacro:property name="DYNAMIXEL_Y" value="0.0585"/>
   <xacro:property name="DYNAMIXEL_Z" value="0.044"/>
-  <xacro:property name="DYNAMIXEL_POS_X" value="${SHOULDER_PLATE_POS_X + SHOULDER_PLATE_X + DYNAMIXEL_X/2}"/>
-  <xacro:property name="DYNAMIXEL_POS_Y" value="${SHOULDER_PLATE_POS_Y - SHOULDER_PLATE_Y/2}"/>
-  <xacro:property name="DYNAMIXEL_TOP_POS_Z" value="${SHOULDER_PLATE_POS_Z + SHOULDER_PLATE_Z - DYNAMIXEL_Z/2}"/>
-  <xacro:property name="DYNAMIXEL_BOT_POS_Z" value="${SHOULDER_PLATE_POS_Z + DYNAMIXEL_Z/2}"/>
+  <xacro:property name="DYNAMIXEL_POS_X" value="${SHOULDER_POS_X + SHOULDER_X + DYNAMIXEL_X/2}"/>
+  <xacro:property name="DYNAMIXEL_POS_Y" value="${SHOULDER_POS_Y - SHOULDER_Y/2}"/>
+  <xacro:property name="DYNAMIXEL_TOP_POS_Z" value="${SHOULDER_POS_Z + SHOULDER_Z - DYNAMIXEL_Z/2}"/>
+  <xacro:property name="DYNAMIXEL_BOT_POS_Z" value="${SHOULDER_POS_Z + DYNAMIXEL_Z/2}"/>
   <!-- JOINT -->
   <xacro:property name="DYNAMIXEL_JOINTB_X" value="0"/>
