Commit message: Feature/hardware interface single arm (#9)
- Added joints to spacediver_ros2_control
- Created URDF
- Created dynamixel hardware pkg
- Added dynamixel hardware interface and joint IDs to spacediver_ros2_control
- Created launch files for gazebo, rviz, hardware

File: spacediver_ros2_control/description/gazebo/models/spacediver.sdf.xacro (robot description, xacro)
@@ -43,8 +43,8 @@
     </link>
     <!-- SHOULDER PLATES -->
-    <link name="left_shoulder_plate">
-      <pose>
-        ${SHOULDER_PLATE_POS_X} ${SHOULDER_PLATE_POS_Y} ${SHOULDER_PLATE_POS_Z}
-        0 0 ${L_SHOULDER_PLATE_ROT_Z}
+    <link name="left_shoulder_link">
+      <pose>
+        ${SHOULDER_POS_X} ${SHOULDER_POS_Y} ${SHOULDER_POS_Z}
+        0 0 ${L_SHOULDER_ROT_Z}
       </pose>
       <collision name="collision">
@@ -69,8 +69,8 @@
       </visual>
     </link>
-    <link name="right_shoulder_plate">
-      <pose>
-        ${-SHOULDER_PLATE_POS_X} ${SHOULDER_PLATE_POS_Y} ${-SHOULDER_PLATE_POS_Z}
-        ${R_SHOULDER_PLATE_ROT_X} ${R_SHOULDER_PLATE_ROT_Y} ${R_SHOULDER_PLATE_ROT_Z}
+    <link name="right_shoulder_link">
+      <pose>
+        ${-SHOULDER_POS_X} ${SHOULDER_POS_Y} ${-SHOULDER_POS_Z}
+        ${R_SHOULDER_ROT_X} ${R_SHOULDER_ROT_Y} ${R_SHOULDER_ROT_Z}
       </pose>
       <collision name="collision">
@@ -441,9 +441,9 @@
     </link>
     <!-- JOINTS -->
-    <joint name="base_to_leftshoulderplate_joint" type="revolute">
+    <joint name="base_to_leftshoulder_joint" type="revolute">
       <parent>base_link</parent>
-      <child>left_shoulder_plate</child>
-      <pose>
-        ${SHOULDER_PLATE_JOINTA_X} ${SHOULDER_PLATE_JOINTA_Y} ${SHOULDER_PLATE_JOINTA_Z}
+      <child>left_shoulder_link</child>
+      <pose>
+        ${SHOULDER_JOINTA_X} ${SHOULDER_JOINTA_Y} ${SHOULDER_JOINTA_Z}
       </pose>
       <axis>
@@ -451,9 +451,9 @@
       </axis>
     </joint>
-    <joint name="base_to_rightshoulderplate_joint" type="revolute">
+    <joint name="base_to_rightshoulder_joint" type="revolute">
       <parent>base_link</parent>
-      <child>right_shoulder_plate</child>
-      <pose>
-        ${SHOULDER_PLATE_JOINTA_X} ${SHOULDER_PLATE_JOINTA_Y} ${SHOULDER_PLATE_JOINTA_Z}
+      <child>right_shoulder_link</child>
+      <pose>
+        ${SHOULDER_JOINTA_X} ${SHOULDER_JOINTA_Y} ${SHOULDER_JOINTA_Z}
       </pose>
       <axis>
@@ -461,19 +461,39 @@
       </axis>
     </joint>
-    <joint name="leftshoulderplate_to_leftdynamixeltop_joint" type="fixed">
-      <parent>left_shoulder_plate</parent>
+    <joint name="leftshoulder_to_leftdynamixeltop_joint" type="fixed">
+      <parent>left_shoulder_link</parent>
       <child>left_dynamixel_top</child>
     </joint>
-    <joint name="rightshoulderplate_to_rightdynamixeltop_joint" type="fixed">
-      <parent>right_shoulder_plate</parent>
+    <joint name="rightshoulder_to_rightdynamixeltop_joint" type="fixed">
+      <parent>right_shoulder_link</parent>
       <child>right_dynamixel_top</child>
     </joint>
-    <joint name="leftshoulderplate_to_leftdynamixelbottom_joint" type="fixed">
-      <parent>left_shoulder_plate</parent>
+    <joint name="leftshoulder_to_leftdynamixelbottom_joint" type="fixed">
+      <parent>left_shoulder_link</parent>
       <child>left_dynamixel_bottom</child>
     </joint>
-    <joint name="rightshoulderplate_to_rightdynamixelbottom_joint" type="fixed">
-      <parent>right_shoulder_plate</parent>
+    <joint name="rightshoulder_to_rightdynamixelbottom_joint" type="fixed">
+      <parent>right_shoulder_link</parent>
       <child>right_dynamixel_bottom</child>
+    </joint>
+    <joint name="leftdynamixeltop_to_leftdriving_joint" type="revolute">
+      <parent>left_dynamixel_top</parent>
+      <child>left_driving_link</child>
+      <pose>
+        ${DRIVING_JOINTA_X} ${DRIVING_JOINTA_Y} ${DRIVING_JOINTA_Z}
+      </pose>
+      <axis>
+        <xyz>0 0 1</xyz>
+      </axis>
+    </joint>
+    <joint name="rightdynamixeltop_to_rightdriving_joint" type="revolute">
+      <parent>right_dynamixel_top</parent>
+      <child>right_driving_link</child>
+      <pose>
+        ${DRIVING_JOINTA_X} ${DRIVING_JOINTA_Y} ${DRIVING_JOINTA_Z}
+      </pose>
+      <axis>
+        <xyz>0 0 1</xyz>
+      </axis>
     </joint>
     <joint name="leftdynamixelbottom_to_leftmisumiln_joint" type="revolute">
@@ -497,24 +517,4 @@
       </axis>
     </joint>
-    <joint name="leftdynamixeltop_to_leftdriving_joint" type="revolute">
-      <parent>left_dynamixel_top</parent>
-      <child>left_driving_link</child>
-      <pose>
-        ${DRIVING_JOINTA_X} ${DRIVING_JOINTA_Y} ${DRIVING_JOINTA_Z}
-      </pose>
-      <axis>
-        <xyz>0 0 1</xyz>
-      </axis>
-    </joint>
-    <joint name="rightdynamixeltop_to_rightdriving_joint" type="revolute">
-      <parent>right_dynamixel_top</parent>
-      <child>right_driving_link</child>
-      <pose>
-        ${DRIVING_JOINTA_X} ${DRIVING_JOINTA_Y} ${DRIVING_JOINTA_Z}
-      </pose>
-      <axis>
-        <xyz>0 0 1</xyz>
-      </axis>
-    </joint>
     <joint name="leftdriving_to_leftdriven_joint" type="revolute">
       <parent>left_driving_link</parent>

File: spacediver_ros2_control/description/ros2_control/spacediver_ros2_control.xacro (robot description, xacro)
@@ -9,115 +9,138 @@
     <xacro:unless value="$(arg use_gazebo)">
       <hardware>
-        <plugin>spacediver_ros2_control/SpacediverSystem</plugin>
+        <plugin>dynamixel_hardware/DynamixelHardware</plugin>
+        <param name="usb_port">/dev/ttyUSB0</param>
+        <param name="baud_rate">57600</param>
       </hardware>
     </xacro:unless>
-    <!-- Joint 1 -->
-    <joint name="active_joint_la">
+    <!-- BASE TO SHOULDER PLATE -->
+    <joint name="${BASE_TO_LEFTSHOULDER_JOINT_NAME}">
+      <param name="id">1</param>
       <command_interface name="position">
-        <param name="min">"${ACTIVE_JOINT_LA_LOWER}"</param>
-        <param name="max">"${ACTIVE_JOINT_LA_UPPER}"</param>
+        <param name="min">${BASE_DYNAMIXEL_LOWER}</param>
+        <param name="max">${BASE_DYNAMIXEL_UPPER}</param>
       </command_interface>
-      <command_interface name="velocity">
-        <param name="min">"-${ACTIVE_JOINT_LA_VELOCITY}"</param>
-        <param name="max">" ${ACTIVE_JOINT_LA_VELOCITY}"</param>
+      <xacro:if value="$(arg use_gazebo)">
+        <command_interface name="velocity">
+          <param name="min">"-${BASE_DYNAMIXEL_VELOCITY}"</param>
+          <param name="max">" ${BASE_DYNAMIXEL_VELOCITY}"</param>
+        </command_interface>
+        <command_interface name="effort">
+          <param name="min">"-${BASE_DYNAMIXEL_EFFORT}"</param>
+          <param name="max">" ${BASE_DYNAMIXEL_EFFORT}"</param>
+        </command_interface>
+      </xacro:if>
+      <state_interface name="position" />
+      <state_interface name="velocity" />
+      <xacro:if value="$(arg use_gazebo)">
+        <state_interface name="effort" />
+      </xacro:if>
+    </joint>
+    <xacro:if value="$(arg use_gazebo)">
+      <joint name="${BASE_TO_RIGHTSHOULDER_JOINT_NAME}">
+        <param name="id">4</param>
+        <command_interface name="position">
+          <param name="min">"${BASE_DYNAMIXEL_UPPER}"</param>
+          <param name="max">"${BASE_DYNAMIXEL_LOWER}"</param>
+        </command_interface>
+        <command_interface name="velocity">
+          <param name="min">"-${BASE_DYNAMIXEL_VELOCITY}"</param>
+          <param name="max">" ${BASE_DYNAMIXEL_VELOCITY}"</param>
+        </command_interface>
+        <command_interface name="effort">
+          <param name="min">"-${BASE_DYNAMIXEL_EFFORT}"</param>
+          <param name="max">" ${BASE_DYNAMIXEL_EFFORT}"</param>
+        </command_interface>
+        <state_interface name="position" />
+        <state_interface name="velocity" />
+        <state_interface name="effort" />
+      </joint>
+    </xacro:if>
+    <!-- TOP DYNAMIXEL TO DRIVING LINK -->
+    <joint name="${LEFTDYNAMIXELTOP_TO_LEFTDRIVING_JOINT_NAME}">
+      <param name="id">2</param>
+      <command_interface name="position">
+        <param name="min">${TOP_DYNAMIXEL_LOWER}</param>
+        <param name="max">${TOP_DYNAMIXEL_UPPER}</param>
       </command_interface>
-      <command_interface name="effort">
-        <param name="min">"-${ACTIVE_JOINT_LA_EFFORT}"</param>
-        <param name="max">" ${ACTIVE_JOINT_LA_EFFORT}"</param>
+      <xacro:if value="$(arg use_gazebo)">
+        <command_interface name="velocity">
+          <param name="min">"-${BASE_DYNAMIXEL_VELOCITY}"</param>
+          <param name="max">" ${BASE_DYNAMIXEL_VELOCITY}"</param>
+        </command_interface>
+        <command_interface name="effort">
+          <param name="min">"-${BASE_DYNAMIXEL_EFFORT}"</param>
+          <param name="max">" ${BASE_DYNAMIXEL_EFFORT}"</param>
+        </command_interface>
+      </xacro:if>
+      <state_interface name="position" />
+      <state_interface name="velocity" />
+      <xacro:if value="$(arg use_gazebo)">
+        <state_interface name="effort" />
+      </xacro:if>
+    </joint>
+    <xacro:if value="$(arg use_gazebo)">
+      <joint name="${RIGHTDYNAMIXELTOP_TO_RIGHTDRIVING_JOINT_NAME}">
+        <param name="id">5</param>
+        <command_interface name="position">
+          <param name="min">"${TOP_DYNAMIXEL_UPPER}"</param>
+          <param name="max">"${TOP_DYNAMIXEL_LOWER}"</param>
+        </command_interface>
+        <command_interface name="velocity">
+          <param name="min">"-${TOP_DYNAMIXEL_VELOCITY}"</param>
+          <param name="max">" ${TOP_DYNAMIXEL_VELOCITY}"</param>
+        </command_interface>
+        <command_interface name="effort">
+          <param name="min">"-${TOP_DYNAMIXEL_EFFORT}"</param>
+          <param name="max">" ${TOP_DYNAMIXEL_EFFORT}"</param>
+        </command_interface>
+        <state_interface name="position" />
+        <state_interface name="velocity" />
+        <state_interface name="effort" />
+      </joint>
+    </xacro:if>
+    <!-- BOTTOM DYNAMIXEL TO MISUMI LN -->
+    <joint name="${LEFT_DYNAMIXELBOT_TO_LEFTMISUMILN_JOINT_NAME}">
+      <param name="id">3</param>
+      <command_interface name="position">
+        <param name="min">${BOT_DYNAMIXEL_LOWER}</param>
+        <param name="max">${BOT_DYNAMIXEL_UPPER}</param>
       </command_interface>
-      <state_interface name="position"/>
-      <state_interface name="velocity"/>
-      <state_interface name="effort"/>
+      <xacro:if value="$(arg use_gazebo)">
+        <command_interface name="velocity">
+          <param name="min">"-${BOT_DYNAMIXEL_VELOCITY}"</param>
+          <param name="max">" ${BOT_DYNAMIXEL_VELOCITY}"</param>
+        </command_interface>
+        <command_interface name="effort">
+          <param name="min">"-${BOT_DYNAMIXEL_EFFORT}"</param>
+          <param name="max">" ${BOT_DYNAMIXEL_EFFORT}"</param>
+        </command_interface>
+      </xacro:if>
+      <state_interface name="position" />
+      <state_interface name="velocity" />
+      <xacro:if value="$(arg use_gazebo)">
+        <state_interface name="effort" />
+      </xacro:if>
     </joint>
-    <!-- Joint 2 -->
-    <joint name="active_joint_lb">
-      <command_interface name="position">
-        <param name="min">"${ACTIVE_JOINT_LB_LOWER}"</param>
-        <param name="max">"${ACTIVE_JOINT_LB_UPPER}"</param>
-      </command_interface>
-      <command_interface name="velocity">
-        <param name="min">"-${ACTIVE_JOINT_LB_VELOCITY}"</param>
-        <param name="max">" ${ACTIVE_JOINT_LB_VELOCITY}"</param>
-      </command_interface>
-      <command_interface name="effort">
-        <param name="min">"-${ACTIVE_JOINT_LB_EFFORT}"</param>
-        <param name="max">" ${ACTIVE_JOINT_LB_EFFORT}"</param>
-      </command_interface>
-      <state_interface name="position"/>
-      <state_interface name="velocity"/>
-      <state_interface name="effort"/>
-    </joint>
-    <!-- Joint 3 -->
-    <joint name="active_joint_lc">
-      <command_interface name="position">
-        <param name="min">"${ACTIVE_JOINT_LC_LOWER}"</param>
-        <param name="max">"${ACTIVE_JOINT_LC_UPPER}"</param>
-      </command_interface>
-      <command_interface name="velocity">
-        <param name="min">"-${ACTIVE_JOINT_LC_VELOCITY}"</param>
-        <param name="max">" ${ACTIVE_JOINT_LC_VELOCITY}"</param>
-      </command_interface>
-      <command_interface name="effort">
-        <param name="min">"-${ACTIVE_JOINT_LC_EFFORT}"</param>
-        <param name="max">" ${ACTIVE_JOINT_LC_EFFORT}"</param>
-      </command_interface>
-      <state_interface name="position"/>
-      <state_interface name="velocity"/>
-      <state_interface name="effort"/>
-    </joint>
-    <!-- Joint 4 -->
-    <joint name="active_joint_ra">
-      <command_interface name="position">
-        <param name="min">"-${ACTIVE_JOINT_RA_UPPER}"</param>
-        <param name="max">"-${ACTIVE_JOINT_RA_LOWER}"</param>
-      </command_interface>
-      <command_interface name="velocity">
-        <param name="min">"-${ACTIVE_JOINT_RA_VELOCITY}"</param>
-        <param name="max">" ${ACTIVE_JOINT_RA_VELOCITY}"</param>
-      </command_interface>
-      <command_interface name="effort">
-        <param name="min">"-${ACTIVE_JOINT_RA_EFFORT}"</param>
-        <param name="max">" ${ACTIVE_JOINT_RA_EFFORT}"</param>
-      </command_interface>
-      <state_interface name="position"/>
-      <state_interface name="velocity"/>
-      <state_interface name="effort"/>
-    </joint>
-    <!-- Joint 5 -->
-    <joint name="active_joint_rb">
-      <command_interface name="position">
-        <param name="min">"-${ACTIVE_JOINT_RB_UPPER}"</param>
-        <param name="max">"-${ACTIVE_JOINT_RB_LOWER}"</param>
-      </command_interface>
-      <command_interface name="velocity">
-        <param name="min">"-${ACTIVE_JOINT_RB_VELOCITY}"</param>
-        <param name="max">" ${ACTIVE_JOINT_RB_VELOCITY}"</param>
-      </command_interface>
-      <command_interface name="effort">
-        <param name="min">"-${ACTIVE_JOINT_RB_EFFORT}"</param>
-        <param name="max">" ${ACTIVE_JOINT_RB_EFFORT}"</param>
-      </command_interface>
-      <state_interface name="position"/>
-      <state_interface name="velocity"/>
-      <state_interface name="effort"/>
-    </joint>
-    <!-- Joint 6 -->
-    <joint name="active_joint_rc">
-      <command_interface name="position">
-        <param name="min">"-${ACTIVE_JOINT_RC_UPPER}"</param>
-        <param name="max">"-${ACTIVE_JOINT_RC_LOWER}"</param>
-      </command_interface>
-      <command_interface name="velocity">
-        <param name="min">"-${ACTIVE_JOINT_RC_VELOCITY}"</param>
-        <param name="max">" ${ACTIVE_JOINT_RC_VELOCITY}"</param>
-      </command_interface>
-      <command_interface name="effort">
-        <param name="min">"-${ACTIVE_JOINT_RC_EFFORT}"</param>
-        <param name="max">" ${ACTIVE_JOINT_RC_EFFORT}"</param>
-      </command_interface>
-      <state_interface name="position"/>
-      <state_interface name="velocity"/>
-      <state_interface name="effort"/>
-    </joint>
+    <xacro:if value="$(arg use_gazebo)">
+      <joint name="${RIGHT_DYNAMIXELBOT_TO_RIGHTMISUMILN_JOINT_NAME}">
+        <param name="id">6</param>
+        <command_interface name="position">
+          <param name="min">"${BOT_DYNAMIXEL_UPPER}"</param>
+          <param name="max">"${BOT_DYNAMIXEL_LOWER}"</param>
+        </command_interface>
+        <command_interface name="velocity">
+          <param name="min">"-${BOT_DYNAMIXEL_VELOCITY}"</param>
+          <param name="max">" ${BOT_DYNAMIXEL_VELOCITY}"</param>
+        </command_interface>
+        <command_interface name="effort">
+          <param name="min">"-${BOT_DYNAMIXEL_EFFORT}"</param>
+          <param name="max">" ${BOT_DYNAMIXEL_EFFORT}"</param>
+        </command_interface>
+        <state_interface name="position" />
+        <state_interface name="velocity" />
+        <state_interface name="effort" />
+      </joint>
+    </xacro:if>
   </ros2_control>
 </robot>
