Commit message: Feature/hardware interface single arm (#9)
- Added joints to spacediver_ros2_control
- Created URDF
- Created dynamixel hardware pkg
- Added dynamixel hardware interface and joint IDs to spacediver_ros2_control
- Created launch files for gazebo, rviz, hardware

File: spacediver_ros2_control/description/urdf/macros/properties.xacro (robot description, xacro)
@@ -3,4 +3,39 @@
   <xacro:property name="PI" value="${math.pi}"/>
   <xacro:property name="ROT" value="${PI/6}"/>
+  <xacro:property name="RPM" value="30"/>
+  <!-- LINK NAMES -->
+  <xacro:property name="BASE_LINK_NAME" value="base_link"/>
+  <xacro:property name="L_SHOULDER_LINK_NAME" value="left_shoulder_link"/>
+  <xacro:property name="R_SHOULDER_LINK_NAME" value="right_shoulder_link"/>
+  <xacro:property name="L_TOP_DYNAMIXEL_LINK_NAME" value="left_dynamixel_top"/>
+  <xacro:property name="R_TOP_DYNAMIXEL_LINK_NAME" value="right_dynamixel_top"/>
+  <xacro:property name="L_BOT_DYNAMIXEL_LINK_NAME" value="left_dynamixel_bottom"/>
+  <xacro:property name="R_BOT_DYNAMIXEL_LINK_NAME" value="right_dynamixel_bottom"/>
+  <xacro:property name="L_MISUMILN_LINK_NAME" value="left_misumi_ln"/>
+  <xacro:property name="R_MISUMILN_LINK_NAME" value="right_misumi_ln"/>
+  <xacro:property name="L_DRIVING_LINK_NAME" value="left_driving_link"/>
+  <xacro:property name="R_DRIVING_LINK_NAME" value="right_driving_link"/>
+  <xacro:property name="L_DRIVEN_LINK_NAME" value="left_driven_link"/>
+  <xacro:property name="R_DRIVEN_LINK_NAME" value="right_driven_link"/>
+  <xacro:property name="L_MISUMIFT_LINK_NAME" value="left_misumi_ft"/>
+  <xacro:property name="R_MISUMIFT_LINK_NAME" value="right_misumi_ft"/>
+  <!-- JOINT NAMES -->
+  <xacro:property name="BASE_TO_LEFTSHOULDER_JOINT_NAME" value="base_to_leftshoulder_joint"/>
+  <xacro:property name="BASE_TO_RIGHTSHOULDER_JOINT_NAME" value="base_to_rightshoulder_joint"/>
+  <xacro:property name="LEFTSHOULDER_TO_LEFTDYNAMIXELTOP_JOINT_NAME" value="leftshoulder_to_leftdynamixeltop_joint"/>
+  <xacro:property name="RIGHTSHOULDER_TO_RIGHTDYNAMIXELTOP_JOINT_NAME" value="rightshoulder_to_rightdynamixeltop_joint"/>
+  <xacro:property name="LEFTSHOULDER_TO_LEFTDYNAMIXELBOT_JOINT_NAME" value="leftshoulder_to_leftdynamixelbottom_joint"/>
+  <xacro:property name="RIGHTSHOULDER_TO_RIGHTDYNAMIXELBOT_JOINT_NAME" value="rightshoulder_to_rightdynamixelbottom_joint"/>
+  <xacro:property name="LEFT_DYNAMIXELBOT_TO_LEFTMISUMILN_JOINT_NAME" value="leftdynamixelbottom_to_leftmisumiln_joint"/>
+  <xacro:property name="RIGHT_DYNAMIXELBOT_TO_RIGHTMISUMILN_JOINT_NAME" value="rightdynamixelbottom_to_rightmisumiln_joint"/>
+  <xacro:property name="LEFTDYNAMIXELTOP_TO_LEFTDRIVING_JOINT_NAME" value="leftdynamixeltop_to_leftdriving_joint"/>
+  <xacro:property name="RIGHTDYNAMIXELTOP_TO_RIGHTDRIVING_JOINT_NAME" value="rightdynamixeltop_to_rightdriving_joint"/>
+  <xacro:property name="LEFTDRIVING_TO_LEFTDRIVEN_JOINT_NAME" value="leftdriving_to_leftdriven_joint"/>
+  <xacro:property name="RIGHTDRIVING_TO_RIGHTDRIVEN_JOINT_NAME" value="rightdriving_to_rightdriven_joint"/>
+  <xacro:property name="LEFTDRIVEN_TO_LEFTMISUMIFT_JOINT_NAME" value="leftdriven_to_leftmisumift_joint"/>
+  <xacro:property name="RIGHTDRIVEN_TO_RIGHTMISUMIFT_JOINT_NAME" value="rightdriven_to_rightmisumift_joint"/>
+  <xacro:property name="LEFTMISUMILN_TO_LEFTMISUMIFT_JOINT_NAME" value="leftmisumiln_to_leftmisumift_joint"/>
+  <xacro:property name="RIGHTMISUMILN_TO_RIGHTMISUMIFT_JOINT_NAME" value="rightmisumiln_to_rightmisumift_joint"/>
+  <!-- BASE -->
   <xacro:property name="BASE_X" value="0.18"/>
   <xacro:property name="BASE_Y" value="0.0585"/>
@@ -8,4 +43,116 @@
   <xacro:property name="BASE_MASS" value="50"/>
   <xacro:property name="BASE_INERTIA_Z" value="0.13526810"/>
+  <!-- JOINT -->
+  <xacro:property name="BASE_DYNAMIXEL_LOWER" value="-${PI}"/>
+  <xacro:property name="BASE_DYNAMIXEL_UPPER" value=" ${PI}"/>
+  <xacro:property name="BASE_DYNAMIXEL_VELOCITY" value="${(RPM) * 2*(PI)/60}"/>
+  <xacro:property name="BASE_DYNAMIXEL_EFFORT" value="1"/>
+  <!-- SHOULDER PLATE -->
+  <xacro:property name="SHOULDER_X" value="0.03"/>
+  <xacro:property name="SHOULDER_Y" value="0.0585"/>
+  <xacro:property name="SHOULDER_Y_ADD" value="0.00275"/>
+  <xacro:property name="SHOULDER_Z" value="0.148"/>
+  <xacro:property name="SHOULDER_JOINTA_X" value="${0.04475}"/>
+  <xacro:property name="SHOULDER_JOINTA_Y" value="${0.005}"/>
+  <xacro:property name="SHOULDER_JOINTA_Z" value="${SHOULDER_Z/2}"/>
+  <xacro:property name="SHOULDER_POS_X" value="${BASE_X/2 + 0.0045}"/>
+  <xacro:property name="SHOULDER_POS_Y" value="${SHOULDER_Y/2}"/>
+  <xacro:property name="SHOULDER_POS_Z" value="${-SHOULDER_Z/2}"/>
+  <!-- LEFT -->
+  <xacro:property name="L_SHOULDER_ROT_Z" value="${-PI/2}"/>
+  <!-- RIGHT -->
+  <xacro:property name="R_SHOULDER_ROT_X" value="${PI}"/>
+  <xacro:property name="R_SHOULDER_ROT_Y" value="${0}"/>
+  <xacro:property name="R_SHOULDER_ROT_Z" value="${-PI/2}"/>
+  <!-- DYNAMIXEL -->
+  <xacro:property name="DYNAMIXEL_X" value="0.0335"/>
+  <xacro:property name="DYNAMIXEL_Y" value="0.0585"/>
+  <xacro:property name="DYNAMIXEL_Z" value="0.044"/>
+  <xacro:property name="DYNAMIXEL_POS_X" value="${SHOULDER_POS_X + SHOULDER_X + DYNAMIXEL_X/2}"/>
+  <xacro:property name="DYNAMIXEL_POS_Y" value="${SHOULDER_POS_Y - SHOULDER_Y/2}"/>
+  <xacro:property name="DYNAMIXEL_TOP_POS_Z" value="${SHOULDER_POS_Z + SHOULDER_Z - DYNAMIXEL_Z/2}"/>
+  <xacro:property name="DYNAMIXEL_BOT_POS_Z" value="${SHOULDER_POS_Z + DYNAMIXEL_Z/2}"/>
+  <!-- JOINT -->
+  <xacro:property name="DYNAMIXEL_JOINTB_X" value="0"/>
+  <xacro:property name="DYNAMIXEL_JOINTB_Y" value="${DYNAMIXEL_Y - 0.04475}"/>
+  <xacro:property name="TOP_DYNAMIXEL_LOWER" value="-${PI}"/>
+  <xacro:property name="TOP_DYNAMIXEL_UPPER" value=" ${PI}"/>
+  <xacro:property name="TOP_DYNAMIXEL_VELOCITY" value="${(RPM) * 2*(PI)/60}"/>
+  <xacro:property name="TOP_DYNAMIXEL_EFFORT" value="1"/>
+  <xacro:property name="BOT_DYNAMIXEL_LOWER" value="-${PI}"/>
+  <xacro:property name="BOT_DYNAMIXEL_UPPER" value=" ${PI}"/>
+  <xacro:property name="BOT_DYNAMIXEL_VELOCITY" value="${(RPM) * 2*(PI)/60}"/>
+  <xacro:property name="BOT_DYNAMIXEL_EFFORT" value="1"/>
+  <!-- MIUSMI LN (LOWER LINK) -->
+  <xacro:property name="MISUMILN_X" value="0.032"/>
+  <xacro:property name="MISUMILN_Y" value="0.225"/>
+  <xacro:property name="MISUMILN_Z" value="0.009"/>
+  <xacro:property name="MISUMILN_JOINTA_X" value="0.016"/>
+  <xacro:property name="MISUMILN_JOINTA_Y" value="0.012"/>
+  <xacro:property name="MISUMILN_JOINTA_Z" value="${MISUMILN_Z/2}"/>
+  <!-- LEFT -->
+  <xacro:property name="L_MISUMILN_ROT_Z" value="${-PI/2+ROT}"/>
+  <xacro:property name="L_MISUMILN_POS_X" value="${DYNAMIXEL_POS_X + math.cos(ROT)*(-MISUMILN_JOINTA_X) - math.sin(ROT)*(MISUMILN_JOINTA_Y)}"/>
+  <xacro:property name="L_MISUMILN_POS_Y" value="${DYNAMIXEL_POS_Y - DYNAMIXEL_JOINTB_Y + math.sin(ROT)*(-MISUMILN_JOINTA_X) + math.cos(ROT)*(MISUMILN_JOINTA_Y)}"/>
+  <!-- RIGHT -->
+  <xacro:property name="R_MISUMILN_ROT_Z" value="${-PI/2-ROT}"/>
+  <xacro:property name="R_MISUMILN_POS_X" value="${-DYNAMIXEL_POS_X + math.cos(-ROT)*(-MISUMILN_JOINTA_X) - math.sin(-ROT)*(MISUMILN_JOINTA_Y)}"/>
+  <xacro:property name="R_MISUMILN_POS_Y" value="${DYNAMIXEL_POS_Y - DYNAMIXEL_JOINTB_Y + math.sin(-ROT)*(-MISUMILN_JOINTA_X) + math.cos(-ROT)*(MISUMILN_JOINTA_Y)}"/>
+  <xacro:property name="MISUMILN_POS_Z" value="${DYNAMIXEL_BOT_POS_Z + DYNAMIXEL_Z/2 + 0.0145}"/>
+  <!-- DRIVING LINK -->
+  <xacro:property name="DRIVING_X" value="0.076"/>
+  <xacro:property name="DRIVING_Y" value="0.026"/>
+  <xacro:property name="DRIVING_Z" value="0.004"/>
+  <xacro:property name="DRIVING_JOINTA_X" value="0.013"/>
+  <xacro:property name="DRIVING_JOINTA_Y" value="0.013"/>
+  <xacro:property name="DRIVING_JOINTA_Z" value="${DRIVING_Z/2}"/>
+  <!-- LEFT -->
+  <xacro:property name="L_DRIVING_ROT_Z" value="${0}"/>
+  <xacro:property name="L_DRIVING_POS_X" value="${DYNAMIXEL_POS_X - DRIVING_JOINTA_X}"/>
+  <xacro:property name="L_DRIVING_POS_Y" value="${DYNAMIXEL_POS_Y - DYNAMIXEL_JOINTB_Y - DRIVING_JOINTA_Y}"/>
+  <!-- RIGHT -->
+  <xacro:property name="R_DRIVING_ROT_Z" value="${PI}"/>
+  <xacro:property name="R_DRIVING_POS_X" value="${-DYNAMIXEL_POS_X + DRIVING_JOINTA_X}"/>
+  <xacro:property name="R_DRIVING_POS_Y" value="${DYNAMIXEL_POS_Y - DYNAMIXEL_JOINTB_Y + DRIVING_JOINTA_Y}"/>
+  <xacro:property name="DRIVING_POS_Z" value="${DYNAMIXEL_TOP_POS_Z - DYNAMIXEL_Z/2 - DRIVING_Z - 0.0045}"/>
+  <xacro:property name="DRIVING_JOINTB_X" value="0.063"/>
+  <xacro:property name="DRIVING_JOINTB_Y" value="0.013"/>
+  <!-- DRIVEN LINK -->
+  <xacro:property name="DRIVEN_X" value="0.026"/>
+  <xacro:property name="DRIVEN_Y" value="0.226"/>
+  <xacro:property name="DRIVEN_Z" value="0.004"/>
+  <xacro:property name="DRIVEN_JOINTA_X" value="0.013"/>
+  <xacro:property name="DRIVEN_JOINTA_Y" value="0.013"/>
+  <xacro:property name="DRIVEN_JOINTA_Z" value="${DRIVEN_Z/2}"/>
+  <!-- LEFT -->
+  <xacro:property name="L_DRIVEN_ROT_Z" value="${-PI/2+ROT}"/>
+  <xacro:property name="L_DRIVEN_POS_X" value="${L_DRIVING_POS_X + DRIVING_JOINTB_X + math.cos(ROT)*(-DRIVEN_JOINTA_X) - math.sin(ROT)*(DRIVEN_JOINTA_Y)}"/>
+  <xacro:property name="L_DRIVEN_POS_Y" value="${L_DRIVING_POS_Y + DRIVING_JOINTB_Y + math.sin(ROT)*(-DRIVEN_JOINTA_X) + math.cos(ROT)*(DRIVEN_JOINTA_Y)}"/>
+  <!-- RIGHT -->
+  <xacro:property name="R_DRIVEN_ROT_Z" value="${-PI/2-ROT}"/>
+  <xacro:property name="R_DRIVEN_POS_X" value="${R_DRIVING_POS_X - DRIVING_JOINTB_X + math.cos(-ROT)*(-DRIVEN_JOINTA_X) - math.sin(-ROT)*(DRIVEN_JOINTA_Y)}"/>
+  <xacro:property name="R_DRIVEN_POS_Y" value="${R_DRIVING_POS_Y - DRIVING_JOINTB_Y + math.sin(-ROT)*(-DRIVEN_JOINTA_X) + math.cos(-ROT)*(DRIVEN_JOINTA_Y)}"/>
+  <xacro:property name="DRIVEN_POS_Z" value="${DRIVING_POS_Z - DRIVING_Z - 0.01}"/>
+  <xacro:property name="DRIVEN_JOINTB_X" value="0.013"/>
+  <xacro:property name="DRIVEN_JOINTB_Y" value="0.213"/>
+  <!-- MISUMI FT (final link) -->
+  <xacro:property name="MISUMIFT_X" value="0.268"/>
+  <xacro:property name="MISUMIFT_Y" value="0.018"/>
+  <xacro:property name="MISUMIFT_Z" value="0.009"/>
+  <xacro:property name="MISUMIFT_JOINTA_X" value="0.009"/>
+  <xacro:property name="MISUMIFT_JOINTA_Y" value="0.009"/>
+  <xacro:property name="MISUMIFT_JOINTA_Z" value="${MISUMIFT_Z/2}"/>
+  <xacro:property name="MISUMIFT_JOINTB_X" value="0.059"/>
+  <xacro:property name="MISUMIFT_JOINTB_Y" value="0.009"/>
+  <xacro:property name="MISUMIFT_JOINTB_Z" value="${MISUMIFT_Z/2}"/>
+  <!-- LEFT -->
+  <xacro:property name="L_MISUMIFT_ROT_Z" value="${PI}"/>
+  <xacro:property name="L_MISUMIFT_POS_X" value="${L_DRIVEN_POS_X + math.cos(ROT)*(DRIVEN_JOINTB_X) - math.sin(ROT)*(-DRIVEN_JOINTB_Y) + MISUMIFT_JOINTA_X}"/>
+  <xacro:property name="L_MISUMIFT_POS_Y" value="${L_DRIVEN_POS_Y + math.sin(ROT)*(DRIVEN_JOINTB_X) + math.cos(ROT)*(-DRIVEN_JOINTB_Y) + MISUMIFT_JOINTA_Y}"/>
+  <!-- RIGHT -->
+  <xacro:property name="R_MISUMIFT_ROT_Z" value="${0}"/>
+  <xacro:property name="R_MISUMIFT_POS_X" value="${R_DRIVEN_POS_X + math.cos(-ROT)*(DRIVEN_JOINTB_X) - math.sin(-ROT)*(-DRIVEN_JOINTB_Y) - MISUMIFT_JOINTA_X}"/>
+  <xacro:property name="R_MISUMIFT_POS_Y" value="${R_DRIVEN_POS_Y + math.sin(-ROT)*(DRIVEN_JOINTB_X) + math.cos(-ROT)*(-DRIVEN_JOINTB_Y) - MISUMIFT_JOINTA_Y}"/>
+  <xacro:property name="MISUMIFT_POS_Z" value="${DRIVEN_POS_Z - MISUMIFT_Z - 0.005}"/>
   <!-- SHOULDER PLATE -->
   <xacro:property name="SHOULDER_PLATE_X" value="0.03"/>

File: spacediver_ros2_control/description/urdf/parts/spacediver_base.xacro (robot description, xacro)
@@ -2,5 +2,5 @@
 <!-- import xacro reffering here https://gbiggs.github.io/rosjp_urdf_tutorial_text/manipulator_urdf.html -->
 <robot xmlns:xacro="http://ros.org/wiki/xacro">
-  <link name="base_link">
+  <link name="${BASE_LINK_NAME}">
     <visual>
       <origin xyz="0 0 0" rpy="0 0 0"/>
@@ -8,5 +8,5 @@
         <box size="${BASE_X} ${BASE_Y} ${BASE_Z}"/>
       </geometry>
-      <material name="white"/>
+      <material name="black"/>
     </visual>
     <collision>
@@ -16,7 +16,9 @@
       </geometry>
     </collision>
-    <xacro:inertial_box mass="${BASE_MASS}" x="${BASE_X/2}" y="${BASE_Y/2}" z="${BASE_Z/2}">
-      <origin xyz="0 0 0" rpy="0 0 0"/>
-    </xacro:inertial_box>
+    <xacro:if value="$(arg use_gazebo)">
+      <xacro:inertial_box mass="${BASE_MASS}" x="${BASE_X/2}" y="${BASE_Y/2}" z="${BASE_Z/2}">
+        <origin xyz="0 0 0" rpy="0 0 0"/>
+      </xacro:inertial_box>
+    </xacro:if>
   </link>
 </robot>

File: spacediver_ros2_control/description/urdf/parts/spacediver_right_arm.xacro (robot description, xacro)
@@ -3,16 +3,16 @@
 https://gbiggs.github.io/rosjp_urdf_tutorial_text/manipulator_urdf.html -->
 <robot xmlns:xacro="http://ros.org/wiki/xacro">
-  <xacro:macro name="left_arm" params="base_name *origin">
+  <xacro:macro name="right_arm" params="base_name *origin">
     <!-- BASE TO SHOULDER -->
-    <joint name="${BASE_TO_LEFTSHOULDER_JOINT_NAME}" type="revolute">
+    <joint name="${BASE_TO_RIGHTSHOULDER_JOINT_NAME}" type="revolute">
       <parent link="${BASE_LINK_NAME}" />
-      <child link="${L_SHOULDER_LINK_NAME}" />
-      <origin
-        xyz="
-        ${SHOULDER_POS_X}
+      <child link="${R_SHOULDER_LINK_NAME}" />
+      <origin
+        xyz="
+        ${-SHOULDER_POS_X}
         ${-(SHOULDER_JOINTA_X-SHOULDER_Y/2)}
         ${0}
       "
-        rpy="0 0 0" />
+        rpy="0 0 ${PI}" />
       <axis xyz="1 0 0" />
       <limit lower="${BASE_DYNAMIXEL_LOWER}" upper="${BASE_DYNAMIXEL_UPPER}"
@@ -20,13 +20,13 @@
     </joint>
     <!-- SHOULDER -->
-    <link name="${L_SHOULDER_LINK_NAME}">
-      <visual>
-        <origin
-          xyz="
-          ${0}
-          ${SHOULDER_JOINTA_X}
-          ${-SHOULDER_Z/2}
-        "
-          rpy="0 0 ${L_SHOULDER_ROT_Z}" />
+    <link name="${R_SHOULDER_LINK_NAME}">
+      <visual>
+        <origin
+          xyz="
+          ${0}
+          ${-SHOULDER_JOINTA_X}
+          ${SHOULDER_Z/2}
+        "
+          rpy="${PI} 0 ${-L_SHOULDER_ROT_Z}" />
         <geometry>
           <mesh
@@ -39,8 +39,8 @@
           xyz="
           ${0}
-          ${SHOULDER_JOINTA_X}
-          ${-SHOULDER_Z/2}
-        "
-          rpy="0 0 ${L_SHOULDER_ROT_Z}" />
+          ${-SHOULDER_JOINTA_X}
+          ${SHOULDER_Z/2}
+        "
+          rpy="${PI} 0 ${-L_SHOULDER_ROT_Z}" />
         <geometry>
           <mesh
@@ -54,11 +54,11 @@
     </link>
     <!-- SHOULDER TO BOTTOM DYNAMIXEL -->
-    <joint name="${LEFTSHOULDER_TO_LEFTDYNAMIXELBOT_JOINT_NAME}" type="fixed">
-      <parent link="${L_SHOULDER_LINK_NAME}" />
-      <child link="${L_BOT_DYNAMIXEL_LINK_NAME}" />
+    <joint name="${RIGHTSHOULDER_TO_RIGHTDYNAMIXELBOT_JOINT_NAME}" type="fixed">
+      <parent link="${R_SHOULDER_LINK_NAME}" />
+      <child link="${R_BOT_DYNAMIXEL_LINK_NAME}" />
       <origin
         xyz="
         ${SHOULDER_X + DYNAMIXEL_X/2}
-        ${SHOULDER_JOINTA_X - DYNAMIXEL_Y/2}
+        ${DYNAMIXEL_Y/2 - SHOULDER_JOINTA_X}
         ${-SHOULDER_Z/2 + DYNAMIXEL_Z/2}
       "
@@ -67,5 +67,5 @@
     </joint>
     <!-- BOTTOM DYNAMIXEL -->
-    <link name="${L_BOT_DYNAMIXEL_LINK_NAME}">
+    <link name="${R_BOT_DYNAMIXEL_LINK_NAME}">
       <visual>
         <origin xyz="0 0 0" rpy="0 0 0" />
@@ -87,13 +87,13 @@
     </link>
     <!-- BOTTOM DYNAMIXEL TO MISUMI LN -->
-    <joint name="${LEFT_DYNAMIXELBOT_TO_LEFTMISUMILN_JOINT_NAME}" type="revolute">
-      <parent link="${L_BOT_DYNAMIXEL_LINK_NAME}" />
-      <child link="${L_MISUMILN_LINK_NAME}" />
+    <joint name="${RIGHT_DYNAMIXELBOT_TO_RIGHTMISUMILN_JOINT_NAME}" type="revolute">
+      <parent link="${R_BOT_DYNAMIXEL_LINK_NAME}" />
+      <child link="${R_MISUMILN_LINK_NAME}" />
       <origin
         xyz="
         ${0}
-        ${DYNAMIXEL_JOINTB_Y-DYNAMIXEL_Y/2}
+        ${DYNAMIXEL_Y/2 - DYNAMIXEL_JOINTB_Y}
         ${MISUMILN_POS_Z-DYNAMIXEL_BOT_POS_Z}"
-        rpy="0 0 ${L_MISUMILN_ROT_Z}" />
+        rpy="0 0 ${-L_MISUMILN_ROT_Z}" />
       <axis xyz="0 0 1" />
       <limit lower="${BOT_DYNAMIXEL_LOWER}" upper="${BOT_DYNAMIXEL_UPPER}"
@@ -101,9 +101,13 @@
     </joint>
     <!-- MISUMI LN -->
-    <link name="${L_MISUMILN_LINK_NAME}">
-      <visual>
-        <origin
-          xyz="${-MISUMILN_JOINTA_Y} ${-MISUMILN_JOINTA_X} 0"
-          rpy="0 0 0" />
+    <link name="${R_MISUMILN_LINK_NAME}">
+      <visual>
+        <origin
+          xyz="
+          ${-MISUMILN_JOINTA_Y}
+          ${-MISUMILN_JOINTA_X}
+          0
+        "
+          rpy="0 0 ${0}" />
         <geometry>
           <mesh
@@ -114,6 +118,10 @@
       <collision>
         <origin
-          xyz="${-MISUMILN_JOINTA_Y} ${-MISUMILN_JOINTA_X} 0"
-          rpy="0 0 0" />
+          xyz="
+          ${-MISUMILN_JOINTA_Y}
+          ${-MISUMILN_JOINTA_X}
+          0
+        "
+          rpy="0 0 ${0}" />
         <geometry>
           <mesh
@@ -127,18 +135,18 @@
     </link>
     <!-- SHOULDER TO TOP DYNAMIXEL -->
-    <joint name="${LEFTSHOULDER_TO_LEFTDYNAMIXELTOP_JOINT_NAME}" type="fixed">
-      <parent link="${L_SHOULDER_LINK_NAME}" />
-      <child link="${L_TOP_DYNAMIXEL_LINK_NAME}" />
-      <origin
-        xyz="
-          ${SHOULDER_X + DYNAMIXEL_X/2}
-          ${SHOULDER_JOINTA_X - DYNAMIXEL_Y/2}
-          ${SHOULDER_Z/2 - DYNAMIXEL_Z/2}
-        "
+    <joint name="${RIGHTSHOULDER_TO_RIGHTDYNAMIXELTOP_JOINT_NAME}" type="fixed">
+      <parent link="${R_SHOULDER_LINK_NAME}" />
+      <child link="${R_TOP_DYNAMIXEL_LINK_NAME}" />
+      <origin
+        xyz="
+        ${SHOULDER_X + DYNAMIXEL_X/2}
+        ${DYNAMIXEL_Y/2 - SHOULDER_JOINTA_X}
+        ${SHOULDER_Z/2 - DYNAMIXEL_Z/2}
+      "
         rpy="0 0 0" />
       <axis xyz="0 0 1" />
     </joint>
     <!-- TOP DYNAMIXEL -->
-    <link name="${L_TOP_DYNAMIXEL_LINK_NAME}">
+    <link name="${R_TOP_DYNAMIXEL_LINK_NAME}">
       <visual>
         <origin xyz="0 0 0" rpy="0 0 0" />
@@ -160,11 +168,11 @@
     </link>
     <!-- TOP DYNAMIXEL TO DRIVING LINK -->
-    <joint name="${LEFTDYNAMIXELTOP_TO_LEFTDRIVING_JOINT_NAME}" type="revolute">
-      <parent link="${L_TOP_DYNAMIXEL_LINK_NAME}" />
-      <child link="${L_DRIVING_LINK_NAME}" />
+    <joint name="${RIGHTDYNAMIXELTOP_TO_RIGHTDRIVING_JOINT_NAME}" type="revolute">
+      <parent link="${R_TOP_DYNAMIXEL_LINK_NAME}" />
+      <child link="${R_DRIVING_LINK_NAME}" />
       <origin
         xyz="
         ${0}
-        ${DYNAMIXEL_JOINTB_Y-DYNAMIXEL_Y/2}
+        ${DYNAMIXEL_Y/2 - DYNAMIXEL_JOINTB_Y}
         ${DRIVING_POS_Z - DYNAMIXEL_TOP_POS_Z}"
         rpy="0 0 ${0}" />
@@ -174,5 +182,5 @@
     </joint>
     <!-- DRIVING LINK -->
-    <link name="${L_DRIVING_LINK_NAME}">
+    <link name="${R_DRIVING_LINK_NAME}">
       <visual>
         <origin

Commit message: added mass to "fix" base in sdf

File: spacediver_ros2_control/description/gazebo/models/spacediver.sdf.xacro (robot description, xacro)
@@ -41,4 +41,15 @@
         </material>
       </visual>
+      <inertial>
+        <mass>10000.0</mass> <!-- Set a very high mass value, e.g., 10,000 kg -->
+        <inertia>
+          <ixx>10000.0</ixx> <!-- Example inertia values (can adjust based on your model's dimensions) -->
+          <iyy>10000.0</iyy>
+          <izz>10000.0</izz>
+          <ixy>0.0</ixy>
+          <ixz>0.0</ixz>
+          <iyz>0.0</iyz>
+        </inertia>
+      </inertial>
     </link>
     <!-- SHOULDER PLATES -->
