Commit message: finished single arm urdf (missing joint between misumilnm and misumilnft)

File: spacediver_ros2_control/description/urdf/parts/spacediver_left_arm.xacro (robot description, xacro)
@@ -30,5 +30,9 @@
       </visual>
       <collision>
-        <origin xyz="${SHOULDER_X/2} ${SHOULDER_Y/2} ${SHOULDER_Z/2}" rpy="0 0 0"/>
+        <origin xyz="
+          ${0}
+          ${SHOULDER_JOINTA_X}
+          ${-SHOULDER_Z/2}
+        " rpy="0 0 ${L_SHOULDER_ROT_Z}"/>
         <geometry>
           <mesh filename="package://spacediver_ros2_control/description/gazebo/models/meshes/shoulder_plate.STL"/>
@@ -97,5 +101,9 @@
       </visual>
       <collision>
-        <origin xyz="0 0 0" rpy="0 0 0"/>
+        <origin xyz="
+          ${L_MISUMILN_POS_X-DYNAMIXEL_POS_X}
+          ${L_MISUMILN_POS_Y+DYNAMIXEL_JOINTB_Y-DYNAMIXEL_POS_Y}
+          0
+        " rpy="0 0 ${L_MISUMILN_ROT_Z}"/>
         <geometry>
           <mesh filename="package://spacediver_ros2_control/description/gazebo/models/meshes/Link_MISUMI_LNMS16-10-200.STL"/>
@@ -164,5 +172,9 @@
       </visual>
       <collision>
-        <origin xyz="0 0 0" rpy="0 0 0"/>
+        <origin xyz="
+          ${-DRIVING_JOINTA_X}
+          ${-DRIVING_JOINTA_Y}
+          ${0}
+        " rpy="0 0 0"/>
         <geometry>
           <mesh filename="package://spacediver_ros2_control/description/gazebo/models/meshes/upper_arm_driving_link.STL"/>
@@ -180,10 +192,10 @@
         ${DRIVING_JOINTB_X-DRIVING_JOINTA_X}
         ${0}
-        ${DRIVEN_POS_Z - DRIVING_POS_Z - DRIVING_Z}
-      "
-        rpy="0 0 ${0}"/>
-      <axis xyz="0 0 1"/>
-      <limit lower="${TOP_DYNAMIXEL_LOWER}" upper="${TOP_DYNAMIXEL_UPPER}"
-        effort="${TOP_DYNAMIXEL_EFFORT}" velocity="${TOP_DYNAMIXEL_VELOCITY}"/>
+        ${DRIVEN_POS_Z - DRIVING_POS_Z}
+      "
+        rpy="0 0 ${0}"/>
+      <axis xyz="0 0 1"/>
+      <limit lower="${-2*PI}" upper="${2*PI}"
+        effort="${10}" velocity="${10}"/>
     </joint>
     <!-- DRIVEN LINK -->
@@ -201,5 +213,9 @@
       </visual>
       <collision>
-        <origin xyz="0 0 0" rpy="0 0 0"/>
+        <origin xyz="
+          ${L_DRIVEN_POS_X - (L_DRIVING_POS_X + DRIVING_JOINTB_X)}
+          ${L_DRIVEN_POS_Y - (L_DRIVING_POS_Y + DRIVING_JOINTB_Y)}
+          ${0}
+        " rpy="0 0 ${L_DRIVEN_ROT_Z}"/>
         <geometry>
           <mesh filename="package://spacediver_ros2_control/description/gazebo/models/meshes/upper_arm_driven_link.STL"/>
@@ -214,8 +230,8 @@
       <visual>
         <origin xyz="
-          ${0}
-          ${0}
-          ${0}
-        " rpy="0 0 ${L_MISUMIFT_ROT_Z}"/>
+          ${MISUMIFT_JOINTA_X}
+          ${MISUMIFT_JOINTA_Y}
+          ${0}"
+          rpy="0 0 ${L_MISUMIFT_ROT_Z}"/>
         <geometry>
           <mesh filename="package://spacediver_ros2_control/description/gazebo/models/meshes/Misumi_LNFTS10-P10-V10-L200-S50-W18-T9.STL"/>
@@ -233,9 +249,4 @@
       </xacro:inertial_box>
     </link>
-<!--
-      ${L_MISUMIFT_POS_X - (L_DRIVEN_POS_X + MISUMIFT_JOINTA_X) + (L_DRIVEN_POS_X - (L_DRIVING_POS_X + DRIVING_JOINTB_X))}
-        ${L_MISUMIFT_POS_Y - (L_DRIVEN_POS_Y + MISUMIFT_JOINTA_Y) + (L_DRIVEN_POS_Y - (L_DRIVING_POS_Y + DRIVING_JOINTB_Y))}
-        ${0}
-     -->
     <!-- DRIVEN LINK TO MISUMI FT -->
     <joint name="${LEFTDRIVEN_TO_LEFTMISUMIFT_JOINT_NAME}" type="revolute">
@@ -245,10 +256,10 @@
         ${L_MISUMIFT_POS_X - (L_DRIVEN_POS_X + MISUMIFT_JOINTA_X) + (L_DRIVEN_POS_X - (L_DRIVING_POS_X + DRIVING_JOINTB_X))}
         ${L_MISUMIFT_POS_Y - (L_DRIVEN_POS_Y + MISUMIFT_JOINTA_Y) + (L_DRIVEN_POS_Y - (L_DRIVING_POS_Y + DRIVING_JOINTB_Y))}
-        ${0}
-      "
-        rpy="0 0 ${0}"/>
-      <axis xyz="0 0 1"/>
-      <limit lower="${TOP_DYNAMIXEL_LOWER}" upper="${TOP_DYNAMIXEL_UPPER}"
-        effort="${TOP_DYNAMIXEL_EFFORT}" velocity="${TOP_DYNAMIXEL_VELOCITY}"/>
+        ${MISUMIFT_POS_Z - DRIVEN_POS_Z}
+      "
+        rpy="0 0 ${0}"/>
+      <axis xyz="0 0 1"/>
+      <limit lower="${-2*PI}" upper="${2*PI}"
+        effort="${10}" velocity="${10}"/>
     </joint>
     <!-- MISUMI LN TO MISUMI FT -->
@@ -263,6 +274,6 @@
         rpy="0 0 ${0}"/>
       <axis xyz="0 0 1"/>
-      <limit lower="${TOP_DYNAMIXEL_LOWER}" upper="${TOP_DYNAMIXEL_UPPER}"
-        effort="${TOP_DYNAMIXEL_EFFORT}" velocity="${TOP_DYNAMIXEL_VELOCITY}"/>
+      <limit lower="${-2*PI}" upper="${2*PI}"
+        effort="${10}" velocity="${10}"/>
     </joint> -->
   </xacro:macro>

Commit message: removed passive links from urdf

File: spacediver_ros2_control/description/urdf/parts/spacediver_left_arm.xacro (robot description, xacro)
@@ -1,280 +1,210 @@
 <?xml version="1.0"?>
-<!-- import xacro reffering here https://gbiggs.github.io/rosjp_urdf_tutorial_text/manipulator_urdf.html -->
+<!-- import xacro reffering here
+https://gbiggs.github.io/rosjp_urdf_tutorial_text/manipulator_urdf.html -->
 <robot xmlns:xacro="http://ros.org/wiki/xacro">
   <xacro:macro name="left_arm" params="base_name *origin">
     <!-- BASE TO SHOULDER -->
     <joint name="${BASE_TO_LEFTSHOULDER_JOINT_NAME}" type="revolute">
-      <parent link="${BASE_LINK_NAME}"/>
-      <child link="${L_SHOULDER_LINK_NAME}"/>
-      <origin xyz="
+      <parent link="${BASE_LINK_NAME}" />
+      <child link="${L_SHOULDER_LINK_NAME}" />
+      <origin
+        xyz="
         ${SHOULDER_POS_X}
         ${-(SHOULDER_JOINTA_X-SHOULDER_Y/2)}
         ${0}
-      " rpy="0 0 0"/>
-      <axis xyz="1 0 0"/>
+      "
+        rpy="0 0 0" />
+      <axis xyz="1 0 0" />
       <limit lower="${BASE_DYNAMIXEL_LOWER}" upper="${BASE_DYNAMIXEL_UPPER}"
-        effort="${BASE_DYNAMIXEL_EFFORT}" velocity="${BASE_DYNAMIXEL_VELOCITY}"/>
+        effort="${BASE_DYNAMIXEL_EFFORT}" velocity="${BASE_DYNAMIXEL_VELOCITY}" />
     </joint>
     <!-- SHOULDER -->
     <link name="${L_SHOULDER_LINK_NAME}">
       <visual>
-        <origin xyz="
+        <origin
+          xyz="
           ${0}
           ${SHOULDER_JOINTA_X}
           ${-SHOULDER_Z/2}
-        " rpy="0 0 ${L_SHOULDER_ROT_Z}"/>
-        <geometry>
-          <mesh filename="package://spacediver_ros2_control/description/gazebo/models/meshes/shoulder_plate.STL"/>
-        </geometry>
-        <material name="grey"/>
-      </visual>
-      <collision>
-        <origin xyz="
+        "
+          rpy="0 0 ${L_SHOULDER_ROT_Z}" />
+        <geometry>
+          <mesh
+            filename="package://spacediver_ros2_control/description/gazebo/models/meshes/shoulder_plate.STL" />
+        </geometry>
+        <material name="grey" />
+      </visual>
+      <collision>
+        <origin
+          xyz="
           ${0}
           ${SHOULDER_JOINTA_X}
           ${-SHOULDER_Z/2}
-        " rpy="0 0 ${L_SHOULDER_ROT_Z}"/>
-        <geometry>
-          <mesh filename="package://spacediver_ros2_control/description/gazebo/models/meshes/shoulder_plate.STL"/>
-        </geometry>
-      </collision>
-      <xacro:inertial_box mass="${LINK_1_MASS}" x="${LINK_1_X/2}" y="${LINK_1_Y/2}" z="${LINK_1_Z/2}">
-        <origin xyz="0 0 ${LINK_1_Z/2}" rpy="0 0 0"/>
+        "
+          rpy="0 0 ${L_SHOULDER_ROT_Z}" />
+        <geometry>
+          <mesh
+            filename="package://spacediver_ros2_control/description/gazebo/models/meshes/shoulder_plate.STL" />
+        </geometry>
+      </collision>
+      <xacro:inertial_box mass="${LINK_1_MASS}" x="${LINK_1_X/2}" y="${LINK_1_Y/2}"
+        z="${LINK_1_Z/2}">
+        <origin xyz="0 0 ${LINK_1_Z/2}" rpy="0 0 0" />
       </xacro:inertial_box>
     </link>
     <!-- SHOULDER TO BOTTOM DYNAMIXEL -->
     <joint name="${LEFTSHOULDER_TO_LEFTDYNAMIXELBOT_JOINT_NAME}" type="fixed">
-      <parent link="${L_SHOULDER_LINK_NAME}"/>
-      <child link="${L_BOT_DYNAMIXEL_LINK_NAME}"/>
-      <origin xyz="
+      <parent link="${L_SHOULDER_LINK_NAME}" />
+      <child link="${L_BOT_DYNAMIXEL_LINK_NAME}" />
+      <origin
+        xyz="
         ${SHOULDER_X + DYNAMIXEL_X/2}
         ${SHOULDER_JOINTA_X - DYNAMIXEL_Y/2}
         ${-SHOULDER_Z/2 + DYNAMIXEL_Z/2}
       "
-        rpy="0 0 0"/>
-      <axis xyz="0 0 1"/>
+        rpy="0 0 0" />
+      <axis xyz="0 0 1" />
     </joint>
     <!-- BOTTOM DYNAMIXEL -->
     <link name="${L_BOT_DYNAMIXEL_LINK_NAME}">
       <visual>
-        <origin xyz="0 0 0" rpy="0 0 0"/>
-        <geometry>
-          <box size="${DYNAMIXEL_X} ${DYNAMIXEL_Y} ${DYNAMIXEL_Z}"/>
-        </geometry>
-        <material name="blue"/>
-      </visual>
-      <collision>
-        <origin xyz="0 0 0" rpy="0 0 0"/>
-        <geometry>
-          <box size="${DYNAMIXEL_X} ${DYNAMIXEL_Y} ${DYNAMIXEL_Z}"/>
-        </geometry>
-      </collision>
-      <xacro:inertial_box mass="${LINK_1_MASS}" x="${LINK_1_X/2}" y="${LINK_1_Y/2}" z="${LINK_1_Z/2}">
-        <origin xyz="0 0 ${LINK_1_Z/2}" rpy="0 0 0"/>
+        <origin xyz="0 0 0" rpy="0 0 0" />
+        <geometry>
+          <box size="${DYNAMIXEL_X} ${DYNAMIXEL_Y} ${DYNAMIXEL_Z}" />
+        </geometry>
+        <material name="blue" />
+      </visual>
+      <collision>
+        <origin xyz="0 0 0" rpy="0 0 0" />
+        <geometry>
+          <box size="${DYNAMIXEL_X} ${DYNAMIXEL_Y} ${DYNAMIXEL_Z}" />
+        </geometry>
+      </collision>
+      <xacro:inertial_box mass="${LINK_1_MASS}" x="${LINK_1_X/2}" y="${LINK_1_Y/2}"
+        z="${LINK_1_Z/2}">
+        <origin xyz="0 0 ${LINK_1_Z/2}" rpy="0 0 0" />
       </xacro:inertial_box>
     </link>
     <!-- BOTTOM DYNAMIXEL TO MISUMI LN -->
     <joint name="${LEFT_DYNAMIXELBOT_TO_LEFTMISUMILN_JOINT_NAME}" type="revolute">
-      <parent link="${L_BOT_DYNAMIXEL_LINK_NAME}"/>
-      <child link="${L_MISUMILN_LINK_NAME}"/>
-      <origin xyz="
+      <parent link="${L_BOT_DYNAMIXEL_LINK_NAME}" />
+      <child link="${L_MISUMILN_LINK_NAME}" />
+      <origin
+        xyz="
         ${0}
         ${DYNAMIXEL_JOINTB_Y-DYNAMIXEL_Y/2}
         ${MISUMILN_POS_Z-DYNAMIXEL_BOT_POS_Z}"
-        rpy="0 0 0"/>
-      <axis xyz="0 0 1"/>
+        rpy="0 0 ${L_MISUMILN_ROT_Z}" />
+      <axis xyz="0 0 1" />
       <limit lower="${BOT_DYNAMIXEL_LOWER}" upper="${BOT_DYNAMIXEL_UPPER}"
-        effort="${BOT_DYNAMIXEL_EFFORT}" velocity="${BOT_DYNAMIXEL_VELOCITY}"/>
+        effort="${BOT_DYNAMIXEL_EFFORT}" velocity="${BOT_DYNAMIXEL_VELOCITY}" />
     </joint>
     <!-- MISUMI LN -->
     <link name="${L_MISUMILN_LINK_NAME}">
       <visual>
-        <origin xyz="
-          ${L_MISUMILN_POS_X-DYNAMIXEL_POS_X}
-          ${L_MISUMILN_POS_Y+DYNAMIXEL_JOINTB_Y-DYNAMIXEL_POS_Y}
-          0
-        " rpy="0 0 ${L_MISUMILN_ROT_Z}"/>
-        <geometry>
-          <mesh filename="package://spacediver_ros2_control/description/gazebo/models/meshes/Link_MISUMI_LNMS16-10-200.STL"/>
-        </geometry>
-        <material name="blue"/>
-      </visual>
-      <collision>
-        <origin xyz="
-          ${L_MISUMILN_POS_X-DYNAMIXEL_POS_X}
-          ${L_MISUMILN_POS_Y+DYNAMIXEL_JOINTB_Y-DYNAMIXEL_POS_Y}
-          0
-        " rpy="0 0 ${L_MISUMILN_ROT_Z}"/>
-        <geometry>
-          <mesh filename="package://spacediver_ros2_control/description/gazebo/models/meshes/Link_MISUMI_LNMS16-10-200.STL"/>
-        </geometry>
-      </collision>
-      <xacro:inertial_box mass="${LINK_1_MASS}" x="${LINK_1_X/2}" y="${LINK_1_Y/2}" z="${LINK_1_Z/2}">
-        <origin xyz="0 0 ${LINK_1_Z/2}" rpy="0 0 0"/>
+        <origin
+          xyz="${-MISUMILN_JOINTA_Y} ${-MISUMILN_JOINTA_X} 0"
+          rpy="0 0 0" />
+        <geometry>
+          <mesh
+            filename="package://spacediver_ros2_control/description/gazebo/models/meshes/Link_MISUMI_LNMS16-10-200.STL" />
+        </geometry>
+        <material name="blue" />
+      </visual>
+      <collision>
+        <origin
+          xyz="${-MISUMILN_JOINTA_Y} ${-MISUMILN_JOINTA_X} 0"
+          rpy="0 0 0" />
+        <geometry>
+          <mesh
+            filename="package://spacediver_ros2_control/description/gazebo/models/meshes/Link_MISUMI_LNMS16-10-200.STL" />
+        </geometry>
+      </collision>
+      <xacro:inertial_box mass="${LINK_1_MASS}" x="${LINK_1_X/2}" y="${LINK_1_Y/2}"
+        z="${LINK_1_Z/2}">
+        <origin xyz="0 0 ${LINK_1_Z/2}" rpy="0 0 0" />
       </xacro:inertial_box>
     </link>
     <!-- SHOULDER TO TOP DYNAMIXEL -->
     <joint name="${LEFTSHOULDER_TO_LEFTDYNAMIXELTOP_JOINT_NAME}" type="fixed">
-      <parent link="${L_SHOULDER_LINK_NAME}"/>
-      <child link="${L_TOP_DYNAMIXEL_LINK_NAME}"/>
-      <origin xyz="
+      <parent link="${L_SHOULDER_LINK_NAME}" />
+      <child link="${L_TOP_DYNAMIXEL_LINK_NAME}" />
+      <origin
+        xyz="
           ${SHOULDER_X + DYNAMIXEL_X/2}
           ${SHOULDER_JOINTA_X - DYNAMIXEL_Y/2}
           ${SHOULDER_Z/2 - DYNAMIXEL_Z/2}
         "
-        rpy="0 0 0"/>
-      <axis xyz="0 0 1"/>
+        rpy="0 0 0" />
+      <axis xyz="0 0 1" />
     </joint>
     <!-- TOP DYNAMIXEL -->
     <link name="${L_TOP_DYNAMIXEL_LINK_NAME}">
       <visual>
-        <origin xyz="0 0 0" rpy="0 0 0"/>
-        <geometry>
-          <box size="${DYNAMIXEL_X} ${DYNAMIXEL_Y} ${DYNAMIXEL_Z}"/>
-        </geometry>
-        <material name="blue"/>
-      </visual>
-      <collision>
-        <origin xyz="0 0 0" rpy="0 0 0"/>
-        <geometry>
-          <box size="${DYNAMIXEL_X} ${DYNAMIXEL_Y} ${DYNAMIXEL_Z}"/>
-        </geometry>
-      </collision>
-      <xacro:inertial_box mass="${LINK_1_MASS}" x="${LINK_1_X/2}" y="${LINK_1_Y/2}" z="${LINK_1_Z/2}">
-        <origin xyz="0 0 ${LINK_1_Z/2}" rpy="0 0 0"/>
+        <origin xyz="0 0 0" rpy="0 0 0" />
+        <geometry>
+          <box size="${DYNAMIXEL_X} ${DYNAMIXEL_Y} ${DYNAMIXEL_Z}" />
+        </geometry>
+        <material name="blue" />
+      </visual>
+      <collision>
+        <origin xyz="0 0 0" rpy="0 0 0" />
+        <geometry>
+          <box size="${DYNAMIXEL_X} ${DYNAMIXEL_Y} ${DYNAMIXEL_Z}" />
+        </geometry>
+      </collision>
+      <xacro:inertial_box mass="${LINK_1_MASS}" x="${LINK_1_X/2}" y="${LINK_1_Y/2}"
+        z="${LINK_1_Z/2}">
+        <origin xyz="0 0 ${LINK_1_Z/2}" rpy="0 0 0" />
       </xacro:inertial_box>
     </link>
     <!-- TOP DYNAMIXEL TO DRIVING LINK -->
     <joint name="${LEFTDYNAMIXELTOP_TO_LEFTDRIVING_JOINT_NAME}" type="revolute">
-      <parent link="${L_TOP_DYNAMIXEL_LINK_NAME}"/>
-      <child link="${L_DRIVING_LINK_NAME}"/>
-      <origin xyz="
+      <parent link="${L_TOP_DYNAMIXEL_LINK_NAME}" />
+      <child link="${L_DRIVING_LINK_NAME}" />
+      <origin
+        xyz="
         ${0}
         ${DYNAMIXEL_JOINTB_Y-DYNAMIXEL_Y/2}
         ${DRIVING_POS_Z - DYNAMIXEL_TOP_POS_Z}"
-        rpy="0 0 ${0}"/>
-      <axis xyz="0 0 1"/>
+        rpy="0 0 ${0}" />
+      <axis xyz="0 0 1" />
       <limit lower="${TOP_DYNAMIXEL_LOWER}" upper="${TOP_DYNAMIXEL_UPPER}"
-        effort="${TOP_DYNAMIXEL_EFFORT}" velocity="${TOP_DYNAMIXEL_VELOCITY}"/>
+        effort="${TOP_DYNAMIXEL_EFFORT}" velocity="${TOP_DYNAMIXEL_VELOCITY}" />
     </joint>
     <!-- DRIVING LINK -->
     <link name="${L_DRIVING_LINK_NAME}">
       <visual>
-        <origin xyz="
+        <origin
+          xyz="
           ${-DRIVING_JOINTA_X}
           ${-DRIVING_JOINTA_Y}
           ${0}
-        " rpy="0 0 0"/>
-        <geometry>
-          <mesh filename="package://spacediver_ros2_control/description/gazebo/models/meshes/upper_arm_driving_link.STL"/>
-        </geometry>
-        <material name="blue"/>
-      </visual>
-      <collision>
-        <origin xyz="
+        "
+          rpy="0 0 0" />
+        <geometry>
+          <mesh
+            filename="package://spacediver_ros2_control/description/gazebo/models/meshes/upper_arm_driving_link.STL" />
+        </geometry>
+        <material name="blue" />
+      </visual>
+      <collision>
+        <origin
+          xyz="
           ${-DRIVING_JOINTA_X}
           ${-DRIVING_JOINTA_Y}
           ${0}
-        " rpy="0 0 0"/>
-        <geometry>
-          <mesh filename="package://spacediver_ros2_control/description/gazebo/models/meshes/upper_arm_driving_link.STL"/>
-        </geometry>
-      </collision>
-      <xacro:inertial_box mass="${LINK_1_MASS}" x="${LINK_1_X/2}" y="${LINK_1_Y/2}" z="${LINK_1_Z/2}">
-        <origin xyz="0 0 ${LINK_1_Z/2}" rpy="0 0 0"/>
-      </xacro:inertial_box>
-    </link>
-    <!-- DRIVING LINK TO DRIVEN LINK-->
-    <joint name="${LEFTDRIVING_TO_LEFTDRIVEN_JOINT_NAME}" type="revolute">
-      <parent link="${L_DRIVING_LINK_NAME}"/>
-      <child link="${L_DRIVEN_LINK_NAME}"/>
-      <origin xyz="
-        ${DRIVING_JOINTB_X-DRIVING_JOINTA_X}
-        ${0}
-        ${DRIVEN_POS_Z - DRIVING_POS_Z}
-      "
-        rpy="0 0 ${0}"/>
-      <axis xyz="0 0 1"/>
-      <limit lower="${-2*PI}" upper="${2*PI}"
-        effort="${10}" velocity="${10}"/>
-    </joint>
-    <!-- DRIVEN LINK -->
-    <link name="${L_DRIVEN_LINK_NAME}">
-      <visual>
-        <origin xyz="
-          ${L_DRIVEN_POS_X - (L_DRIVING_POS_X + DRIVING_JOINTB_X)}
-          ${L_DRIVEN_POS_Y - (L_DRIVING_POS_Y + DRIVING_JOINTB_Y)}
-          ${0}
-        " rpy="0 0 ${L_DRIVEN_ROT_Z}"/>
-        <geometry>
-          <mesh filename="package://spacediver_ros2_control/description/gazebo/models/meshes/upper_arm_driven_link.STL"/>
-        </geometry>
-        <material name="blue"/>
-      </visual>
-      <collision>
-        <origin xyz="
-          ${L_DRIVEN_POS_X - (L_DRIVING_POS_X + DRIVING_JOINTB_X)}
-          ${L_DRIVEN_POS_Y - (L_DRIVING_POS_Y + DRIVING_JOINTB_Y)}
-          ${0}
-        " rpy="0 0 ${L_DRIVEN_ROT_Z}"/>
-        <geometry>
-          <mesh filename="package://spacediver_ros2_control/description/gazebo/models/meshes/upper_arm_driven_link.STL"/>
-        </geometry>
-      </collision>
-      <xacro:inertial_box mass="${LINK_1_MASS}" x="${LINK_1_X/2}" y="${LINK_1_Y/2}" z="${LINK_1_Z/2}">
-        <origin xyz="0 0 ${LINK_1_Z/2}" rpy="0 0 0"/>
-      </xacro:inertial_box>
-    </link>
-    <!-- MISUMI FT -->
-    <link name="${L_MISUMIFT_LINK_NAME}">
-      <visual>
-        <origin xyz="
-          ${MISUMIFT_JOINTA_X}
-          ${MISUMIFT_JOINTA_Y}
-          ${0}"
-          rpy="0 0 ${L_MISUMIFT_ROT_Z}"/>
-        <geometry>
-          <mesh filename="package://spacediver_ros2_control/description/gazebo/models/meshes/Misumi_LNFTS10-P10-V10-L200-S50-W18-T9.STL"/>
-        </geometry>
-        <material name="blue"/>
-      </visual>
-      <collision>
-        <origin xyz="0 0 0" rpy="0 0 0"/>
-        <geometry>
-          <mesh filename="package://spacediver_ros2_control/description/gazebo/models/meshes/Misumi_LNFTS10-P10-V10-L200-S50-W18-T9.STL"/>
-        </geometry>
-      </collision>
-      <xacro:inertial_box mass="${LINK_1_MASS}" x="${LINK_1_X/2}" y="${LINK_1_Y/2}" z="${LINK_1_Z/2}">
-        <origin xyz="0 0 ${LINK_1_Z/2}" rpy="0 0 0"/>
-      </xacro:inertial_box>
-    </link>
-    <!-- DRIVEN LINK TO MISUMI FT -->
-    <joint name="${LEFTDRIVEN_TO_LEFTMISUMIFT_JOINT_NAME}" type="revolute">
-      <parent link="${L_DRIVEN_LINK_NAME}"/>
-      <child link="${L_MISUMIFT_LINK_NAME}"/>
-      <origin xyz="
-        ${L_MISUMIFT_POS_X - (L_DRIVEN_POS_X + MISUMIFT_JOINTA_X) + (L_DRIVEN_POS_X - (L_DRIVING_POS_X + DRIVING_JOINTB_X))}
-        ${L_MISUMIFT_POS_Y - (L_DRIVEN_POS_Y + MISUMIFT_JOINTA_Y) + (L_DRIVEN_POS_Y - (L_DRIVING_POS_Y + DRIVING_JOINTB_Y))}
-        ${MISUMIFT_POS_Z - DRIVEN_POS_Z}
-      "
-        rpy="0 0 ${0}"/>
-      <axis xyz="0 0 1"/>
-      <limit lower="${-2*PI}" upper="${2*PI}"
-        effort="${10}" velocity="${10}"/>
-    </joint>
-    <!-- MISUMI LN TO MISUMI FT -->
-    <!-- <joint name="${LEFTMISUMILN_TO_LEFTMISUMIFT_JOINT_NAME}" type="revolute">
-      <parent link="${L_MISUMILN_LINK_NAME}"/>
-      <child link="${L_MISUMIFT_LINK_NAME}"/>
-      <origin xyz="
-        ${0}
-        ${0}
-        ${0}
-      "
-        rpy="0 0 ${0}"/>
-      <axis xyz="0 0 1"/>
-      <limit lower="${-2*PI}" upper="${2*PI}"
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