Commit message: first_test only left_arm

File: spacediver_ros2_control/description/urdf/parts/spacediver_left_arm.xacro (robot description, xacro)
@@ -48,8 +48,18 @@
         </geometry>
       </collision>
-      <xacro:inertial_box mass="${LINK_1_MASS}" x="${LINK_1_X/2}" y="${LINK_1_Y/2}"
-        z="${LINK_1_Z/2}">
-        <origin xyz="0 0 ${LINK_1_Z/2}" rpy="0 0 0" />
-      </xacro:inertial_box>
+      <inertial>
+        <origin
+          xyz="157.37 15.17 32.18"
+          rpy="0 0 ${radians(90)}" />
+        <mass
+          value="152" />
+        <inertia
+          ixx="400463.56"
+          ixy="0.00"
+          ixz="156.80"
+          iyy="54063.82"
+          iyz="-1.4424E-06"
+          izz="369542.91" />
+      </inertial>
     </link>
     <!-- SHOULDER TO BOTTOM DYNAMIXEL -->
@@ -81,4 +91,95 @@
         </geometry>
       </collision>
+      <inertial>
+        <origin
+          xyz="0 0 -0.0030083"
+          rpy="0 0 ${radians(90)}" />
+        <mass
+          value="3.1152" />
+        <!-- 不明点 -->
+        <xacro:inertial_box mass="${LINK_1_MASS}" x="${LINK_1_X/2}" y="${LINK_1_Y/2}"
+          z="${LINK_1_Z/2}">
+          <origin xyz="0 0 ${LINK_1_Z/2}" rpy="0 0 0" />
+        </xacro:inertial_box>
+    </link>
+    <!-- BOTTOM DYNAMIXEL TO MISUMI LN -->
+    <joint name="${LEFT_DYNAMIXELBOT_TO_LEFTMISUMILN_JOINT_NAME}" type="revolute">
+      <parent link="${L_BOT_DYNAMIXEL_LINK_NAME}" />
+      <child link="${L_MISUMILN_LINK_NAME}" />
+      <origin
+        xyz="
+        ${0}
+        ${DYNAMIXEL_JOINTB_Y-DYNAMIXEL_Y/2}
+        ${MISUMILN_POS_Z-DYNAMIXEL_BOT_POS_Z}"
+        rpy="0 0 ${L_MISUMILN_ROT_Z}" />
+      <axis xyz="0 0 1" />
+      <limit lower="${BOT_DYNAMIXEL_LOWER}" upper="${BOT_DYNAMIXEL_UPPER}"
+        effort="${BOT_DYNAMIXEL_EFFORT}" velocity="${BOT_DYNAMIXEL_VELOCITY}" />
+    </joint>
+    <!-- MISUMI LN -->
+    <link name="${L_MISUMILN_LINK_NAME}">
+      <visual>
+        <origin
+          xyz="${-MISUMILN_JOINTA_Y} ${-MISUMILN_JOINTA_X} 0"
+          rpy="0 0 0" />
+        <geometry>
+          <mesh
+            filename="package://spacediver_ros2_control/description/gazebo/models/meshes/Link_MISUMI_LNMS16-10-200.STL" />
+        </geometry>
+        <material name="blue" />
+      </visual>
+      <collision>
+        <origin
+          xyz="${-MISUMILN_JOINTA_Y} ${-MISUMILN_JOINTA_X} 0"
+          rpy="0 0 0" />
+        <geometry>
+          <mesh
+            filename="package://spacediver_ros2_control/description/gazebo/models/meshes/Link_MISUMI_LNMS16-10-200.STL" />
+        </geometry>
+      </collision>
+      <inertial>
+        <origin
+          xyz=" 234.53 4.17 139.95"
+          rpy="0 0 ${radians(90)}" />
+        <mass
+          value="473" />
+        <inertia
+          ixx="1474475.79"
+          ixy="0.00"
+          ixz="678078.58"
+          iyy="1833808.78"
+          iyz="0.00"
+          izz="365725.00" />
+      </inertial>
+    </link>
+    <!-- SHOULDER TO TOP DYNAMIXEL -->
+    <joint name="${LEFTSHOULDER_TO_LEFTDYNAMIXELTOP_JOINT_NAME}" type="fixed">
+      <parent link="${L_SHOULDER_LINK_NAME}" />
+      <child link="${L_TOP_DYNAMIXEL_LINK_NAME}" />
+      <origin
+        xyz="
+          ${SHOULDER_X + DYNAMIXEL_X/2}
+          ${SHOULDER_JOINTA_X - DYNAMIXEL_Y/2}
+          ${SHOULDER_Z/2 - DYNAMIXEL_Z/2}
+        "
+        rpy="0 0 0" />
+      <axis xyz="0 0 1" />
+    </joint>
+    <!-- TOP DYNAMIXEL -->
+    <link name="${L_TOP_DYNAMIXEL_LINK_NAME}">
+      <visual>
+        <origin xyz="0 0 0" rpy="0 0 0" />
+        <geometry>
+          <box size="${DYNAMIXEL_X} ${DYNAMIXEL_Y} ${DYNAMIXEL_Z}" />
+        </geometry>
+        <material name="blue" />
+      </visual>
+      <collision>
+        <origin xyz="0 0 0" rpy="0 0 0" />
+        <geometry>
+          <box size="${DYNAMIXEL_X} ${DYNAMIXEL_Y} ${DYNAMIXEL_Z}" />
+        </geometry>
+      </collision>
+      <!-- 不明点 -->
       <xacro:inertial_box mass="${LINK_1_MASS}" x="${LINK_1_X/2}" y="${LINK_1_Y/2}"
         z="${LINK_1_Z/2}">
@@ -86,77 +187,4 @@
       </xacro:inertial_box>
     </link>
-    <!-- BOTTOM DYNAMIXEL TO MISUMI LN -->
-    <joint name="${LEFT_DYNAMIXELBOT_TO_LEFTMISUMILN_JOINT_NAME}" type="revolute">
-      <parent link="${L_BOT_DYNAMIXEL_LINK_NAME}" />
-      <child link="${L_MISUMILN_LINK_NAME}" />
-      <origin
-        xyz="
-        ${0}
-        ${DYNAMIXEL_JOINTB_Y-DYNAMIXEL_Y/2}
-        ${MISUMILN_POS_Z-DYNAMIXEL_BOT_POS_Z}"
-        rpy="0 0 ${L_MISUMILN_ROT_Z}" />
-      <axis xyz="0 0 1" />
-      <limit lower="${BOT_DYNAMIXEL_LOWER}" upper="${BOT_DYNAMIXEL_UPPER}"
-        effort="${BOT_DYNAMIXEL_EFFORT}" velocity="${BOT_DYNAMIXEL_VELOCITY}" />
-    </joint>
-    <!-- MISUMI LN -->
-    <link name="${L_MISUMILN_LINK_NAME}">
-      <visual>
-        <origin
-          xyz="${-MISUMILN_JOINTA_Y} ${-MISUMILN_JOINTA_X} 0"
-          rpy="0 0 0" />
-        <geometry>
-          <mesh
-            filename="package://spacediver_ros2_control/description/gazebo/models/meshes/Link_MISUMI_LNMS16-10-200.STL" />
-        </geometry>
-        <material name="blue" />
-      </visual>
-      <collision>
-        <origin
-          xyz="${-MISUMILN_JOINTA_Y} ${-MISUMILN_JOINTA_X} 0"
-          rpy="0 0 0" />
-        <geometry>
-          <mesh
-            filename="package://spacediver_ros2_control/description/gazebo/models/meshes/Link_MISUMI_LNMS16-10-200.STL" />
-        </geometry>
-      </collision>
-      <xacro:inertial_box mass="${LINK_1_MASS}" x="${LINK_1_X/2}" y="${LINK_1_Y/2}"
-        z="${LINK_1_Z/2}">
-        <origin xyz="0 0 ${LINK_1_Z/2}" rpy="0 0 0" />
-      </xacro:inertial_box>
-    </link>
-    <!-- SHOULDER TO TOP DYNAMIXEL -->
-    <joint name="${LEFTSHOULDER_TO_LEFTDYNAMIXELTOP_JOINT_NAME}" type="fixed">
-      <parent link="${L_SHOULDER_LINK_NAME}" />
-      <child link="${L_TOP_DYNAMIXEL_LINK_NAME}" />
-      <origin
-        xyz="
-          ${SHOULDER_X + DYNAMIXEL_X/2}
-          ${SHOULDER_JOINTA_X - DYNAMIXEL_Y/2}
-          ${SHOULDER_Z/2 - DYNAMIXEL_Z/2}
-        "
-        rpy="0 0 0" />
-      <axis xyz="0 0 1" />
-    </joint>
-    <!-- TOP DYNAMIXEL -->
-    <link name="${L_TOP_DYNAMIXEL_LINK_NAME}">
-      <visual>
-        <origin xyz="0 0 0" rpy="0 0 0" />
-        <geometry>
-          <box size="${DYNAMIXEL_X} ${DYNAMIXEL_Y} ${DYNAMIXEL_Z}" />
-        </geometry>
-        <material name="blue" />
-      </visual>
-      <collision>
-        <origin xyz="0 0 0" rpy="0 0 0" />
-        <geometry>
-          <box size="${DYNAMIXEL_X} ${DYNAMIXEL_Y} ${DYNAMIXEL_Z}" />
-        </geometry>
-      </collision>
-      <xacro:inertial_box mass="${LINK_1_MASS}" x="${LINK_1_X/2}" y="${LINK_1_Y/2}"
-        z="${LINK_1_Z/2}">
-        <origin xyz="0 0 ${LINK_1_Z/2}" rpy="0 0 0" />
-      </xacro:inertial_box>
-    </link>
     <!-- TOP DYNAMIXEL TO DRIVING LINK -->
     <joint name="${LEFTDYNAMIXELTOP_TO_LEFTDRIVING_JOINT_NAME}" type="revolute">
@@ -202,8 +230,18 @@
         </geometry>
       </collision>
-      <xacro:inertial_box mass="${LINK_1_MASS}" x="${LINK_1_X/2}" y="${LINK_1_Y/2}"
-        z="${LINK_1_Z/2}">
-        <origin xyz="0 0 ${LINK_1_Z/2}" rpy="0 0 0" />
-      </xacro:inertial_box>
+      <inertial>
+        <origin
+          xyz="214.98 38.67 39.12"
+          rpy="0 0 ${radians(90)}" />
+        <mass
+          value="7.30" />
+        <inertia
+          ixx="706.95"
+          ixy="0.00"
+          ixz="-788.79"
+          iyy="3292.20"
+          iyz="0.00"
+          izz="2604.72" />
+      </inertial>
     </link>
   </xacro:macro>

Commit message: Left arm URDF completed

File: spacediver_ros2_control/description/urdf/parts/spacediver_left_arm.xacro (robot description, xacro)
@@ -35,30 +35,17 @@
         <material name="grey" />
       </visual>
-      <collision>
-        <origin
-          xyz="
-          ${0}
-          ${SHOULDER_JOINTA_X}
-          ${-SHOULDER_Z/2}
-        "
-          rpy="0 0 ${L_SHOULDER_ROT_Z}" />
-        <geometry>
-          <mesh
-            filename="package://spacediver_ros2_control/description/gazebo/models/meshes/shoulder_plate.STL" />
-        </geometry>
-      </collision>
-      <inertial>
-        <origin
-          xyz="157.37 15.17 32.18"
-          rpy="0 0 ${radians(90)}" />
-        <mass
-          value="152" />
-        <inertia
-          ixx="400463.56"
-          ixy="0.00"
-          ixz="156.80"
-          iyy="54063.82"
-          iyz="-1.4424E-06"
-          izz="369542.91" />
+      <inertial>
+        <origin
+          xyz="-0.05806 0.01517 0.03218"
+          rpy="0 0 ${radians(90)}" />
+        <mass
+          value="0.152" />
+        <inertia
+          ixx="0.40046356"
+          ixy="0.00"
+          ixz="0.00015680"
+          iyy="0.05406382"
+          iyz="0.00"
+          izz="0.36954291" />
       </inertial>
     </link>
@@ -85,21 +72,18 @@
         <material name="blue" />
       </visual>
-      <collision>
-        <origin xyz="0 0 0" rpy="0 0 0" />
-        <geometry>
-          <box size="${DYNAMIXEL_X} ${DYNAMIXEL_Y} ${DYNAMIXEL_Z}" />
-        </geometry>
-      </collision>
-      <inertial>
-        <origin
-          xyz="0 0 -0.0030083"
-          rpy="0 0 ${radians(90)}" />
-        <mass
-          value="3.1152" />
-        <!-- 不明点 -->
-        <xacro:inertial_box mass="${LINK_1_MASS}" x="${LINK_1_X/2}" y="${LINK_1_Y/2}"
-          z="${LINK_1_Z/2}">
-          <origin xyz="0 0 ${LINK_1_Z/2}" rpy="0 0 0" />
-        </xacro:inertial_box>
+      <inertial>
+        <origin
+          xyz="0.190.91 -0.03620 0.03207"
+          rpy="0 0 ${radians(90)}" />
+        <mass
+          value="0.08395" />
+        <inertia
+          ixx="0.03680554"
+          ixy="0.00"
+          ixz="0.00"
+          iyy="0.03139792"
+          iyz="0.00078981"
+          izz="0.02106717" />
+      </inertial>
     </link>
     <!-- BOTTOM DYNAMIXEL TO MISUMI LN -->
@@ -143,12 +127,12 @@
           rpy="0 0 ${radians(90)}" />
         <mass
-          value="473" />
-        <inertia
-          ixx="1474475.79"
-          ixy="0.00"
-          ixz="678078.58"
-          iyy="1833808.78"
+          value="0.473" />
+        <inertia
+          ixx="1.47447579"
+          ixy="0.00"
+          ixz="0.67807858"
+          iyy="1.83380878"
           iyz="0.00"
-          izz="365725.00" />
+          izz="0.36572500" />
       </inertial>
     </link>
@@ -175,15 +159,18 @@
         <material name="blue" />
       </visual>
-      <collision>
-        <origin xyz="0 0 0" rpy="0 0 0" />
-        <geometry>
-          <box size="${DYNAMIXEL_X} ${DYNAMIXEL_Y} ${DYNAMIXEL_Z}" />
-        </geometry>
-      </collision>
-      <!-- 不明点 -->
-      <xacro:inertial_box mass="${LINK_1_MASS}" x="${LINK_1_X/2}" y="${LINK_1_Y/2}"
-        z="${LINK_1_Z/2}">
-        <origin xyz="0 0 ${LINK_1_Z/2}" rpy="0 0 0" />
-      </xacro:inertial_box>
+      <inertial>
+        <origin
+          xyz="0.190.91 0.06654 0.03207"
+          rpy="0 0 ${radians(90)}" />
+        <mass
+          value="0.08395" />
+        <inertia
+          ixx="0.03680554"
+          ixy="0.00"
+          ixz="0.00"
+          iyy="0.03139792"
+          iyz="0.00078981"
+          izz="0.02106717" />
+      </inertial>
     </link>
     <!-- TOP DYNAMIXEL TO DRIVING LINK -->
@@ -235,12 +222,12 @@
           rpy="0 0 ${radians(90)}" />
         <mass
-          value="7.30" />
-        <inertia
-          ixx="706.95"
-          ixy="0.00"
-          ixz="-788.79"
-          iyy="3292.20"
+          value="0.00730" />
+        <inertia
+          ixx="0.00070695"
+          ixy="0.00"
+          ixz="-0.00078879"
+          iyy="0.00329220"
           iyz="0.00"
-          izz="2604.72" />
+          izz="0.00260472" />
       </inertial>
     </link>
