Commit message: updated dual arm urdf

File: spacediver_ros2_control/description/urdf/parts/spacediver_left_arm.xacro (robot description, xacro)
@@ -61,5 +61,5 @@
       </inertial>
     </link>
-    <!-- Joint 2 -->
+    <!-- Joint 3 -->
     <joint name="${LEFTDYNAMIXELTOP_TO_LEFTDRIVING_JOINT_NAME}" type="revolute">
       <parent link="${L_MISUMILN_LINK_NAME}" />

File: spacediver_ros2_control/description/urdf/parts/spacediver_right_arm.xacro (robot description, xacro)
@@ -9,13 +9,8 @@
       <child link="${R_SHOULDER_LINK_NAME}" />
       <origin
-        xyz="
-        ${-SHOULDER_POS_X}
-        ${-(SHOULDER_JOINTA_X-SHOULDER_Y/2)}
-        ${0}
-      "
-        rpy="0 0 ${PI}" />
-      <axis xyz="1 0 0" />
-      <limit lower="${BASE_DYNAMIXEL_LOWER}" upper="${BASE_DYNAMIXEL_UPPER}"
-        effort="${BASE_DYNAMIXEL_EFFORT}" velocity="${BASE_DYNAMIXEL_VELOCITY}" />
+        xyz="${SHOULDER_POS_X} ${SHOULDER_JOINTA_X-SHOULDER_Y/2} 0"
+        rpy="0 ${PI/2} 0" />
+      <axis xyz="0 0 1" />
+      <limit lower="-1.57" upper="1.57" effort="10" velocity="1" />
     </joint>
     <!-- SHOULDER -->
@@ -23,195 +18,77 @@
       <visual>
         <origin
-          xyz="
-          ${0}
-          ${-SHOULDER_JOINTA_X}
-          ${SHOULDER_Z/2}
-        "
-          rpy="${PI} 0 ${-L_SHOULDER_ROT_Z}" />
+          xyz="${-SHOULDER_Z/2} ${-SHOULDER_JOINTA_X} 0"
+          rpy="${PI/2} 0 ${PI/2}" />
         <geometry>
           <mesh
             filename="package://spacediver_ros2_control/description/gazebo/models/meshes/shoulder_plate.STL" />
         </geometry>
-        <material name="grey" />
       </visual>
-      <collision>
-        <origin
-          xyz="
-          ${0}
-          ${-SHOULDER_JOINTA_X}
-          ${SHOULDER_Z/2}
-        "
-          rpy="${PI} 0 ${-L_SHOULDER_ROT_Z}" />
-        <geometry>
-          <mesh
-            filename="package://spacediver_ros2_control/description/gazebo/models/meshes/shoulder_plate.STL" />
-        </geometry>
-      </collision>
-      <xacro:inertial_box mass="${LINK_1_MASS}" x="${LINK_1_X/2}" y="${LINK_1_Y/2}"
-        z="${LINK_1_Z/2}">
-        <origin xyz="0 0 ${LINK_1_Z/2}" rpy="0 0 0" />
-      </xacro:inertial_box>
+      <inertial>
+        <origin xyz="0 0 0.25" rpy="0 0 0" />
+        <mass value="1.0" />
+        <inertia ixx="0.01" ixy="0.0" ixz="0.0" iyy="0.01" iyz="0.0" izz="0.01" />
+      </inertial>
     </link>
-    <!-- SHOULDER TO BOTTOM DYNAMIXEL -->
-    <joint name="${RIGHTSHOULDER_TO_RIGHTDYNAMIXELBOT_JOINT_NAME}" type="fixed">
+    <!-- Joint 2 -->
+    <joint name="${RIGHT_DYNAMIXELBOT_TO_RIGHTMISUMILN_JOINT_NAME}" type="revolute">
       <parent link="${R_SHOULDER_LINK_NAME}" />
-      <child link="${R_BOT_DYNAMIXEL_LINK_NAME}" />
-      <origin
-        xyz="
-        ${SHOULDER_X + DYNAMIXEL_X/2}
-        ${DYNAMIXEL_Y/2 - SHOULDER_JOINTA_X}
-        ${-SHOULDER_Z/2 + DYNAMIXEL_Z/2}
-      "
-        rpy="0 0 0" />
-      <axis xyz="0 0 1" />
-    </joint>
-    <!-- BOTTOM DYNAMIXEL -->
-    <link name="${R_BOT_DYNAMIXEL_LINK_NAME}">
-      <visual>
-        <origin xyz="0 0 0" rpy="0 0 0" />
-        <geometry>
-          <box size="${DYNAMIXEL_X} ${DYNAMIXEL_Y} ${DYNAMIXEL_Z}" />
-        </geometry>
-        <material name="blue" />
-      </visual>
-      <collision>
-        <origin xyz="0 0 0" rpy="0 0 0" />
-        <geometry>
-          <box size="${DYNAMIXEL_X} ${DYNAMIXEL_Y} ${DYNAMIXEL_Z}" />
-        </geometry>
-      </collision>
-      <xacro:inertial_box mass="${LINK_1_MASS}" x="${LINK_1_X/2}" y="${LINK_1_Y/2}"
-        z="${LINK_1_Z/2}">
-        <origin xyz="0 0 ${LINK_1_Z/2}" rpy="0 0 0" />
-      </xacro:inertial_box>
-    </link>
-    <!-- BOTTOM DYNAMIXEL TO MISUMI LN -->
-    <joint name="${RIGHT_DYNAMIXELBOT_TO_RIGHTMISUMILN_JOINT_NAME}" type="revolute">
-      <parent link="${R_BOT_DYNAMIXEL_LINK_NAME}" />
       <child link="${R_MISUMILN_LINK_NAME}" />
       <origin
-        xyz="
-        ${0}
-        ${DYNAMIXEL_Y/2 - DYNAMIXEL_JOINTB_Y}
-        ${MISUMILN_POS_Z-DYNAMIXEL_BOT_POS_Z}"
-        rpy="0 0 ${-L_MISUMILN_ROT_Z}" />
+        xyz="${SHOULDER_Z/2 - DYNAMIXEL_Z - 0.0145} 0 ${SHOULDER_X + DYNAMIXEL_X/2}"
+        rpy="${-PI/2} ${-ROT} ${PI/2}" />
       <axis xyz="0 0 1" />
-      <limit lower="${BOT_DYNAMIXEL_LOWER}" upper="${BOT_DYNAMIXEL_UPPER}"
-        effort="${BOT_DYNAMIXEL_EFFORT}" velocity="${BOT_DYNAMIXEL_VELOCITY}" />
+      <limit lower="-1.57" upper="1.57" effort="10" velocity="1" />
     </joint>
-    <!-- MISUMI LN -->
+    <!-- FIRST LINK -->
     <link name="${R_MISUMILN_LINK_NAME}">
       <visual>
         <origin
-          xyz="
-          ${-MISUMILN_JOINTA_Y}
-          ${-MISUMILN_JOINTA_X}
-          0
-        "
-          rpy="0 0 ${0}" />
+          xyz="${-MISUMILN_JOINTA_Y} ${-MISUMILN_JOINTA_X} 0"
+          rpy="0 0 0" />
         <geometry>
           <mesh
             filename="package://spacediver_ros2_control/description/gazebo/models/meshes/Link_MISUMI_LNMS16-10-200.STL" />
         </geometry>
-        <material name="blue" />
+        <material name="green">
+          <color rgba="0 1 0 1" />
+        </material>
       </visual>
-      <collision>
-        <origin
-          xyz="
-          ${-MISUMILN_JOINTA_Y}
-          ${-MISUMILN_JOINTA_X}
-          0
-        "
-          rpy="0 0 ${0}" />
-        <geometry>
-          <mesh
-            filename="package://spacediver_ros2_control/description/gazebo/models/meshes/Link_MISUMI_LNMS16-10-200.STL" />
-        </geometry>
-      </collision>
-      <xacro:inertial_box mass="${LINK_1_MASS}" x="${LINK_1_X/2}" y="${LINK_1_Y/2}"
-        z="${LINK_1_Z/2}">
-        <origin xyz="0 0 ${LINK_1_Z/2}" rpy="0 0 0" />
-      </xacro:inertial_box>
+      <inertial>
+        <origin xyz="0 0 0.1" rpy="0 0 0" />
+        <mass value="1.0" />
+        <inertia ixx="0.01" ixy="0.0" ixz="0.0" iyy="0.01" iyz="0.0" izz="0.01" />
+      </inertial>
     </link>
-    <!-- SHOULDER TO TOP DYNAMIXEL -->
-    <joint name="${RIGHTSHOULDER_TO_RIGHTDYNAMIXELTOP_JOINT_NAME}" type="fixed">
-      <parent link="${R_SHOULDER_LINK_NAME}" />
-      <child link="${R_TOP_DYNAMIXEL_LINK_NAME}" />
-      <origin
-        xyz="
-        ${SHOULDER_X + DYNAMIXEL_X/2}
-        ${DYNAMIXEL_Y/2 - SHOULDER_JOINTA_X}
-        ${SHOULDER_Z/2 - DYNAMIXEL_Z/2}
-      "
-        rpy="0 0 0" />
-      <axis xyz="0 0 1" />
-    </joint>
-    <!-- TOP DYNAMIXEL -->
-    <link name="${R_TOP_DYNAMIXEL_LINK_NAME}">
-      <visual>
-        <origin xyz="0 0 0" rpy="0 0 0" />
-        <geometry>
-          <box size="${DYNAMIXEL_X} ${DYNAMIXEL_Y} ${DYNAMIXEL_Z}" />
-        </geometry>
-        <material name="blue" />
-      </visual>
-      <collision>
-        <origin xyz="0 0 0" rpy="0 0 0" />
-        <geometry>
-          <box size="${DYNAMIXEL_X} ${DYNAMIXEL_Y} ${DYNAMIXEL_Z}" />
-        </geometry>
-      </collision>
-      <xacro:inertial_box mass="${LINK_1_MASS}" x="${LINK_1_X/2}" y="${LINK_1_Y/2}"
-        z="${LINK_1_Z/2}">
-        <origin xyz="0 0 ${LINK_1_Z/2}" rpy="0 0 0" />
-      </xacro:inertial_box>
-    </link>
-    <!-- TOP DYNAMIXEL TO DRIVING LINK -->
+    <!-- Joint 3 -->
     <joint name="${RIGHTDYNAMIXELTOP_TO_RIGHTDRIVING_JOINT_NAME}" type="revolute">
-      <parent link="${R_TOP_DYNAMIXEL_LINK_NAME}" />
+      <parent link="${R_MISUMILN_LINK_NAME}" />
       <child link="${R_DRIVING_LINK_NAME}" />
       <origin
-        xyz="
-        ${0}
-        ${DYNAMIXEL_Y/2 - DYNAMIXEL_JOINTB_Y}
-        ${DRIVING_POS_Z - DYNAMIXEL_TOP_POS_Z}"
-        rpy="0 0 ${0}" />
+        xyz="${MISUMILN_JOINTB_Y} 0 ${MISUMILN_Z}"
+        rpy="0 0 ${PI/2 + ROT}" />
       <axis xyz="0 0 1" />
-      <limit lower="${TOP_DYNAMIXEL_LOWER}" upper="${TOP_DYNAMIXEL_UPPER}"
-        effort="${TOP_DYNAMIXEL_EFFORT}" velocity="${TOP_DYNAMIXEL_VELOCITY}" />
+      <limit lower="-1.57" upper="1.57" effort="10" velocity="1" />
+      <mimic joint="${LEFT_DYNAMIXELBOT_TO_LEFTMISUMILN_JOINT_NAME}" multiplier="1" offset="0" />
     </joint>
-    <!-- DRIVING LINK -->
+    <!-- SECOND LINK -->
     <link name="${R_DRIVING_LINK_NAME}">
       <visual>
         <origin
-          xyz="
-          ${-DRIVING_JOINTA_X}
-          ${-DRIVING_JOINTA_Y}
-          ${0}
-        "
+          xyz="${-MISUMIFT_JOINTB_X} ${-MISUMIFT_JOINTB_Y} 0"
           rpy="0 0 0" />
         <geometry>
           <mesh
-            filename="package://spacediver_ros2_control/description/gazebo/models/meshes/upper_arm_driving_link.STL" />
+            filename="package://spacediver_ros2_control/description/gazebo/models/meshes/Misumi_LNFTS10-P10-V10-L200-S50-W18-T9.STL" />
         </geometry>
-        <material name="blue" />
+        <material name="red">
+          <color rgba="1 0 0 1" />
+        </material>
       </visual>
-      <collision>
-        <origin
-          xyz="
-          ${-DRIVING_JOINTA_X}
-          ${-DRIVING_JOINTA_Y}
-          ${0}
-        "
-          rpy="0 0 0" />
-        <geometry>
-          <mesh
-            filename="package://spacediver_ros2_control/description/gazebo/models/meshes/upper_arm_driving_link.STL" />
-        </geometry>
-      </collision>
-      <xacro:inertial_box mass="${LINK_1_MASS}" x="${LINK_1_X/2}" y="${LINK_1_Y/2}"
-        z="${LINK_1_Z/2}">
-        <origin xyz="0 0 ${LINK_1_Z/2}" rpy="0 0 0" />
-      </xacro:inertial_box>
+      <inertial>
+        <origin xyz="0 0 0" rpy="0 0 0" />
+        <mass value="1.0" />
+        <inertia ixx="0.01" ixy="0.0" ixz="0.0" iyy="0.01" iyz="0.0" izz="0.01" />
+      </inertial>
     </link>
   </xacro:macro>

File: spacediver_ros2_control/description/urdf/spacediver.urdf.xacro (robot description, xacro)
@@ -1,11 +1,14 @@
-<robot name="single_arm_robot" xmlns:xacro="http://ros.org/wiki/xacro">
+<robot name="dual_arm_robot" xmlns:xacro="http://ros.org/wiki/xacro">
   <!-- Include macros -->
   <xacro:include
     filename="$(find spacediver_ros2_control)/description/urdf/macros/inertial_macros.xacro" />
-  <xacro:include filename="$(find spacediver_ros2_control)/description/urdf/macros/properties.xacro" />
-  <xacro:include filename="$(find spacediver_ros2_control)/description/urdf/macros/materials.xacro" />
+  <xacro:include
+    filename="$(find spacediver_ros2_control)/description/urdf/macros/properties.xacro" />
+  <xacro:include
+    filename="$(find spacediver_ros2_control)/description/urdf/macros/materials.xacro" />
   <!-- Select if the robot is going to be used in gazebo -->
   <!-- This is set in spacediver.launch.py -->
   <xacro:arg name="use_gazebo" default="true" />
+  <xacro:arg name="single_arm" default="false" />
   <!-- robot shape and phisics -->
   <!-- Base Link -->
@@ -18,6 +21,14 @@
     <origin xyz="0 0 0" rpy="0 0 0" />
   </xacro:left_arm>
+  <!-- Right Arm -->
+  <xacro:unless value="$(arg single_arm)">
+    <xacro:include
+      filename="$(find spacediver_ros2_control)/description/urdf/parts/spacediver_right_arm.xacro" />
+    <xacro:right_arm base_name="base_link">
+      <origin xyz="0 0 0" rpy="0 0 0" />
+    </xacro:right_arm>
+  </xacro:unless>
   <!-- ros2 control plugin -->
   <xacro:include
-    filename="$(find spacediver_ros2_control)/description/ros2_control/spacediver_single_arm_ros2_control.xacro" />
+    filename="$(find spacediver_ros2_control)/description/ros2_control/spacediver_ros2_control.xacro" />
 </robot>

File: spacediver_ros2_control/description/urdf/spacediver_single_arm.urdf.xacro (robot description, xacro)
@@ -1,10 +1,8 @@
-<robot name="dual_arm_robot" xmlns:xacro="http://ros.org/wiki/xacro">
+<robot name="single_arm_robot" xmlns:xacro="http://ros.org/wiki/xacro">
   <!-- Include macros -->
   <xacro:include
     filename="$(find spacediver_ros2_control)/description/urdf/macros/inertial_macros.xacro" />
-  <xacro:include
-    filename="$(find spacediver_ros2_control)/description/urdf/macros/properties.xacro" />
-  <xacro:include
-    filename="$(find spacediver_ros2_control)/description/urdf/macros/materials.xacro" />
+  <xacro:include filename="$(find spacediver_ros2_control)/description/urdf/macros/properties.xacro" />
+  <xacro:include filename="$(find spacediver_ros2_control)/description/urdf/macros/materials.xacro" />
   <!-- Select if the robot is going to be used in gazebo -->
   <!-- This is set in spacediver.launch.py -->
@@ -20,12 +18,6 @@
     <origin xyz="0 0 0" rpy="0 0 0" />
   </xacro:left_arm>
-  <!-- Right Arm -->
-  <xacro:include
-    filename="$(find spacediver_ros2_control)/description/urdf/parts/spacediver_right_arm.xacro" />
-  <xacro:right_arm base_name="base_link">
-    <origin xyz="0 0 0" rpy="0 0 0" />
-  </xacro:right_arm>
   <!-- ros2 control plugin -->
   <xacro:include
-    filename="$(find spacediver_ros2_control)/description/ros2_control/spacediver_ros2_control.xacro" />
+    filename="$(find spacediver_ros2_control)/description/ros2_control/spacediver_single_arm_ros2_control.xacro" />
 </robot>
