Commit message: update xacros

File: spacediver_ros2_control/description/urdf/parts/spacediver_base.xacro (robot description, xacro)
@@ -2,6 +2,4 @@
 <!-- import xacro reffering here https://gbiggs.github.io/rosjp_urdf_tutorial_text/manipulator_urdf.html -->
 <robot xmlns:xacro="http://ros.org/wiki/xacro">
-  <xacro:include filename="$(find spacediver_ros2_control)/description/urdf/macros/inertial_macros.xacro"/>
-  <xacro:include filename="$(find spacediver_ros2_control)/description/urdf/macros/properties.xacro"/>
   <xacro:property name="BASE_LINK_NAME" value="base_link" />
   <link name="${BASE_LINK_NAME}">

File: spacediver_ros2_control/description/urdf/parts/spacediver_left_arm.xacro (robot description, xacro)
@@ -2,6 +2,4 @@
 <!-- import xacro reffering here https://gbiggs.github.io/rosjp_urdf_tutorial_text/manipulator_urdf.html -->
 <robot xmlns:xacro="http://ros.org/wiki/xacro">
-  <xacro:include filename="$(find spacediver_ros2_control)/description/urdf/macros/inertial_macros.xacro"/>
-  <xacro:include filename="$(find spacediver_ros2_control)/description/urdf/macros/properties.xacro"/>
   <xacro:macro name="left_arm" params="base_name *origin">
     <!-- Active joint 1 -->
@@ -38,5 +36,5 @@
       <child link="link_2"/>
       <origin xyz="0 0 ${LINK_1_Z}" rpy="0 0 0"/>
-      <axis xyz="0 1 0"/>
+      <axis xyz="0 0 1"/>
       <limit lower="${ACTIVE_JOINT_LB_LOWER}" upper="${ACTIVE_JOINT_LB_UPPER}"
         effort="${ACTIVE_JOINT_LB_EFFORT}" velocity="${ACTIVE_JOINT_LB_VELOCITY}"/>
@@ -66,5 +64,5 @@
       <child link="link_3"/>
       <origin xyz="${LINK_2_X} 0 0" rpy="0 0 0"/>
-      <axis xyz="0 1 0"/>
+      <axis xyz="0 0 1"/>
       <limit lower="${ACTIVE_JOINT_LC_LOWER}" upper="${ACTIVE_JOINT_LC_UPPER}"
         effort="${ACTIVE_JOINT_LC_EFFORT}" velocity="${ACTIVE_JOINT_LC_VELOCITY}"/>

File: spacediver_ros2_control/description/urdf/spacediver.urdf.xacro (robot description, xacro)
@@ -2,4 +2,5 @@
   <xacro:include filename="$(find spacediver_ros2_control)/description/urdf/macros/inertial_macros.xacro"/>
   <xacro:include filename="$(find spacediver_ros2_control)/description/urdf/macros/properties.xacro"/>
+  <xacro:include filename="$(find spacediver_ros2_control)/description/urdf/macros/materials.xacro"/>
   <!-- robot shape and phisics -->
   <!-- Base Link -->
@@ -8,5 +9,5 @@
   <xacro:include filename="$(find spacediver_ros2_control)/description/urdf/parts/spacediver_left_arm.xacro" />
   <xacro:left_arm base_name="${BASE_LINK_NAME}">
-    <origin xyz="0 0 ${BASE_Z}" rpy="0 0 0"/>
+    <origin xyz="0 0 ${BASE_Z/2}" rpy="0 0 0"/>
   </xacro:left_arm>
   <!-- gazebo pulgin -->

Commit message: WIP urdf single arm

File: spacediver_ros2_control/description/urdf/parts/spacediver_base.xacro (robot description, xacro)
@@ -2,5 +2,5 @@
 <!-- import xacro reffering here https://gbiggs.github.io/rosjp_urdf_tutorial_text/manipulator_urdf.html -->
 <robot xmlns:xacro="http://ros.org/wiki/xacro">
-  <link name="base_link">
+  <link name="${BASE_LINK_NAME}">
     <visual>
       <origin xyz="0 0 0" rpy="0 0 0"/>
@@ -8,5 +8,5 @@
         <box size="${BASE_X} ${BASE_Y} ${BASE_Z}"/>
       </geometry>
-      <material name="white"/>
+      <material name="black"/>
     </visual>
     <collision>

File: spacediver_ros2_control/description/urdf/parts/spacediver_left_arm.xacro (robot description, xacro)
@@ -3,88 +3,267 @@
 <robot xmlns:xacro="http://ros.org/wiki/xacro">
   <xacro:macro name="left_arm" params="base_name *origin">
-    <!-- Active joint 1 -->
-    <joint name="active_joint_la" type="revolute">
-      <parent link="${base_name}"/>
-      <child link="link_1"/>
-      <xacro:insert_block name="origin"/>
-      <axis xyz="0 0 1"/>
-      <limit lower="${ACTIVE_JOINT_LA_LOWER}" upper="${ACTIVE_JOINT_LA_UPPER}"
-        effort="${ACTIVE_JOINT_LA_EFFORT}" velocity="${ACTIVE_JOINT_LA_VELOCITY}"/>
-    </joint>
-    <!-- Link 1 -->
-    <link name="link_1">
-      <visual>
-        <origin xyz="0 0 ${LINK_1_Z/2}" rpy="0 0 0"/>
-        <geometry>
-          <box size="${LINK_1_X} ${LINK_1_Y} ${LINK_1_Z}"/>
-        </geometry>
-        <material name="white"/>
-      </visual>
-      <collision>
-        <origin xyz="0 0 ${LINK_1_Z/2}" rpy="0 0 0"/>
-        <geometry>
-          <box size="${LINK_1_X} ${LINK_1_Y} ${LINK_1_Z}"/>
-        </geometry>
-      </collision>
-      <xacro:inertial_box mass="${LINK_1_MASS}" x="${LINK_1_X/2}" y="${LINK_1_Y/2}" z="${LINK_1_Z/2}">
-        <origin xyz="0 0 ${LINK_1_Z/2}" rpy="0 0 0"/>
-      </xacro:inertial_box>
-    </link>
-    <!-- Joint 2 -->
-    <joint name="active_joint_lb" type="revolute">
-      <parent link="link_1"/>
-      <child link="link_2"/>
-      <origin xyz="0 0 ${LINK_1_Z}" rpy="0 0 0"/>
-      <axis xyz="0 0 1"/>
-      <limit lower="${ACTIVE_JOINT_LB_LOWER}" upper="${ACTIVE_JOINT_LB_UPPER}"
-        effort="${ACTIVE_JOINT_LB_EFFORT}" velocity="${ACTIVE_JOINT_LB_VELOCITY}"/>
-    </joint>
-    <!-- Link 2 -->
-    <link name="link_2">
-      <visual>
-        <origin xyz="${LINK_2_X/2} 0 0" rpy="0 0 0"/>
-        <geometry>
-          <box size="${LINK_2_X} ${LINK_2_Y} ${LINK_2_Z}"/>
-        </geometry>
-        <material name="white"/>
-      </visual>
-      <collision>
-        <origin xyz="${LINK_2_X/2} 0 0" rpy="0 0 0"/>
-        <geometry>
-          <box size="${LINK_2_X} ${LINK_2_Y} ${LINK_2_Z}"/>
-        </geometry>
-      </collision>
-      <xacro:inertial_box mass="${LINK_2_MASS}" x="${LINK_2_X/2}" y="${LINK_2_Y/2}" z="${LINK_2_Z/2}">
-        <origin xyz="${LINK_2_X/2} 0 0" rpy="0 0 0"/>
-      </xacro:inertial_box>
-    </link>
-    <!-- Joint 3 -->
-    <joint name="active_joint_lc" type="revolute">
-      <parent link="link_2"/>
-      <child link="link_3"/>
-      <origin xyz="${LINK_2_X} 0 0" rpy="0 0 0"/>
-      <axis xyz="0 0 1"/>
-      <limit lower="${ACTIVE_JOINT_LC_LOWER}" upper="${ACTIVE_JOINT_LC_UPPER}"
-        effort="${ACTIVE_JOINT_LC_EFFORT}" velocity="${ACTIVE_JOINT_LC_VELOCITY}"/>
-    </joint>
-    <!-- Link 3 -->
-    <link name="link_3">
-      <visual>
-        <origin xyz="${LINK_3_X/2} 0 0" rpy="0 0 0"/>
-        <geometry>
-          <box size="${LINK_3_X} ${LINK_3_Y} ${LINK_3_Z}"/>
-        </geometry>
-        <material name="white"/>
-      </visual>
-      <collision>
-        <origin xyz="${LINK_3_X/2} 0 0" rpy="0 0 0"/>
-        <geometry>
-          <box size="${LINK_3_X} ${LINK_3_Y} ${LINK_3_Z}"/>
-        </geometry>
-      </collision>
-      <xacro:inertial_box mass="${LINK_3_MASS}" x="${LINK_3_X/2}" y="${LINK_3_Y/2}" z="${LINK_3_Z/2}">
-        <origin xyz="${LINK_3_X/2} 0 0" rpy="0 0 0"/>
-      </xacro:inertial_box>
-    </link>
+    <!-- BASE TO SHOULDER -->
+    <joint name="${BASE_TO_LEFTSHOULDER_JOINT_NAME}" type="revolute">
+      <parent link="${BASE_LINK_NAME}"/>
+      <child link="${L_SHOULDER_LINK_NAME}"/>
+      <origin xyz="
+        ${SHOULDER_POS_X}
+        ${-(SHOULDER_JOINTA_X-SHOULDER_Y/2)}
+        ${0}
+      " rpy="0 0 0"/>
+      <axis xyz="1 0 0"/>
+      <limit lower="${BASE_DYNAMIXEL_LOWER}" upper="${BASE_DYNAMIXEL_UPPER}"
+        effort="${BASE_DYNAMIXEL_EFFORT}" velocity="${BASE_DYNAMIXEL_VELOCITY}"/>
+    </joint>
+    <!-- SHOULDER -->
+    <link name="${L_SHOULDER_LINK_NAME}">
+      <visual>
+        <origin xyz="
+          ${0}
+          ${SHOULDER_JOINTA_X}
+          ${-SHOULDER_Z/2}
+        " rpy="0 0 ${L_SHOULDER_ROT_Z}"/>
+        <geometry>
+          <mesh filename="package://spacediver_ros2_control/description/gazebo/models/meshes/shoulder_plate.STL"/>
+        </geometry>
+        <material name="grey"/>
+      </visual>
+      <collision>
+        <origin xyz="${SHOULDER_X/2} ${SHOULDER_Y/2} ${SHOULDER_Z/2}" rpy="0 0 0"/>
+        <geometry>
+          <mesh filename="package://spacediver_ros2_control/description/gazebo/models/meshes/shoulder_plate.STL"/>
+        </geometry>
+      </collision>
+      <xacro:inertial_box mass="${LINK_1_MASS}" x="${LINK_1_X/2}" y="${LINK_1_Y/2}" z="${LINK_1_Z/2}">
+        <origin xyz="0 0 ${LINK_1_Z/2}" rpy="0 0 0"/>
+      </xacro:inertial_box>
+    </link>
+    <!-- SHOULDER TO BOTTOM DYNAMIXEL -->
+    <joint name="${LEFTSHOULDER_TO_LEFTDYNAMIXELBOT_JOINT_NAME}" type="fixed">
+      <parent link="${L_SHOULDER_LINK_NAME}"/>
+      <child link="${L_BOT_DYNAMIXEL_LINK_NAME}"/>
+      <origin xyz="
+        ${SHOULDER_X + DYNAMIXEL_X/2}
+        ${SHOULDER_JOINTA_X - DYNAMIXEL_Y/2}
+        ${-SHOULDER_Z/2 + DYNAMIXEL_Z/2}
+      "
+        rpy="0 0 0"/>
+      <axis xyz="0 0 1"/>
+    </joint>
+    <!-- BOTTOM DYNAMIXEL -->
+    <link name="${L_BOT_DYNAMIXEL_LINK_NAME}">
+      <visual>
+        <origin xyz="0 0 0" rpy="0 0 0"/>
+        <geometry>
+          <box size="${DYNAMIXEL_X} ${DYNAMIXEL_Y} ${DYNAMIXEL_Z}"/>
+        </geometry>
+        <material name="blue"/>
+      </visual>
+      <collision>
+        <origin xyz="0 0 0" rpy="0 0 0"/>
+        <geometry>
+          <box size="${DYNAMIXEL_X} ${DYNAMIXEL_Y} ${DYNAMIXEL_Z}"/>
+        </geometry>
+      </collision>
+      <xacro:inertial_box mass="${LINK_1_MASS}" x="${LINK_1_X/2}" y="${LINK_1_Y/2}" z="${LINK_1_Z/2}">
+        <origin xyz="0 0 ${LINK_1_Z/2}" rpy="0 0 0"/>
+      </xacro:inertial_box>
+    </link>
+    <!-- BOTTOM DYNAMIXEL TO MISUMI LN -->
+    <joint name="${LEFT_DYNAMIXELBOT_TO_LEFTMISUMILN_JOINT_NAME}" type="revolute">
+      <parent link="${L_BOT_DYNAMIXEL_LINK_NAME}"/>
+      <child link="${L_MISUMILN_LINK_NAME}"/>
+      <origin xyz="
+        ${0}
+        ${DYNAMIXEL_JOINTB_Y-DYNAMIXEL_Y/2}
+        ${MISUMILN_POS_Z-DYNAMIXEL_BOT_POS_Z}"
+        rpy="0 0 0"/>
+      <axis xyz="0 0 1"/>
+      <limit lower="${BOT_DYNAMIXEL_LOWER}" upper="${BOT_DYNAMIXEL_UPPER}"
+        effort="${BOT_DYNAMIXEL_EFFORT}" velocity="${BOT_DYNAMIXEL_VELOCITY}"/>
+    </joint>
+    <!-- MISUMI LN -->
+    <link name="${L_MISUMILN_LINK_NAME}">
+      <visual>
+        <origin xyz="
+          ${L_MISUMILN_POS_X-DYNAMIXEL_POS_X}
+          ${L_MISUMILN_POS_Y+DYNAMIXEL_JOINTB_Y-DYNAMIXEL_POS_Y}
+          0
+        " rpy="0 0 ${L_MISUMILN_ROT_Z}"/>
+        <geometry>
+          <mesh filename="package://spacediver_ros2_control/description/gazebo/models/meshes/Link_MISUMI_LNMS16-10-200.STL"/>
+        </geometry>
+        <material name="blue"/>
+      </visual>
+      <collision>
+        <origin xyz="0 0 0" rpy="0 0 0"/>
+        <geometry>
+          <mesh filename="package://spacediver_ros2_control/description/gazebo/models/meshes/Link_MISUMI_LNMS16-10-200.STL"/>
+        </geometry>
+      </collision>
+      <xacro:inertial_box mass="${LINK_1_MASS}" x="${LINK_1_X/2}" y="${LINK_1_Y/2}" z="${LINK_1_Z/2}">
+        <origin xyz="0 0 ${LINK_1_Z/2}" rpy="0 0 0"/>
+      </xacro:inertial_box>
+    </link>
+    <!-- SHOULDER TO TOP DYNAMIXEL -->
+    <joint name="${LEFTSHOULDER_TO_LEFTDYNAMIXELTOP_JOINT_NAME}" type="fixed">
+      <parent link="${L_SHOULDER_LINK_NAME}"/>
+      <child link="${L_TOP_DYNAMIXEL_LINK_NAME}"/>
+      <origin xyz="
+          ${SHOULDER_X + DYNAMIXEL_X/2}
+          ${SHOULDER_JOINTA_X - DYNAMIXEL_Y/2}
+          ${SHOULDER_Z/2 - DYNAMIXEL_Z/2}
+        "
+        rpy="0 0 0"/>
+      <axis xyz="0 0 1"/>
+    </joint>
+    <!-- TOP DYNAMIXEL -->
+    <link name="${L_TOP_DYNAMIXEL_LINK_NAME}">
+      <visual>
+        <origin xyz="0 0 0" rpy="0 0 0"/>
+        <geometry>
+          <box size="${DYNAMIXEL_X} ${DYNAMIXEL_Y} ${DYNAMIXEL_Z}"/>
+        </geometry>
+        <material name="blue"/>
+      </visual>
+      <collision>
+        <origin xyz="0 0 0" rpy="0 0 0"/>
+        <geometry>
+          <box size="${DYNAMIXEL_X} ${DYNAMIXEL_Y} ${DYNAMIXEL_Z}"/>
+        </geometry>
+      </collision>
+      <xacro:inertial_box mass="${LINK_1_MASS}" x="${LINK_1_X/2}" y="${LINK_1_Y/2}" z="${LINK_1_Z/2}">
+        <origin xyz="0 0 ${LINK_1_Z/2}" rpy="0 0 0"/>
+      </xacro:inertial_box>
+    </link>
+    <!-- TOP DYNAMIXEL TO DRIVING LINK -->
+    <joint name="${LEFTDYNAMIXELTOP_TO_LEFTDRIVING_JOINT_NAME}" type="revolute">
+      <parent link="${L_TOP_DYNAMIXEL_LINK_NAME}"/>
+      <child link="${L_DRIVING_LINK_NAME}"/>
+      <origin xyz="
+        ${0}
+        ${DYNAMIXEL_JOINTB_Y-DYNAMIXEL_Y/2}
+        ${DRIVING_POS_Z - DYNAMIXEL_TOP_POS_Z}"
+        rpy="0 0 ${0}"/>
+      <axis xyz="0 0 1"/>
+      <limit lower="${TOP_DYNAMIXEL_LOWER}" upper="${TOP_DYNAMIXEL_UPPER}"
+        effort="${TOP_DYNAMIXEL_EFFORT}" velocity="${TOP_DYNAMIXEL_VELOCITY}"/>
+    </joint>
+    <!-- DRIVING LINK -->
+    <link name="${L_DRIVING_LINK_NAME}">
+      <visual>
+        <origin xyz="
+          ${-DRIVING_JOINTA_X}
+          ${-DRIVING_JOINTA_Y}
+          ${0}
+        " rpy="0 0 0"/>
+        <geometry>
+          <mesh filename="package://spacediver_ros2_control/description/gazebo/models/meshes/upper_arm_driving_link.STL"/>
+        </geometry>
+        <material name="blue"/>
+      </visual>
+      <collision>
+        <origin xyz="0 0 0" rpy="0 0 0"/>
+        <geometry>
+          <mesh filename="package://spacediver_ros2_control/description/gazebo/models/meshes/upper_arm_driving_link.STL"/>
+        </geometry>
+      </collision>
+      <xacro:inertial_box mass="${LINK_1_MASS}" x="${LINK_1_X/2}" y="${LINK_1_Y/2}" z="${LINK_1_Z/2}">
+        <origin xyz="0 0 ${LINK_1_Z/2}" rpy="0 0 0"/>
+      </xacro:inertial_box>
+    </link>
+    <!-- DRIVING LINK TO DRIVEN LINK-->
+    <joint name="${LEFTDRIVING_TO_LEFTDRIVEN_JOINT_NAME}" type="revolute">
+      <parent link="${L_DRIVING_LINK_NAME}"/>
+      <child link="${L_DRIVEN_LINK_NAME}"/>
+      <origin xyz="
+        ${DRIVING_JOINTB_X-DRIVING_JOINTA_X}
+        ${0}
+        ${DRIVEN_POS_Z - DRIVING_POS_Z - DRIVING_Z}
+      "
+        rpy="0 0 ${0}"/>
+      <axis xyz="0 0 1"/>
+      <limit lower="${TOP_DYNAMIXEL_LOWER}" upper="${TOP_DYNAMIXEL_UPPER}"
+        effort="${TOP_DYNAMIXEL_EFFORT}" velocity="${TOP_DYNAMIXEL_VELOCITY}"/>
+    </joint>
+    <!-- DRIVEN LINK -->
+    <link name="${L_DRIVEN_LINK_NAME}">
+      <visual>
+        <origin xyz="
+          ${L_DRIVEN_POS_X - (L_DRIVING_POS_X + DRIVING_JOINTB_X)}
+          ${L_DRIVEN_POS_Y - (L_DRIVING_POS_Y + DRIVING_JOINTB_Y)}
+          ${0}
+        " rpy="0 0 ${L_DRIVEN_ROT_Z}"/>
+        <geometry>
+          <mesh filename="package://spacediver_ros2_control/description/gazebo/models/meshes/upper_arm_driven_link.STL"/>
+        </geometry>
+        <material name="blue"/>
+      </visual>
+      <collision>
+        <origin xyz="0 0 0" rpy="0 0 0"/>
+        <geometry>
+          <mesh filename="package://spacediver_ros2_control/description/gazebo/models/meshes/upper_arm_driven_link.STL"/>
+        </geometry>
+      </collision>
+      <xacro:inertial_box mass="${LINK_1_MASS}" x="${LINK_1_X/2}" y="${LINK_1_Y/2}" z="${LINK_1_Z/2}">
+        <origin xyz="0 0 ${LINK_1_Z/2}" rpy="0 0 0"/>
+      </xacro:inertial_box>
+    </link>
+    <!-- MISUMI FT -->
+    <link name="${L_MISUMIFT_LINK_NAME}">
+      <visual>
+        <origin xyz="
+          ${0}
+          ${0}
+          ${0}
+        " rpy="0 0 ${L_MISUMIFT_ROT_Z}"/>
+        <geometry>
+          <mesh filename="package://spacediver_ros2_control/description/gazebo/models/meshes/Misumi_LNFTS10-P10-V10-L200-S50-W18-T9.STL"/>
+        </geometry>
+        <material name="blue"/>
+      </visual>
+      <collision>
+        <origin xyz="0 0 0" rpy="0 0 0"/>
+        <geometry>
+          <mesh filename="package://spacediver_ros2_control/description/gazebo/models/meshes/Misumi_LNFTS10-P10-V10-L200-S50-W18-T9.STL"/>
+        </geometry>
+      </collision>
+      <xacro:inertial_box mass="${LINK_1_MASS}" x="${LINK_1_X/2}" y="${LINK_1_Y/2}" z="${LINK_1_Z/2}">
+        <origin xyz="0 0 ${LINK_1_Z/2}" rpy="0 0 0"/>
+      </xacro:inertial_box>
+    </link>
+<!--
+      ${L_MISUMIFT_POS_X - (L_DRIVEN_POS_X + MISUMIFT_JOINTA_X) + (L_DRIVEN_POS_X - (L_DRIVING_POS_X + DRIVING_JOINTB_X))}
+        ${L_MISUMIFT_POS_Y - (L_DRIVEN_POS_Y + MISUMIFT_JOINTA_Y) + (L_DRIVEN_POS_Y - (L_DRIVING_POS_Y + DRIVING_JOINTB_Y))}
+        ${0}
+     -->
+    <!-- DRIVEN LINK TO MISUMI FT -->
+    <joint name="${LEFTDRIVEN_TO_LEFTMISUMIFT_JOINT_NAME}" type="revolute">
+      <parent link="${L_DRIVEN_LINK_NAME}"/>
+      <child link="${L_MISUMIFT_LINK_NAME}"/>
+      <origin xyz="
+        ${L_MISUMIFT_POS_X - (L_DRIVEN_POS_X + MISUMIFT_JOINTA_X) + (L_DRIVEN_POS_X - (L_DRIVING_POS_X + DRIVING_JOINTB_X))}
+        ${L_MISUMIFT_POS_Y - (L_DRIVEN_POS_Y + MISUMIFT_JOINTA_Y) + (L_DRIVEN_POS_Y - (L_DRIVING_POS_Y + DRIVING_JOINTB_Y))}
+        ${0}
+      "
+        rpy="0 0 ${0}"/>
+      <axis xyz="0 0 1"/>
+      <limit lower="${TOP_DYNAMIXEL_LOWER}" upper="${TOP_DYNAMIXEL_UPPER}"
+        effort="${TOP_DYNAMIXEL_EFFORT}" velocity="${TOP_DYNAMIXEL_VELOCITY}"/>
+    </joint>
+    <!-- MISUMI LN TO MISUMI FT -->
+    <!-- <joint name="${LEFTMISUMILN_TO_LEFTMISUMIFT_JOINT_NAME}" type="revolute">
+      <parent link="${L_MISUMILN_LINK_NAME}"/>
+      <child link="${L_MISUMIFT_LINK_NAME}"/>
+      <origin xyz="
+        ${0}
+        ${0}
+        ${0}
+      "
+        rpy="0 0 ${0}"/>
+      <axis xyz="0 0 1"/>
+      <limit lower="${TOP_DYNAMIXEL_LOWER}" upper="${TOP_DYNAMIXEL_UPPER}"
+        effort="${TOP_DYNAMIXEL_EFFORT}" velocity="${TOP_DYNAMIXEL_VELOCITY}"/>
+    </joint> -->
   </xacro:macro>
 </robot>

Commit message: give base inertia only for gazebo

File: spacediver_ros2_control/description/urdf/parts/spacediver_base.xacro (robot description, xacro)
@@ -16,7 +16,9 @@
       </geometry>
     </collision>
-    <!-- <xacro:inertial_box mass="${BASE_MASS}" x="${BASE_X/2}" y="${BASE_Y/2}" z="${BASE_Z/2}">
-      <origin xyz="0 0 0" rpy="0 0 0"/>
-    </xacro:inertial_box> -->
+    <xacro:if value="$(arg use_gazebo)">
+      <xacro:inertial_box mass="${BASE_MASS}" x="${BASE_X/2}" y="${BASE_Y/2}" z="${BASE_Z/2}">
+        <origin xyz="0 0 0" rpy="0 0 0"/>
+      </xacro:inertial_box>
+    </xacro:if>
   </link>
 </robot>

Commit message: updated base urdf xacro

File: spacediver_ros2_control/description/urdf/parts/spacediver_base.xacro (robot description, xacro)
@@ -10,15 +10,9 @@
       <material name="black"/>
     </visual>
-    <collision>
-      <origin xyz="0 0 0" rpy="0 0 0"/>
-      <geometry>
-        <box size="${BASE_X} ${BASE_Y} ${BASE_Z}"/>
-      </geometry>
-    </collision>
-    <xacro:if value="$(arg use_gazebo)">
-      <xacro:inertial_box mass="${BASE_MASS}" x="${BASE_X/2}" y="${BASE_Y/2}" z="${BASE_Z/2}">
-        <origin xyz="0 0 0" rpy="0 0 0"/>
-      </xacro:inertial_box>
-    </xacro:if>
+    <inertial>
+      <origin xyz="0 0 0" rpy="0 0 0" />
+      <mass value="${BASE_MASS}" />
+      <inertia ixx="0.0" ixy="0.0" ixz="0.0" iyy="0.0" iyz="0.0" izz="0.0" />
+    </inertial>
   </link>
 </robot>

Commit message: updated base

File: spacediver_ros2_control/description/urdf/parts/spacediver_base.xacro (robot description, xacro)
@@ -13,5 +13,8 @@
       <origin xyz="0 0 0" rpy="0 0 0" />
       <mass value="${BASE_MASS}" />
-      <inertia ixx="0.0" ixy="0.0" ixz="0.0" iyy="0.0" iyz="0.0" izz="0.0" />
+      <inertia
+        ixx="${1/12*BASE_MASS*(BASE_Y**2+BASE_Z**2)}" ixy="0.0" ixz="0.0"
+        iyy="${1/12*BASE_MASS*(BASE_X**2+BASE_Z**2)}" iyz="0.0"
+        izz="${1/12*BASE_MASS*(BASE_X**2+BASE_Y**2)}" />
     </inertial>
   </link>
