Commit message: shifted misumi ln because of corrected mesh file

File: spacediver_ros2_control/description/urdf/macros/properties.xacro (robot description, xacro)
@@ -45,5 +45,5 @@
   <xacro:property name="R_MISUMILN_POS_X" value="${-DYNAMIXEL_POS_X + math.cos(-ROT)*(-MISUMILN_JOINTA_X) - math.sin(-ROT)*(MISUMILN_JOINTA_Y)}"/>
   <xacro:property name="R_MISUMILN_POS_Y" value="${DYNAMIXEL_POS_Y - DYNAMIXEL_JOINTB_Y + math.sin(-ROT)*(-MISUMILN_JOINTA_X) + math.cos(-ROT)*(MISUMILN_JOINTA_Y)}"/>
-  <xacro:property name="MISUMILN_POS_Z" value="${DYNAMIXEL_BOT_POS_Z + DYNAMIXEL_Z/2 + 0.0045}"/>
+  <xacro:property name="MISUMILN_POS_Z" value="${DYNAMIXEL_BOT_POS_Z + DYNAMIXEL_Z/2 + 0.0145}"/>
   <!-- DRIVING LINK -->
   <xacro:property name="DRIVING_X" value="0.076"/>

Commit message: added link and joint names to properties.xacro

File: spacediver_ros2_control/description/urdf/macros/properties.xacro (robot description, xacro)
@@ -4,4 +4,37 @@
   <xacro:property name="ROT" value="${PI/6}"/>
   <xacro:property name="RPM" value="30"/>
+  <!-- LINK NAMES -->
+  <xacro:property name="BASE_LINK_NAME" value="base_link"/>
+  <xacro:property name="L_SHOULDER_LINK_NAME" value="left_shoulder_link"/>
+  <xacro:property name="R_SHOULDER_LINK_NAME" value="right_shoulder_link"/>
+  <xacro:property name="L_TOP_DYNAMIXEL_LINK_NAME" value="left_dynamixel_top"/>
+  <xacro:property name="R_TOP_DYNAMIXEL_LINK_NAME" value="right_dynamixel_top"/>
+  <xacro:property name="L_BOT_DYNAMIXEL_LINK_NAME" value="left_dynamixel_bottom"/>
+  <xacro:property name="R_BOT_DYNAMIXEL_LINK_NAME" value="right_dynamixel_bottom"/>
+  <xacro:property name="L_MISUMILN_LINK_NAME" value="left_misumi_ln"/>
+  <xacro:property name="R_MISUMILN_LINK_NAME" value="right_misumi_ln"/>
+  <xacro:property name="L_DRIVING_LINK_NAME" value="left_driving_link"/>
+  <xacro:property name="R_DRIVING_LINK_NAME" value="right_driving_link"/>
+  <xacro:property name="L_DRIVEN_LINK_NAME" value="left_driven_link"/>
+  <xacro:property name="R_DRIVEN_LINK_NAME" value="right_driven_link"/>
+  <xacro:property name="L_MISUMIFT_LINK_NAME" value="left_misumi_ft"/>
+  <xacro:property name="R_MISUMIFT_LINK_NAME" value="right_misumi_ft"/>
+  <!-- JOINT NAMES -->
+  <xacro:property name="BASE_TO_LEFTSHOULDER_JOINT_NAME" value="base_to_leftshoulder_joint"/>
+  <xacro:property name="BASE_TO_RIGHTSHOULDER_JOINT_NAME" value="base_to_rightshoulder_joint"/>
+  <xacro:property name="LEFTSHOULDER_TO_LEFTDYNAMIXELTOP_JOINT_NAME" value="leftshoulder_to_leftdynamixeltop_joint"/>
+  <xacro:property name="RIGHTSHOULDER_TO_RIGHTDYNAMIXELTOP_JOINT_NAME" value="rightshoulder_to_rightdynamixeltop_joint"/>
+  <xacro:property name="LEFTSHOULDER_TO_LEFTDYNAMIXELBOT_JOINT_NAME" value="leftshoulder_to_leftdynamixelbottom_joint"/>
+  <xacro:property name="RIGHTSHOULDER_TO_RIGHTDYNAMIXELBOT_JOINT_NAME" value="rightshoulder_to_rightdynamixelbottom_joint"/>
+  <xacro:property name="LEFT_DYNAMIXELBOT_TO_LEFTMISUMILN_JOINT_NAME" value="leftdynamixelbottom_to_leftmisumiln_joint"/>
+  <xacro:property name="RIGHT_DYNAMIXELBOT_TO_RIGHTMISUMILN_JOINT_NAME" value="rightdynamixelbottom_to_rightmisumiln_joint"/>
+  <xacro:property name="LEFTDYNAMIXELTOP_TO_LEFTDRIVING_JOINT_NAME" value="leftdynamixeltop_to_leftdriving_joint"/>
+  <xacro:property name="RIGHTDYNAMIXELTOP_TO_RIGHTDRIVING_JOINT_NAME" value="rightdynamixeltop_to_rightdriving_joint"/>
+  <xacro:property name="LEFTDRIVING_TO_LEFTDRIVEN_JOINT_NAME" value="leftdriving_to_leftdriven_joint"/>
+  <xacro:property name="RIGHTDRIVING_TO_RIGHTDRIVEN_JOINT_NAME" value="rightdriving_to_rightdriven_joint"/>
+  <xacro:property name="LEFTDRIVEN_TO_LEFTMISUMIFT_JOINT_NAME" value="leftdriven_to_leftmisumift_joint"/>
+  <xacro:property name="RIGHTDRIVEN_TO_RIGHTMISUMIFT_JOINT_NAME" value="rightdriven_to_rightmisumift_joint"/>
+  <xacro:property name="LEFTMISUMILN_TO_LEFTMISUMIFT_JOINT_NAME" value="leftmisumiln_to_leftmisumift_joint"/>
+  <xacro:property name="RIGHTMISUMILN_TO_RIGHTMISUMIFT_JOINT_NAME" value="rightmisumiln_to_rightmisumift_joint"/>
   <!-- BASE -->
   <xacro:property name="BASE_X" value="0.18"/>

Commit message: updated left arm urdf with meshes

File: spacediver_ros2_control/description/urdf/macros/properties.xacro (robot description, xacro)
@@ -41,5 +41,5 @@
   <xacro:property name="BASE_Y" value="0.0585"/>
   <xacro:property name="BASE_Z" value="0.0415"/>
-  <xacro:property name="BASE_MASS" value="50"/>
+  <xacro:property name="BASE_MASS" value="10000"/>
   <xacro:property name="BASE_INERTIA_Z" value="0.13526810"/>
   <!-- JOINT -->
@@ -91,4 +91,5 @@
   <xacro:property name="MISUMILN_JOINTA_Y" value="0.012"/>
   <xacro:property name="MISUMILN_JOINTA_Z" value="${MISUMILN_Z/2}"/>
+  <xacro:property name="MISUMILN_JOINTB_Y" value="0.2"/>
   <!-- LEFT -->
   <xacro:property name="L_MISUMILN_ROT_Z" value="${-PI/2+ROT}"/>

File: spacediver_ros2_control/description/urdf/parts/spacediver_left_arm.xacro (robot description, xacro)
@@ -4,18 +4,13 @@
 <robot xmlns:xacro="http://ros.org/wiki/xacro">
   <xacro:macro name="left_arm" params="base_name *origin">
-    <!-- BASE TO SHOULDER -->
+    <!-- Joint 1 -->
     <joint name="${BASE_TO_LEFTSHOULDER_JOINT_NAME}" type="revolute">
       <parent link="${BASE_LINK_NAME}" />
       <child link="${L_SHOULDER_LINK_NAME}" />
       <origin
-        xyz="
-        ${SHOULDER_POS_X}
-        ${-(SHOULDER_JOINTA_X-SHOULDER_Y/2)}
-        ${0}
-      "
-        rpy="0 0 0" />
-      <axis xyz="1 0 0" />
-      <limit lower="${BASE_DYNAMIXEL_LOWER}" upper="${BASE_DYNAMIXEL_UPPER}"
-        effort="${BASE_DYNAMIXEL_EFFORT}" velocity="${BASE_DYNAMIXEL_VELOCITY}" />
+        xyz="${-SHOULDER_POS_X} ${SHOULDER_JOINTA_X-SHOULDER_Y/2} 0"
+        rpy="0 ${-PI/2} 0" />
+      <axis xyz="0 0 1" />
+      <limit lower="-1.57" upper="1.57" effort="10" velocity="1" />
     </joint>
     <!-- SHOULDER -->
@@ -23,82 +18,28 @@
       <visual>
         <origin
-          xyz="
-          ${0}
-          ${SHOULDER_JOINTA_X}
-          ${-SHOULDER_Z/2}
-        "
-          rpy="0 0 ${L_SHOULDER_ROT_Z}" />
+          xyz="${-SHOULDER_Z/2} ${-SHOULDER_JOINTA_X} 0"
+          rpy="${PI/2} 0 ${PI/2}" />
         <geometry>
           <mesh
             filename="package://spacediver_ros2_control/description/gazebo/models/meshes/shoulder_plate.STL" />
         </geometry>
-        <material name="grey" />
       </visual>
-      <collision>
-        <origin
-          xyz="
-          ${0}
-          ${SHOULDER_JOINTA_X}
-          ${-SHOULDER_Z/2}
-        "
-          rpy="0 0 ${L_SHOULDER_ROT_Z}" />
-        <geometry>
-          <mesh
-            filename="package://spacediver_ros2_control/description/gazebo/models/meshes/shoulder_plate.STL" />
-        </geometry>
-      </collision>
-      <xacro:inertial_box mass="${LINK_1_MASS}" x="${LINK_1_X/2}" y="${LINK_1_Y/2}"
-        z="${LINK_1_Z/2}">
-        <origin xyz="0 0 ${LINK_1_Z/2}" rpy="0 0 0" />
-      </xacro:inertial_box>
+      <inertial>
+        <origin xyz="0 0 0.25" rpy="0 0 0" />
+        <mass value="1.0" />
+        <inertia ixx="0.01" ixy="0.0" ixz="0.0" iyy="0.01" iyz="0.0" izz="0.01" />
+      </inertial>
     </link>
-    <!-- SHOULDER TO BOTTOM DYNAMIXEL -->
-    <joint name="${LEFTSHOULDER_TO_LEFTDYNAMIXELBOT_JOINT_NAME}" type="fixed">
+    <!-- Joint 2 -->
+    <joint name="${LEFT_DYNAMIXELBOT_TO_LEFTMISUMILN_JOINT_NAME}" type="revolute">
       <parent link="${L_SHOULDER_LINK_NAME}" />
-      <child link="${L_BOT_DYNAMIXEL_LINK_NAME}" />
-      <origin
-        xyz="
-        ${SHOULDER_X + DYNAMIXEL_X/2}
-        ${SHOULDER_JOINTA_X - DYNAMIXEL_Y/2}
-        ${-SHOULDER_Z/2 + DYNAMIXEL_Z/2}
-      "
-        rpy="0 0 0" />
-      <axis xyz="0 0 1" />
-    </joint>
-    <!-- BOTTOM DYNAMIXEL -->
-    <link name="${L_BOT_DYNAMIXEL_LINK_NAME}">
-      <visual>
-        <origin xyz="0 0 0" rpy="0 0 0" />
-        <geometry>
-          <box size="${DYNAMIXEL_X} ${DYNAMIXEL_Y} ${DYNAMIXEL_Z}" />
-        </geometry>
-        <material name="blue" />
-      </visual>
-      <collision>
-        <origin xyz="0 0 0" rpy="0 0 0" />
-        <geometry>
-          <box size="${DYNAMIXEL_X} ${DYNAMIXEL_Y} ${DYNAMIXEL_Z}" />
-        </geometry>
-      </collision>
-      <xacro:inertial_box mass="${LINK_1_MASS}" x="${LINK_1_X/2}" y="${LINK_1_Y/2}"
-        z="${LINK_1_Z/2}">
-        <origin xyz="0 0 ${LINK_1_Z/2}" rpy="0 0 0" />
-      </xacro:inertial_box>
-    </link>
-    <!-- BOTTOM DYNAMIXEL TO MISUMI LN -->
-    <joint name="${LEFT_DYNAMIXELBOT_TO_LEFTMISUMILN_JOINT_NAME}" type="revolute">
-      <parent link="${L_BOT_DYNAMIXEL_LINK_NAME}" />
       <child link="${L_MISUMILN_LINK_NAME}" />
       <origin
-        xyz="
-        ${0}
-        ${DYNAMIXEL_JOINTB_Y-DYNAMIXEL_Y/2}
-        ${MISUMILN_POS_Z-DYNAMIXEL_BOT_POS_Z}"
-        rpy="0 0 ${L_MISUMILN_ROT_Z}" />
+        xyz="${-SHOULDER_Z/2 + DYNAMIXEL_Z + 0.0145} 0 ${SHOULDER_X + DYNAMIXEL_X/2}"
+        rpy="${PI/2} ${-ROT} ${PI/2}" />
       <axis xyz="0 0 1" />
-      <limit lower="${BOT_DYNAMIXEL_LOWER}" upper="${BOT_DYNAMIXEL_UPPER}"
-        effort="${BOT_DYNAMIXEL_EFFORT}" velocity="${BOT_DYNAMIXEL_VELOCITY}" />
+      <limit lower="-1.57" upper="1.57" effort="10" velocity="1" />
     </joint>
-    <!-- MISUMI LN -->
+    <!-- FIRST LINK -->
     <link name="${L_MISUMILN_LINK_NAME}">
       <visual>
@@ -110,100 +51,44 @@
             filename="package://spacediver_ros2_control/description/gazebo/models/meshes/Link_MISUMI_LNMS16-10-200.STL" />
         </geometry>
-        <material name="blue" />
+        <material name="green">
+          <color rgba="0 1 0 1" />
+        </material>
       </visual>
-      <collision>
+      <inertial>
+        <origin xyz="0 0 0.1" rpy="0 0 0" />
+        <mass value="1.0" />
+        <inertia ixx="0.01" ixy="0.0" ixz="0.0" iyy="0.01" iyz="0.0" izz="0.01" />
+      </inertial>
+    </link>
+    <!-- Joint 2 -->
+    <joint name="${LEFTDYNAMIXELTOP_TO_LEFTDRIVING_JOINT_NAME}" type="revolute">
+      <parent link="${L_MISUMILN_LINK_NAME}" />
+      <child link="${L_DRIVING_LINK_NAME}" />
+      <origin
+        xyz="${MISUMILN_JOINTB_Y} 0 ${MISUMILN_Z}"
+        rpy="0 0 ${-PI/2 - ROT}" />
+      <axis xyz="0 0 1" />
+      <limit lower="-1.57" upper="1.57" effort="10" velocity="1" />
+      <mimic joint="${LEFT_DYNAMIXELBOT_TO_LEFTMISUMILN_JOINT_NAME}" multiplier="1" offset="0" />
+    </joint>
+    <!-- SECOND LINK -->
+    <link name="${L_DRIVING_LINK_NAME}">
+      <visual>
         <origin
-          xyz="${-MISUMILN_JOINTA_Y} ${-MISUMILN_JOINTA_X} 0"
+          xyz="${-MISUMIFT_JOINTB_X} ${-MISUMIFT_JOINTB_Y} 0"
           rpy="0 0 0" />
         <geometry>
           <mesh
-            filename="package://spacediver_ros2_control/description/gazebo/models/meshes/Link_MISUMI_LNMS16-10-200.STL" />
+            filename="package://spacediver_ros2_control/description/gazebo/models/meshes/Misumi_LNFTS10-P10-V10-L200-S50-W18-T9.STL" />
         </geometry>
-      </collision>
-      <xacro:inertial_box mass="${LINK_1_MASS}" x="${LINK_1_X/2}" y="${LINK_1_Y/2}"
-        z="${LINK_1_Z/2}">
-        <origin xyz="0 0 ${LINK_1_Z/2}" rpy="0 0 0" />
-      </xacro:inertial_box>
-    </link>
-    <!-- SHOULDER TO TOP DYNAMIXEL -->
-    <joint name="${LEFTSHOULDER_TO_LEFTDYNAMIXELTOP_JOINT_NAME}" type="fixed">
-      <parent link="${L_SHOULDER_LINK_NAME}" />
-      <child link="${L_TOP_DYNAMIXEL_LINK_NAME}" />
-      <origin
-        xyz="
-          ${SHOULDER_X + DYNAMIXEL_X/2}
-          ${SHOULDER_JOINTA_X - DYNAMIXEL_Y/2}
-          ${SHOULDER_Z/2 - DYNAMIXEL_Z/2}
-        "
-        rpy="0 0 0" />
-      <axis xyz="0 0 1" />
-    </joint>
-    <!-- TOP DYNAMIXEL -->
-    <link name="${L_TOP_DYNAMIXEL_LINK_NAME}">
-      <visual>
+        <material name="red">
+          <color rgba="1 0 0 1" />
+        </material>
+      </visual>
+      <inertial>
         <origin xyz="0 0 0" rpy="0 0 0" />
-        <geometry>
-          <box size="${DYNAMIXEL_X} ${DYNAMIXEL_Y} ${DYNAMIXEL_Z}" />
-        </geometry>
-        <material name="blue" />
-      </visual>
-      <collision>
-        <origin xyz="0 0 0" rpy="0 0 0" />
-        <geometry>
-          <box size="${DYNAMIXEL_X} ${DYNAMIXEL_Y} ${DYNAMIXEL_Z}" />
-        </geometry>
-      </collision>
-      <xacro:inertial_box mass="${LINK_1_MASS}" x="${LINK_1_X/2}" y="${LINK_1_Y/2}"
-        z="${LINK_1_Z/2}">
-        <origin xyz="0 0 ${LINK_1_Z/2}" rpy="0 0 0" />
-      </xacro:inertial_box>
-    </link>
-    <!-- TOP DYNAMIXEL TO DRIVING LINK -->
-    <joint name="${LEFTDYNAMIXELTOP_TO_LEFTDRIVING_JOINT_NAME}" type="revolute">
-      <parent link="${L_TOP_DYNAMIXEL_LINK_NAME}" />
-      <child link="${L_DRIVING_LINK_NAME}" />
-      <origin
-        xyz="
-        ${0}
-        ${DYNAMIXEL_JOINTB_Y-DYNAMIXEL_Y/2}
-        ${DRIVING_POS_Z - DYNAMIXEL_TOP_POS_Z}"
-        rpy="0 0 ${0}" />
-      <axis xyz="0 0 1" />
-      <limit lower="${TOP_DYNAMIXEL_LOWER}" upper="${TOP_DYNAMIXEL_UPPER}"
-        effort="${TOP_DYNAMIXEL_EFFORT}" velocity="${TOP_DYNAMIXEL_VELOCITY}" />
-    </joint>
-    <!-- DRIVING LINK -->
-    <link name="${L_DRIVING_LINK_NAME}">
-      <visual>
-        <origin
-          xyz="
-          ${-DRIVING_JOINTA_X}
-          ${-DRIVING_JOINTA_Y}
-          ${0}
-        "
-          rpy="0 0 0" />
-        <geometry>
-          <mesh
-            filename="package://spacediver_ros2_control/description/gazebo/models/meshes/upper_arm_driving_link.STL" />
-        </geometry>
-        <material name="blue" />
-      </visual>
-      <collision>
-        <origin
-          xyz="
-          ${-DRIVING_JOINTA_X}
-          ${-DRIVING_JOINTA_Y}
-          ${0}
-        "
-          rpy="0 0 0" />
-        <geometry>
-          <mesh
-            filename="package://spacediver_ros2_control/description/gazebo/models/meshes/upper_arm_driving_link.STL" />
-        </geometry>
-      </collision>
-      <xacro:inertial_box mass="${LINK_1_MASS}" x="${LINK_1_X/2}" y="${LINK_1_Y/2}"
-        z="${LINK_1_Z/2}">
-        <origin xyz="0 0 ${LINK_1_Z/2}" rpy="0 0 0" />
-      </xacro:inertial_box>
+        <mass value="1.0" />
+        <inertia ixx="0.01" ixy="0.0" ixz="0.0" iyy="0.01" iyz="0.0" izz="0.01" />
+      </inertial>
     </link>
   </xacro:macro>

File: spacediver_ros2_control/description/urdf/spacediver.urdf.xacro (robot description, xacro)
@@ -14,7 +14,7 @@
   <!-- Left Arm -->
   <xacro:include
-    filename="$(find spacediver_ros2_control)/description/urdf/parts/simple_left_arm.xacro" />
+    filename="$(find spacediver_ros2_control)/description/urdf/parts/spacediver_left_arm.xacro" />
   <xacro:left_arm base_name="base_link">
-    <origin xyz="0 0 ${BASE_Z/2}" rpy="0 0 0" />
+    <origin xyz="0 0 0" rpy="0 0 0" />
   </xacro:left_arm>
   <!-- ros2 control plugin -->

Commit message: changed starting position to PI/4

File: spacediver_ros2_control/description/urdf/macros/properties.xacro (robot description, xacro)
@@ -2,5 +2,5 @@
 <robot xmlns:xacro="http://ros.org/wiki/xacro">
   <xacro:property name="PI" value="${math.pi}"/>
-  <xacro:property name="ROT" value="${PI/6}"/>
+  <xacro:property name="ROT" value="${PI/4}"/>
   <xacro:property name="RPM" value="30"/>
   <!-- LINK NAMES -->
